File: RFBitBanger/_saved_RFBitBanger.sch (KiCad schematic (older format))
At the start: 161 parts, among them J1 POWER, J10 Conn_01x03, J11 SPEAKER, J12 Conn_Coaxial, J2 Barrel_Jack, J3 Conn_01x01, J4 Conn_01x01, J5 Conn_01x04, J6 Conn_01x01, J7 Conn_01x01, J9 ICSP, Q1 SS8050, Q2 SS9018, Q3 SS8050, Q4 S8050, Q5 SS8050, Q6 SS8050, Q7 SS8050, Q8 2N3906, SW1 SW_Push, SW2 SW_Push, SW3 SW_Push, SW4 SW_Push, SW5 SW_Push, T1 Trifilar, T2 Trifilar, U1 ATMEGA328-PU, U2 LM7805_TO220, U3 LM386, U4 LM358, U5 LCD-016N002L, U6 SI5351A, Y1 16 MHz, Y2 7.023 MHz, Y3 27 MHz

Commit message: Before changing to 74HC86
Parts:
- gave numbers to parts that had none: 1
