File: RFBitBanger/RFBitBanger.sch (KiCad schematic (older format))
At the start: 161 parts, among them J1 POWER, J10 Conn_01x03, J11 SPEAKER, J12 Conn_Coaxial, J2 Barrel_Jack, J3 Conn_01x01, J4 Conn_01x01, J5 Conn_01x04, J6 Conn_01x01, J7 Conn_01x01, J9 ICSP, Q1 SS8050, Q2 SS9018, Q3 SS8050, Q4 S8050, Q5 SS8050, Q6 SS8050, Q7 SS8050, Q8 2N3906, SW1 SW_Push, SW2 SW_Push, SW3 SW_Push, SW4 SW_Push, SW5 SW_Push, T1 Trifilar, T2 Trifilar, U1 ATMEGA328-PU, U2 LM7805_TO220, U3 LM386, U4 LM358, U5 LCD-016N002L, U6 SI5351A, Y1 16 MHz, Y2 7.023 MHz, Y3 27 MHz

Commit message: Before rearrange audio section
Parts:
- added R40: NC, Resistors_THT:R_Axial_DIN0207_L6.3mm_D2.5mm_P7.62mm_Horizontal, symbol R
- R22: value 100R -> 51R
- R5: value 1k -> 470R
Connections:
- net GND: now also R40.2
- net MUTEAUDIO: now also U1.4 ((PCINT18/INT0)PD2); no longer U1.11 ((PCINT21/OC0B/T1)PD5)
- net TRANSMIT: now also R8.2, U1.11 ((PCINT21/OC0B/T1)PD5); no longer L9.2, U1.4 ((PCINT18/INT0)PD2)
- net at C14.1, R10.2: now also L9.1; no longer R8.1
- net at R25.1, RLY1.3 (NC): now also R40.1
- new net: L9.2, R8.1
Other:
- note added: "3 TURNS"
- note added: "3 TURNS\n"
- note added: "9 TURNS\n"
- moved on the sheet: C32, L9, R8

Commit message: Added RF current sensor and Bridge Board
Parts:
- removed C27, C46: 100 nF, Capacitors_THT:C_Disc_D5.0mm_W2.5mm_P2.50mm, symbol C_Small
- removed C40: 10 nF, Capacitors_THT:C_Disc_D5.0mm_W2.5mm_P5.00mm, symbol C_Small
- added C27: 10 uF, Capacitors_THT:CP_Radial_D5.0mm_P2.50mm, symbol CP_Small
- added C39: 2.2 uH, Capacitors_THT:CP_Radial_D5.0mm_P2.50mm, symbol CP_Small
- added C40: 100 uF, Capacitors_THT:CP_Radial_D5.0mm_P2.50mm, symbol CP_Small
- added D16: LED, LEDs:LED_D3.0mm, symbol LED
- added JP2: Sample, Pin_Headers:Pin_Header_Straight_1x02_Pitch2.54mm, symbol Jumper_NC_Small
- added JP6: BYPASS, Pin_Headers:Pin_Header_Straight_1x02_Pitch2.54mm, symbol Jumper_NC_Small
- added R28: 1k, Resistors_THT:R_Axial_DIN0207_L6.3mm_D2.5mm_P7.62mm_Horizontal, symbol R
- added T3: Current, RFBitBanger:SamplingTransformer, symbol Current
- C32: value 470 pF -> 100 nF
- R21, R26, R27: value 10k -> 1k
- R32, R34: value 100k -> 10k
- RV2: value 10k -> 100k
Connections:
- net +12V: no longer D8.1 (K)
- net AUDIO: now also U4.1, C39.2; no longer R27.2, U4.7
- net AUDIOFILT: now also R24.1; no longer R27.1
- net GND: now also C43.2, D8.2 (A), RLY1.1 (Coil), C40.2, JP6.1, R28.1, T3.4 (SAMPLE); no longer C28.1, C31.1, L10.1, L8.1
- net at C29.1, C31.2, JP4.2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: now also JP2.2, T3.1 (RF); no longer J12.1 (In)
- net at C24.1, D15.1 (K), L5.2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: no longer D8.2 (A), RLY1.1 (Coil)
- net at C35.2, R23.1, R24.2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: now also U4.7; no longer U4.1
- net at C35.1, R26.1: now also U4.6 (-); no longer U4.2 (-)
- net at C45.1, R18.2, R19.1: now also U4.3 (+), U4.5 (+), C40.1; no longer U4.3 (+), U4.5 (+)
- net at C45.2, R23.2, R26.2: now also R27.1; no longer R21.1
- net at R21.2: now also C27.1
- net at C43.1: now also C32.2, R22.2, C27.2; no longer R24.1
- net at RV2.1, RV2.2: now also R21.1, U4.2 (-); no longer C43.2, U4.6 (-)
- net at Q8.3 (C), RLY1.5 (Coil): now also D8.1 (K)
- new net: C28.1, C31.1, JP6.2, L10.1, L8.1
- new net: C39.1, R27.2
- new net: J12.1 (In), JP2.1, T3.2 (RF)
- new net: D16.2 (A), T3.3 (SAMPLE)
- new net: D16.1 (K), R28.2
Other:
- moved on the sheet: C25, C33, C35, C43, C45, D8, J12, JP4, Q8, R18, R19, R21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

Commit message: Added CW decode
Parts:
- removed L5: 100 uH, Inductors_THT:L_Axial_L6.6mm_D2.7mm_P10.16mm_Horizontal_Vishay_IM-2, symbol L
- added C46: 100 nF, Capacitors_THT:C_Disc_D5.0mm_W2.5mm_P2.50mm, symbol C_Small
- added D17: 1N4148, Diodes_THT:D_DO-35_SOD27_P7.62mm_Horizontal, symbol D
- added Q9: SS8050, TO_SOT_Packages_THT:TO-92_Inline_Wide, symbol 2N3904
- added R41: 470R, Resistors_THT:R_Axial_DIN0207_L6.3mm_D2.5mm_P7.62mm_Horizontal, symbol R
- added R51: 100R, Resistors_THT:R_Axial_DIN0207_L6.3mm_D2.5mm_P7.62mm_Horizontal, symbol R
- C23: value 10 nF -> 100 nF
- R20: value 33k -> 1k
Connections:
- net GND: now also C46.1, R41.1
- net at C20.2, C38.2, L4.2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: now also C46.2, Q9.3 (C); no longer R20.1
- net at C23.2, Q3.2 (B), Q5.2 (B)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: now also D17.1 (K); no longer R20.2
- net at C24.1, D15.1 (K), Q1.3 (C)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: now also D17.2 (A)
- new net: C23.1, R51.2
- new net: JP5.2, R20.2
- new net: Q9.1 (E), R41.2, R5.2, R51.1
- new net: Q9.2 (B), R20.1
Other:
- note removed: "9 TURNS\n"
- moved on the sheet: C22, C23, C24, JP5, R17

Commit message: Cleaned up layout
Parts:
- added R52: 4k7, Resistors_THT:R_Axial_DIN0207_L6.3mm_D2.5mm_P7.62mm_Horizontal, symbol R
- added R53: 2k2, Resistors_THT:R_Axial_DIN0207_L6.3mm_D2.5mm_P7.62mm_Horizontal, symbol R
- C24: footprint Capacitors_THT:C_Disc_D5.0mm_W2.5mm_P5.00mm -> Capacitors_THT:C_Disc_D5.0mm_W2.5mm_P2.50mm
- R41: value 470R -> 220R
- R51: value 100R -> 22R
Connections:
- net at C20.2, C38.2, C46.2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: now also R52.1, R53.2
- net at C23.2, D17.1 (K), Q3.2 (B)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: now also R53.1
- net at Q9.2 (B), R20.1: now also R52.2
Changed lines of the file:
@@
 F 0 "C24" H 7810 2770 50  0000 L CNN
 F 1 "100 nF" V 7650 2550 50  0000 L CNN
-F 2 "Capacitors_THT:C_Disc_D5.0mm_W2.5mm_P5.00mm" H 7800 2700 50  0001 C CNN
+F 2 "Capacitors_THT:C_Disc_D5.0mm_W2.5mm_P2.50mm" H 7800 2700 50  0001 C CNN
 F 3 "" H 7800 2700 50  0001 C CNN
 	1    7800 2700
@@
 	9550 2250 9650 2250
 Wire Wire Line
-	7050 1600 7050 2000
+	7050 1550 7050 2000
 Wire Wire Line
 	7800 2800 7800 2850
@@
 P 6700 2550
 F 0 "R41" V 6780 2550 50  0000 C CNN
-F 1 "470R" V 6700 2550 50  0000 C CNN
+F 1 "220R" V 6700 2550 50  0000 C CNN
 F 2 "Resistors_THT:R_Axial_DIN0207_L6.3mm_D2.5mm_P7.62mm_Horizontal" V 6630 2550 50  0001 C CNN
 F 3 "" H 6700 2550 50  0001 C CNN
@@
 P 6850 2250
 F 0 "R51" V 6930 2250 50  0000 C CNN
-F 1 "100R" V 6850 2250 50  0000 C CNN
+F 1 "22R" V 6850 2250 50  0000 C CNN
 F 2 "Resistors_THT:R_Axial_DIN0207_L6.3mm_D2.5mm_P7.62mm_Horizontal" V 6780 2250 50  0001 C CNN
 F 3 "" H 6850 2250 50  0001 C CNN
@@
 Wire Wire Line
 	6850 2400 6700 2400
+$Comp
+L R R52
+U 1 1 6195474B
+P 6400 1400
+F 0 "R52" V 6480 1400 50  0000 C CNN
+F 1 "4k7" V 6400 1400 50  0000 C CNN
+F 2 "Resistors_THT:R_Axial_DIN0207_L6.3mm_D2.5mm_P7.62mm_Horizontal" V 6330 1400 50  0001 C CNN
+F 3 "" H 6400 1400 50  0001 C CNN
+	1    6400 1400
+	1    0    0    -1
+$EndComp
+Wire Wire Line
+	6400 1550 6400 1900
+Wire Wire Line
+	6400 1250 6400 1200
+Connection ~ 6400 1200
+$Comp
+L R R53
+U 1 1 61956AD8
+P 7050 1400
+F 0 "R53" V 7130 1400 50  0000 C CNN
+F 1 "2k2" V 7050 1400 50  0000 C CNN
+F 2 "Resistors_THT:R_Axial_DIN0207_L6.3mm_D2.5mm_P7.62mm_Horizontal" V 6980 1400 50  0001 C CNN
+F 3 "" H 7050 1400 50  0001 C CNN
+	1    7050 1400
+	-1   0    0    1
+$EndComp
+Connection ~ 7050 1600
+Wire Wire Line
+	7050 1250 7050 1200
+Connection ~ 7050 1200
 $EndSCHEMATC

Commit message: cwmod
Parts:
- added C48: 100 nF, Capacitors_THT:C_Disc_D5.0mm_W2.5mm_P2.50mm, symbol C_Small
- C43: value 10 uF -> 2.2 uF
- L6: value 22 uH -> 220 uH
- R24: value 1k -> 10k
Connections:
- net at D4.1 (K), D5.1 (K), D6.1 (K)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: now also C48.2; no longer Y2.2
- new net: C48.1, Y2.2
Other:
- moved on the sheet: Y2
Changed lines of the file:
@@
 L Crystal Y2
 U 1 1 6159590C
-P 5300 1950
-F 0 "Y2" H 5300 2100 50  0000 C CNN
-F 1 "7.023 MHz" V 5500 1950 50  0000 C CNN
-F 2 "Crystals:Crystal_HC49-U_Vertical" H 5300 1950 50  0001 C CNN
-F 3 "" H 5300 1950 50  0001 C CNN
-	1    5300 1950
+P 5300 1800
+F 0 "Y2" H 5300 1950 50  0000 C CNN
+F 1 "7.023 MHz" V 5500 1800 50  0000 C CNN
+F 2 "Crystals:Crystal_HC49-U_Vertical" H 5300 1800 50  0001 C CNN
+F 3 "" H 5300 1800 50  0001 C CNN
+	1    5300 1800
 	0    1    1    0
 $EndComp
@@
 P 8250 1400
 F 0 "L6" V 8200 1400 50  0000 C CNN
-F 1 "22 uH" V 8325 1400 50  0000 C CNN
+F 1 "220 uH" V 8325 1400 50  0000 C CNN
 F 2 "Inductors_THT:L_Axial_L6.6mm_D2.7mm_P10.16mm_Horizontal_Vishay_IM-2" H 8250 1400 50  0001 C CNN
 F 3 "" H 8250 1400 50  0001 C CNN
@@
 P 10700 5600
 F 0 "R24" V 10780 5600 50  0000 C CNN
-F 1 "1k" V 10700 5600 50  0000 C CNN
+F 1 "10k" V 10700 5600 50  0000 C CNN
 F 2 "Resistors_THT:R_Axial_DIN0207_L6.3mm_D2.5mm_P7.62mm_Horizontal" V 10630 5600 50  0001 C CNN
 F 3 "" H 10700 5600 50  0001 C CNN
@@
 P 7900 4550
 F 0 "C43" V 7700 4500 50  0000 L CNN
-F 1 "10 uF" V 7800 4450 50  0000 L CNN
+F 1 "2.2 uF" V 7800 4450 50  0000 L CNN
 F 2 "Capacitors_THT:CP_Radial_D5.0mm_P2.50mm" H 7900 4550 50  0001 C CNN
 F 3 "" H 7900 4550 50  0001 C CNN
@@
 Connection ~ 6000 1250
 Wire Wire Line
-	5300 1650 5300 1800
+	5300 1650 5700 1650
 Wire Wire Line
 	5550 2700 5550 2600
@@
 	5800 1900 6200 1900
 Wire Wire Line
-	5300 1650 5700 1650
-Wire Wire Line
 	5300 2650 5300 2750
 Wire Wire Line
-	5300 2100 5300 2350
+	5300 2300 5300 2350
 Connection ~ 4800 1800
 Wire Wire Line
@@
 	7050 1250 7050 1200
 Connection ~ 7050 1200
+$Comp
+L C_Small C48
+U 1 1 619BE2C2
+P 5300 2200
+F 0 "C48" V 5150 2150 50  0000 L CNN
+F 1 "100 nF" V 5400 2050 50  0000 L CNN
+F 2 "Capacitors_THT:C_Disc_D5.0mm_W2.5mm_P2.50mm" H 5300 2200 50  0001 C CNN
+F 3 "" H 5300 2200 50  0001 C CNN
+	1    5300 2200
+	1    0    0    -1
+$EndComp
+Wire Wire Line
+	5300 2100 5300 1950
 $EndSCHEMATC

Commit message: Completely remade board with common base input
Parts:
- removed C12, C14, C27: 10 uF, Capacitors_THT:CP_Radial_D5.0mm_P2.50mm, symbol CP_Small
- removed C13, C20, C23, C24, C25, C33, C38, C45, C46, C47, C48: 100 nF, Capacitors_THT:C_Disc_D5.0mm_W2.5mm_P2.50mm, symbol C_Small
- removed C21, C22, C29: 100 pF, Capacitors_THT:C_Disc_D5.0mm_W2.5mm_P5.00mm, symbol C_Small
- removed C26, C30: 10 nF, Capacitors_THT:C_Disc_D5.0mm_W2.5mm_P2.50mm, symbol C_Small
- removed C28, C31: 470 pF, Capacitors_THT:C_Disc_D5.0mm_W2.5mm_P5.00mm, symbol C_Small
- removed C32: 100 nF, Capacitors_THT:C_Disc_D5.0mm_W2.5mm_P5.00mm, symbol C_Small
- removed C35, C41: 1 nF, Capacitors_THT:C_Disc_D5.0mm_W2.5mm_P5.00mm, symbol C_Small
- removed C36: 4.7 uF, Capacitors_THT:CP_Radial_D5.0mm_P2.50mm, symbol CP_Small
- removed C39: 2.2 uH, Capacitors_THT:CP_Radial_D5.0mm_P2.50mm, symbol CP_Small
- removed C40: 100 uF, Capacitors_THT:CP_Radial_D5.0mm_P2.50mm, symbol CP_Small
- removed C43: 2.2 uF, Capacitors_THT:CP_Radial_D5.0mm_P2.50mm, symbol CP_Small
- removed D10, D11, D12, D13, D14, D17, D9: 1N4148, Diodes_THT:D_DO-35_SOD27_P7.62mm_Horizontal, symbol D
- removed D15, D4, D5, D6, D7, D8: 1N4007, Diodes_THT:D_DO-41_SOD81_P7.62mm_Horizontal, symbol D
- removed D16: LED, LEDs:LED_D3.0mm, symbol LED
- removed J12: Conn_Coaxial, RFBitBanger:bnc_90_1-1337543-0_pad_combo, symbol Conn_Coaxial
- removed JP1: QSK, Pin_Headers:Pin_Header_Straight_1x02_Pitch2.54mm, symbol Jumper_NC_Small
- removed JP2: Sample, Pin_Headers:Pin_Header_Straight_1x02_Pitch2.54mm, symbol Jumper_NC_Small
- removed JP4: BYPASS, Pin_Headers:Pin_Header_Straight_1x02_Pitch2.54mm, symbol Jumper_NO_Small
- removed JP5: JREF1, Pin_Headers:Pin_Header_Straight_1x03_Pitch2.54mm, symbol Jumper_NC_Dual
- removed JP6: BYPASS, Pin_Headers:Pin_Header_Straight_1x02_Pitch2.54mm, symbol Jumper_NC_Small
- removed L10, L8: 1 uH, Inductors_THT:L_Axial_L6.6mm_D2.7mm_P10.16mm_Horizontal_Vishay_IM-2, symbol L
- removed L3, L4, L9: 100 uH, Inductors_THT:L_Axial_L6.6mm_D2.7mm_P10.16mm_Horizontal_Vishay_IM-2, symbol L
- removed L6: 220 uH, Inductors_THT:L_Axial_L6.6mm_D2.7mm_P10.16mm_Horizontal_Vishay_IM-2, symbol L
- removed L7: 4.7 uH, Inductors_THT:L_Axial_L6.6mm_D2.7mm_P10.16mm_Horizontal_Vishay_IM-2, symbol L
- removed Q1, Q3, Q5, Q6, Q7, Q9: SS8050, TO_SOT_Packages_THT:TO-92_Inline_Wide, symbol 2N3904
- removed Q2: SS9018, TO_SOT_Packages_THT:TO-92_Inline_Wide, symbol 2N3904
- removed Q8: 2N3906, TO_SOT_Packages_THT:TO-92_Inline_Wide, symbol 2N3906
- removed R10, R17, R5, R8: 470R, Resistors_THT:R_Axial_DIN0207_L6.3mm_D2.5mm_P7.62mm_Horizontal, symbol R
- removed R14, R40, R50: NC, Resistors_THT:R_Axial_DIN0207_L6.3mm_D2.5mm_P7.62mm_Horizontal, symbol R
- removed R15: 47k, Resistors_THT:R_Axial_DIN0207_L6.3mm_D2.5mm_P7.62mm_Horizontal, symbol R
- removed R16: 470k, Resistors_THT:R_Axial_DIN0207_L6.3mm_D2.5mm_P7.62mm_Horizontal, symbol R
- removed R18, R19, R20, R21, R26, R27, R28, R36, R37: 1k, Resistors_THT:R_Axial_DIN0207_L6.3mm_D2.5mm_P7.62mm_Horizontal, symbol R
- removed R22, R25: 51R, Resistors_THT:R_Axial_DIN0207_L6.3mm_D2.5mm_P7.62mm_Horizontal, symbol R
- removed R23: 220k, Resistors_THT:R_Axial_DIN0207_L6.3mm_D2.5mm_P7.62mm_Horizontal, symbol R
- removed R24, R35, R48, R7: 10k, Resistors_THT:R_Axial_DIN0207_L6.3mm_D2.5mm_P7.62mm_Horizontal, symbol R
- removed R38: 33R, Resistors_THT:R_Axial_DIN0207_L6.3mm_D2.5mm_P7.62mm_Horizontal, symbol R
- removed R39: 22k, Resistors_THT:R_Axial_DIN0207_L6.3mm_D2.5mm_P7.62mm_Horizontal, symbol R
- removed R41: 220R, Resistors_THT:R_Axial_DIN0207_L6.3mm_D2.5mm_P7.62mm_Horizontal, symbol R
- removed R42, R43, R44, R45: 0R5, Resistors_THT:R_Axial_DIN0207_L6.3mm_D2.5mm_P7.62mm_Horizontal, symbol R
- removed R49: 0R, Resistors_THT:R_Axial_DIN0207_L6.3mm_D2.5mm_P7.62mm_Horizontal, symbol R
- removed R51: 22R, Resistors_THT:R_Axial_DIN0207_L6.3mm_D2.5mm_P7.62mm_Horizontal, symbol R
- removed R52: 4k7, Resistors_THT:R_Axial_DIN0207_L6.3mm_D2.5mm_P7.62mm_Horizontal, symbol R
- removed R53: 2k2, Resistors_THT:R_Axial_DIN0207_L6.3mm_D2.5mm_P7.62mm_Horizontal, symbol R
- removed R9: 100k, Resistors_THT:R_Axial_DIN0207_L6.3mm_D2.5mm_P7.62mm_Horizontal, symbol R
- removed RLY1: DPDTRelay, RFBitBanger:G2VRelay, symbol DPDTRelay
- removed RV2: 100k, Potentiometers:Potentiometer_WirePads, symbol POT
- removed T1, T2: Trifilar, RFBitBanger:TripleWindingTransformer, symbol TripleWindingTransformer
- removed T3: Current, RFBitBanger:SamplingTransformer, symbol Current
- removed U4: LM358, Housings_DIP:DIP-8_W7.62mm_Socket, symbol LM358
- removed U6: SI5351A, Housings_SSOP:MSOP-10_3x3mm_Pitch0.5mm, symbol SI5351A
- removed Y2: 7.023 MHz, Crystals:Crystal_HC49-U_Vertical, symbol Crystal
- removed Y3: 27 MHz, Crystals:Crystal_HC49-U_Vertical, symbol Crystal
- added C57: 10 nF, Capacitors_THT:C_Disc_D5.0mm_W2.5mm_P2.50mm, symbol C_Small
- added J13, J8: Conn_01x01, Connectors:1pin, symbol Conn_01x01
- added P1: Mini-DIN_6pins_ver4, RFBitBanger:Connector_Mini-DIN_Female_6Pin_2rows, symbol Mini-DIN_6pins_ver4
- added R64, R70: 10k, Resistors_THT:R_Axial_DIN0207_L6.3mm_D2.5mm_P7.62mm_Horizontal, symbol R
- Q4: value S8050 -> 2N3904
Connections:
- net +5V: now also P1.4, R64.2, R70.1
- net DB4: now also U1.11 ((PCINT21/OC0B/T1)PD5); no longer U1.13 ((PCINT23/AIN1)PD7)
- net DB5: now also U1.12 ((PCINT22/OC0A/AIN0)PD6); no longer U1.14 ((PCINT0/CLKO/ICP1)PB0)
- net DB6: now also U1.13 ((PCINT23/AIN1)PD7); no longer U1.15 ((PCINT1/OC1A)PB1)
- net DB7: now also U1.14 ((PCINT0/CLKO/ICP1)PB0); no longer U1.16 ((PCINT2/OC1B/~SS~)PB2)
- net E: now also U1.25 ((PCINT10/ADC2)PC2); no longer U1.26 ((PCINT11/ADC3)PC3)
- net GND: now also C57.2, P1.3, P1.7 (Shell)
- net MISO: now also P1.1, R70.2
- net MUTEAUDIO: now also U1.6 ((PCINT20/XCK/T0)PD4); no longer U1.4 ((PCINT18/INT0)PD2)
- net RS: now also U1.26 ((PCINT11/ADC3)PC3); no longer U1.25 ((PCINT10/ADC2)PC2)
- net TRANSMIT: now also U1.15 ((PCINT1/OC1A)PB1); no longer U1.11 ((PCINT21/OC0B/T1)PD5)
- net TUNING: now also U1.16 ((PCINT2/OC1B/~SS~)PB2); no longer U1.12 ((PCINT22/OC0A/AIN0)PD6)
- net at Q4.3 (C), R32.2, R34.1: now also C57.1
- new net PS2CLK: P1.5, R64.1, U1.4 ((PCINT18/INT0)PD2)
Other:
- note removed: "3 TURNS"
- note removed: "3 TURNS\n"
- note removed: "ALTERNATE SI5351A\nOSCILLATOR"
- note removed: "AMPLIFIER AND OUTPUT FILTER"
- note removed: "AUDIO AMPLIFICATION"
- note removed: "BALANCED\nRING MIXER"
- note removed: "COLPITTS CRYSTAL\nOSCILLATOR"
- note removed: "VALUES FOR 40 M BAND\nFOR 80 M BAND:\nL8,L10=1.2 uH, C28,C31=1500 pF\nL7=12 uH, C29=150 pF"
- moved on the sheet: C1, C10, C11, C15, C16, C17, C18, C19, C2, C3, C34, C37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

Commit message: Started RFBitBanger code project
Parts:
- C10, C11, C16, C17: value 10 nF -> 100 nF
- R12, R13, R33, R6: value 10k -> 1k
- R29, R3, R46, R47: value 100k -> 10k
Changed lines of the file:
@@
 P 7500 1650
 F 0 "C10" H 7510 1720 50  0000 L CNN
-F 1 "10 nF" V 7350 1600 50  0000 L CNN
+F 1 "100 nF" V 7350 1600 50  0000 L CNN
 F 2 "Capacitors_THT:C_Disc_D5.0mm_W2.5mm_P2.50mm" H 7500 1650 50  0001 C CNN
 F 3 "" H 7500 1650 50  0001 C CNN
@@
 P 7750 1300
 F 0 "R6" V 7830 1300 50  0000 C CNN
-F 1 "10k" V 7750 1300 50  0000 C CNN
+F 1 "1k" V 7750 1300 50  0000 C CNN
 F 2 "Resistors_THT:R_Axial_DIN0207_L6.3mm_D2.5mm_P7.62mm_Horizontal" V 7680 1300 50  0001 C CNN
 F 3 "" H 7750 1300 50  0001 C CNN
@@
 P 8700 1600
 F 0 "C16" H 8500 1700 50  0000 L CNN
-F 1 "10 nF" V 8850 1600 50  0000 L CNN
+F 1 "100 nF" V 8850 1600 50  0000 L CNN
 F 2 "Capacitors_THT:C_Disc_D5.0mm_W2.5mm_P2.50mm" H 8700 1600 50  0001 C CNN
 F 3 "" H 8700 1600 50  0001 C CNN
@@
 P 8950 1300
 F 0 "R12" V 9030 1300 50  0000 C CNN
-F 1 "10k" V 8950 1300 50  0000 C CNN
+F 1 "1k" V 8950 1300 50  0000 C CNN
 F 2 "Resistors_THT:R_Axial_DIN0207_L6.3mm_D2.5mm_P7.62mm_Horizontal" V 8880 1300 50  0001 C CNN
 F 3 "" H 8950 1300 50  0001 C CNN
@@
 P 8700 2550
 F 0 "C17" H 8800 2550 50  0000 L CNN
-F 1 "10 nF" V 8600 2500 50  0000 L CNN
+F 1 "100 nF" V 8600 2500 50  0000 L CNN
 F 2 "Capacitors_THT:C_Disc_D5.0mm_W2.5mm_P2.50mm" H 8700 2550 50  0001 C CNN
 F 3 "" H 8700 2550 50  0001 C CNN
@@
 P 8950 2200
 F 0 "R13" V 9030 2200 50  0000 C CNN
-F 1 "10k" V 8950 2200 50  0000 C CNN
+F 1 "1k" V 8950 2200 50  0000 C CNN
 F 2 "Resistors_THT:R_Axial_DIN0207_L6.3mm_D2.5mm_P7.62mm_Horizontal" V 8880 2200 50  0001 C CNN
 F 3 "" H 8950 2200 50  0001 C CNN
@@
 P 7500 2500
 F 0 "C11" H 7510 2570 50  0000 L CNN
-F 1 "10 nF" V 7350 2450 50  0000 L CNN
+F 1 "100 nF" V 7350 2450 50  0000 L CNN
 F 2 "Capacitors_THT:C_Disc_D5.0mm_W2.5mm_P2.50mm" H 7500 2500 50  0001 C CNN
 F 3 "" H 7500 2500 50  0001 C CNN
@@
 P 7750 2150
 F 0 "R33" V 7830 2150 50  0000 C CNN
-F 1 "10k" V 7750 2150 50  0000 C CNN
+F 1 "1k" V 7750 2150 50  0000 C CNN
 F 2 "Resistors_THT:R_Axial_DIN0207_L6.3mm_D2.5mm_P7.62mm_Horizontal" V 7680 2150 50  0001 C CNN
 F 3 "" H 7750 2150 50  0001 C CNN
@@
 P 7300 1550
 F 0 "R29" V 7380 1550 50  0000 C CNN
-F 1 "100k" V 7300 1550 50  0000 C CNN
+F 1 "10k" V 7300 1550 50  0000 C CNN
 F 2 "Resistors_THT:R_Axial_DIN0207_L6.3mm_D2.5mm_P7.62mm_Horizontal" V 7230 1550 50  0001 C CNN
 F 3 "" H 7300 1550 50  0001 C CNN
@@
 P 8500 1500
 F 0 "R47" V 8580 1500 50  0000 C CNN
-F 1 "100k" V 8500 1500 50  0000 C CNN
+F 1 "10k" V 8500 1500 50  0000 C CNN
 F 2 "Resistors_THT:R_Axial_DIN0207_L6.3mm_D2.5mm_P7.62mm_Horizontal" V 8430 1500 50  0001 C CNN
 F 3 "" H 8500 1500 50  0001 C CNN
@@
 P 7250 2350
 F 0 "R3" V 7330 2350 50  0000 C CNN
-F 1 "100k" V 7250 2350 50  0000 C CNN
+F 1 "10k" V 7250 2350 50  0000 C CNN
 F 2 "Resistors_THT:R_Axial_DIN0207_L6.3mm_D2.5mm_P7.62mm_Horizontal" V 7180 2350 50  0001 C CNN
 F 3 "" H 7250 2350 50  0001 C CNN
@@
 P 8450 2400
 F 0 "R46" V 8530 2400 50  0000 C CNN
-F 1 "100k" V 8450 2400 50  0000 C CNN
+F 1 "10k" V 8450 2400 50  0000 C CNN
 F 2 "Resistors_THT:R_Axial_DIN0207_L6.3mm_D2.5mm_P7.62mm_Horizontal" V 8380 2400 50  0001 C CNN
 F 3 "" H 8450 2400 50  0001 C CNN

Commit message: Added bias potentiometer and user interface
Parts:
- added Q14: 2N3904, TO_SOT_Packages_THT:TO-92_Inline_Wide, symbol 2N3904
- added R72: 10k, Resistors_THT:R_Axial_DIN0207_L6.3mm_D2.5mm_P7.62mm_Horizontal, symbol R
Connections:
- net GND: now also Q14.1 (E); no longer U5.16 (K)
- net MOSI: now also R72.2
- new net: Q14.3 (C), U5.16 (K)
- new net: Q14.2 (B), R72.1
Changed lines of the file:
@@
 SCL
-$Comp
-L GND #PWR25
-U 1 1 616D2D06
-P 6150 6200
-F 0 "#PWR25" H 6150 5950 50  0001 C CNN
-F 1 "GND" H 6150 6050 50  0000 C CNN
-F 2 "" H 6150 6200 50  0001 C CNN
-F 3 "" H 6150 6200 50  0001 C CNN
-	1    6150 6200
-	1    0    0    -1
-$EndComp
 $Comp
 L Conn_01x03 J10
@@
 	1    0    0    -1
 $EndComp
+$Comp
+L 2N3904 Q14
+U 1 1 61C6B72A
+P 6250 6400
+F 0 "Q14" H 6100 6250 50  0000 L CNN
+F 1 "2N3904" H 6050 6150 50  0000 L CNN
+F 2 "TO_SOT_Packages_THT:TO-92_Inline_Wide" H 6450 6325 50  0001 L CIN
+F 3 "" H 6250 6400 50  0001 L CNN
+	1    6250 6400
+	-1   0    0    -1
+$EndComp
+$Comp
+L GND #PWR25
+U 1 1 616D2D06
+P 6150 6750
+F 0 "#PWR25" H 6150 6500 50  0001 C CNN
+F 1 "GND" H 6150 6600 50  0000 C CNN
+F 2 "" H 6150 6750 50  0001 C CNN
+F 3 "" H 6150 6750 50  0001 C CNN
+	1    6150 6750
+	1    0    0    -1
+$EndComp
+Wire Wire Line
+	6150 6750 6150 6600
+$Comp
+L R R72
+U 1 1 61C6C093
+P 6600 6200
+F 0 "R72" V 6680 6200 50  0000 C CNN
+F 1 "10k" V 6600 6200 50  0000 C CNN
+F 2 "Resistors_THT:R_Axial_DIN0207_L6.3mm_D2.5mm_P7.62mm_Horizontal" V 6530 6200 50  0001 C CNN
+F 3 "" H 6600 6200 50  0001 C CNN
+	1    6600 6200
+	-1   0    0    1
+$EndComp
+Wire Wire Line
+	6600 6350 6600 6400
+Wire Wire Line
+	6600 6400 6450 6400
+Text GLabel 6600 5950 1    60   Input ~ 0
+MOSI
+Wire Wire Line
+	6600 5950 6600 6050
 $EndSCHEMATC
