File: RFBitBanger/RFBitBanger.sch (KiCad schematic (older format))
At the start: 73 parts, among them J1 POWER, J10 Conn_01x03, J11 SPEAKER, J13 Conn_01x01, J2 Barrel_Jack, J3 Conn_01x01, J4 Conn_01x01, J5 Conn_01x04, J6 Conn_01x01, J7 Conn_01x01, J8 Conn_01x01, J9 ICSP, P1 Mini-DIN_6pins_ver4, Q14 2N3904, Q4 2N3904, SW1 SW_Push, SW2 SW_Push, SW3 SW_Push, SW4 SW_Push, SW5 SW_Push, U1 ATMEGA328-PU, U2 LM7805_TO220, U3 LM386, U5 LCD-016N002L, Y1 16 MHz

Commit message: Added common mode choke, put back LPF
Parts:
- added C41: 10 nF, Capacitors_THT:C_Disc_D5.0mm_W2.5mm_P5.00mm, symbol C_Small
- added C58: 100 nF, Capacitors_THT:C_Disc_D5.0mm_W2.5mm_P2.50mm, symbol C_Small
- added T4: Common-Mode Choke, RFBitBanger:DoubleWindingTransformer, symbol DoubleWindingTransformer
Connections:
- net +12V: now also T4.2; no longer J1.2 (Pin_2), J2.1
- net GND: now also J3.1 (Pin_1), J4.1 (Pin_1), J6.1 (Pin_1), J7.1 (Pin_1), C41.2, T4.4; no longer J1.1 (Pin_1), J2.2
- net at C19.2, J11.1 (Pin_1): now also C41.1
- new net: C58.2, J1.2 (Pin_2), J2.1, T4.1
- new net: C58.1, J1.1 (Pin_1), J2.2, T4.3
Other:
- moved on the sheet: C3, C44, C6, D1, D3, J1, J11, J2, R4, U2

Commit message: Added overvoltage zener and extra key inputs
Parts:
- removed J10: Conn_01x03, Pin_Headers:Pin_Header_Straight_1x03_Pitch2.54mm, symbol Conn_01x03
- added C59: 100 nF, Capacitors_THT:C_Disc_D5.0mm_W2.5mm_P2.50mm, symbol C_Small
- added J10: Conn_01x05, Pin_Headers:Pin_Header_Straight_1x05_Pitch2.54mm, symbol Conn_01x05
- added R75, R76: 1k, Resistors_THT:R_Axial_DIN0207_L6.3mm_D2.5mm_P7.62mm_Horizontal, symbol R
Connections:
- net +5V: now also C59.1, J10.3 (Pin_3)
- net GND: now also C59.2, J10.5 (Pin_5)
- net MOSI: now also R75.2
- net SCK: now also R76.2
- net at C7.2, U1.24 ((PCINT9/ADC1)PC1): now also J10.4 (Pin_4)
- new net: J10.1 (Pin_1), R75.1
- new net: J10.2 (Pin_2), R76.1
Other:
- moved on the sheet: C7

Commit message: Fixed overcommited MOSI pin
Parts:
- removed J10: Conn_01x05, Pin_Headers:Pin_Header_Straight_1x05_Pitch2.54mm, symbol Conn_01x05
- removed R75: 1k, Resistors_THT:R_Axial_DIN0207_L6.3mm_D2.5mm_P7.62mm_Horizontal, symbol R
- added J10: Conn_01x04, Pin_Headers:Pin_Header_Straight_1x04_Pitch2.54mm, symbol Conn_01x04
Connections:
- net +5V: now also J10.2 (Pin_2)
- net GND: now also J10.4 (Pin_4)
- net at C7.2, U1.24 ((PCINT9/ADC1)PC1): now also J10.3 (Pin_3)
- net at R76.1: now also J10.1 (Pin_1)
Changed lines of the file:
@@
 Wire Wire Line
 	2200 6150 2200 6200
-$Comp
-L Conn_01x05 J10
-U 1 1 61CE6260
-P 4800 2900
-F 0 "J10" H 4800 3200 50  0000 C CNN
-F 1 "Conn_01x05" H 4800 2600 50  0000 C CNN
-F 2 "Pin_Headers:Pin_Header_Straight_1x05_Pitch2.54mm" H 4800 2900 50  0001 C CNN
-F 3 "" H 4800 2900 50  0001 C CNN
-	1    4800 2900
-	1    0    0    -1
-$EndComp
 Wire Wire Line
 	3950 2800 3950 2900
@@
 Wire Wire Line
 	3250 2650 3200 2650
-Text GLabel 4150 3500 3    60   Input ~ 0
-MOSI
 Text GLabel 4300 3500 3    60   Input ~ 0
 SCK
-$Comp
-L R R75
-U 1 1 61CE922E
-P 4150 3300
-F 0 "R75" V 4230 3300 50  0000 C CNN
-F 1 "1k" V 4150 3300 50  0000 C CNN
-F 2 "Resistors_THT:R_Axial_DIN0207_L6.3mm_D2.5mm_P7.62mm_Horizontal" V 4080 3300 50  0001 C CNN
-F 3 "" H 4150 3300 50  0001 C CNN
-	1    4150 3300
-	1    0    0    -1
-$EndComp
 $Comp
 L R R76
@@
 	4300 2800 4600 2800
 Wire Wire Line
-	4150 3150 4150 2700
-Wire Wire Line
-	4150 2700 4600 2700
-Wire Wire Line
 	4300 3450 4300 3500
-Wire Wire Line
-	4150 3450 4150 3500
+$Comp
+L Conn_01x04 J10
+U 1 1 61D154E8
+P 4800 2900
+F 0 "J10" H 4800 3100 50  0000 C CNN
+F 1 "Conn_01x04" H 4800 2600 50  0000 C CNN
+F 2 "Pin_Headers:Pin_Header_Straight_1x04_Pitch2.54mm" H 4800 2900 50  0001 C CNN
+F 3 "" H 4800 2900 50  0001 C CNN
+	1    4800 2900
+	1    0    0    -1
+$EndComp
 $EndSCHEMATC

Commit message: Lots of changes...
Parts:
- removed C18: 100 nF, Capacitors_THT:C_Disc_D5.0mm_W2.5mm_P2.50mm, symbol C_Small
- removed C57: 10 nF, Capacitors_THT:C_Disc_D5.0mm_W2.5mm_P2.50mm, symbol C_Small
- added C18: 1 uF, Capacitors_THT:CP_Radial_D5.0mm_P2.50mm, symbol CP_Small
- added C53: 100 uF, Capacitors_THT:CP_Radial_D5.0mm_P2.50mm, symbol CP_Small
- added J14, J15, J16: Conn_01x01, Pin_Headers:Pin_Header_Straight_1x01_Pitch2.54mm, symbol Conn_01x01
- added L10: 100 uH, Inductors_THT:L_Axial_L6.6mm_D2.7mm_P10.16mm_Horizontal_Vishay_IM-2, symbol L
- C3: value 100 uF -> 1000 uF; footprint Capacitors_THT:CP_Radial_D5.0mm_P2.50mm -> Capacitors_THT:CP_Radial_D8.0mm_P3.50mm
- C41: value 10 nF -> 100 nF
- C7: value 10 nF -> 1 nF; footprint Capacitors_THT:C_Disc_D5.0mm_W2.5mm_P2.50mm -> Capacitors_THT:C_Disc_D5.0mm_W2.5mm_P5.00mm
- R11: value 10R -> 47R
- R30, R31: value 100k -> 10k
- R32, R34: value 10k -> 1k
Connections:
- net +12V: now also C53.1
- net AUDIOFILT: now also J14.1 (Pin_1)
- net GND: now also C18.2, C53.2, J15.1 (Pin_1), J16.1 (Pin_1); no longer R11.1
- net at C19.2, J11.1 (Pin_1): no longer C41.1
- net at U3.5: now also R11.2, L10.1; no longer C19.1
- net at Q4.3 (C), R32.2, R34.1: now also C18.1
- new net: C19.1, C41.1, L10.2, R11.1
Other:
- moved on the sheet: C19, C41, J11

Commit message: Implemented timers, fixed beep audio, fixed key shaping
Parts:
- C15: value NC -> 10 uF
- P1: footprint RFBitBanger:Connector_Mini-DIN_Female_6Pin_2rows -> MiniDin 6
- R31: value 10k -> 220k
Other:
- note added: "AUDIO AMPLIFIER OUTPUT"
- note added: "HD44780 DISPLAY\nAND PUSHBUTTONS"
- note added: "POWER SUPPLY AND FILTER"
- note added: "PS/2 KEYBOARD\nCONNECTOR"
- note added: "RFBITBANGER\n20m to 80m BAND\nDRAFT V5 BY KW4TI"
- note removed: "ARDUINO OOK/FSK TRANSMISSION RECEPTION\n40/80 METER BAND\nDRAFT V3 BY KW4TI"
- moved on the sheet: C1, C10, C11, C15, C16, C17, C18, C19, C2, C3, C34, C37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
