File: RFBitBanger/RFBitBanger.sch (KiCad schematic (older format))
At the start: 82 parts, among them J1 POWER, J10 Conn_01x04, J11 SPEAKER, J13 Conn_01x01, J14 Conn_01x01, J15 Conn_01x01, J16 Conn_01x01, J2 Barrel_Jack, J3 Conn_01x01, J4 Conn_01x01, J5 Conn_01x04, J6 Conn_01x01, J7 Conn_01x01, J8 Conn_01x01, J9 ICSP, P1 Mini-DIN_6pins_ver4, Q14 2N3904, Q4 2N3904, SW1 SW_Push, SW2 SW_Push, SW3 SW_Push, SW4 SW_Push, SW5 SW_Push, T4 Common-Mode Choke, U1 ATMEGA328-PU, U2 LM7805_TO220, U3 LM386, U5 LCD-016N002L, Y1 16 MHz

Commit message: Rearranged parts for better layout
Parts:
- added C57: 100 nF, Capacitors_THT:C_Disc_D5.0mm_W2.5mm_P2.50mm, symbol C_Small
- added J19: Conn_01x04, Pin_Headers:Pin_Header_Straight_1x04_Pitch2.54mm, symbol Conn_01x04
Connections:
- net GND: now also C57.2, J19.4 (Pin_4)
- net at U1.21 (AREF): now also C57.1
Other:
- moved on the sheet: C1, C59

Commit message: Changed DSP to higher audible frequencies
Parts:
- removed C18: 1 uF, Capacitors_THT:CP_Radial_D5.0mm_P2.50mm, symbol CP_Small
- added C18, C?: NC, Capacitors_THT:C_Disc_D5.0mm_W2.5mm_P5.00mm, symbol C_Small
- added R?: 100k, Resistors_THT:R_Axial_DIN0207_L6.3mm_D2.5mm_P7.62mm_Horizontal, symbol R
- C15: value 10 uF -> NC
- R31: value 220k -> 100k
- R32, R34: value 1k -> 100k
Connections:
- net BEEPOUT: now also R?.1; no longer R31.1
- net GND: now also C18.2, C?.1
- net at Q4.3 (C), R32.2, R34.1: now also C18.1
- new net: C?.2, R31.1, R?.2
Changed lines of the file:
@@
 P 8850 4050
 F 0 "C15" H 8860 4120 50  0000 L CNN
-F 1 "10 uF" V 8700 3950 50  0000 L CNN
+F 1 "NC" V 8700 3950 50  0000 L CNN
 F 2 "Capacitors_THT:CP_Radial_D5.0mm_P2.50mm" H 8850 4050 50  0001 C CNN
 F 3 "" H 8850 4050 50  0001 C CNN
@@
 	1    0    0    -1
 $EndComp
-Text GLabel 7600 2850 0    60   Input ~ 0
+Text GLabel 7250 2850 0    60   Input ~ 0
 BEEPOUT
 Text GLabel 3200 4500 2    60   Input ~ 0
@@
 P 7900 2850
 F 0 "R31" V 7980 2850 50  0000 C CNN
-F 1 "220k" V 7900 2850 50  0000 C CNN
+F 1 "100k" V 7900 2850 50  0000 C CNN
 F 2 "Resistors_THT:R_Axial_DIN0207_L6.3mm_D2.5mm_P7.62mm_Horizontal" V 7830 2850 50  0001 C CNN
 F 3 "" H 7900 2850 50  0001 C CNN
@@
 P 7900 3100
 F 0 "R34" V 7980 3100 50  0000 C CNN
-F 1 "1k" V 7900 3100 50  0000 C CNN
+F 1 "100k" V 7900 3100 50  0000 C CNN
 F 2 "Resistors_THT:R_Axial_DIN0207_L6.3mm_D2.5mm_P7.62mm_Horizontal" V 7830 3100 50  0001 C CNN
 F 3 "" H 7900 3100 50  0001 C CNN
@@
 P 7500 3100
 F 0 "R32" V 7580 3100 50  0000 C CNN
-F 1 "1k" V 7500 3100 50  0000 C CNN
+F 1 "100k" V 7500 3100 50  0000 C CNN
 F 2 "Resistors_THT:R_Axial_DIN0207_L6.3mm_D2.5mm_P7.62mm_Horizontal" V 7430 3100 50  0001 C CNN
 F 3 "" H 7500 3100 50  0001 C CNN
@@
 F 3 "" H 5050 3700 50  0001 C CNN
 	1    5050 3700
-	1    0    0    -1
-$EndComp
-$Comp
-L GND #PWR34
-U 1 1 61C12E08
-P 7550 3500
-F 0 "#PWR34" H 7550 3250 50  0001 C CNN
-F 1 "GND" H 7550 3350 50  0000 C CNN
-F 2 "" H 7550 3500 50  0001 C CNN
-F 3 "" H 7550 3500 50  0001 C CNN
-	1    7550 3500
 	1    0    0    -1
 $EndComp
@@
 	8050 2850 8100 2850
 Wire Wire Line
-	7750 2850 7600 2850
-Wire Wire Line
 	3200 4800 3150 4800
 Wire Wire Line
@@
 Wire Wire Line
 	7350 3100 7300 3100
-Wire Wire Line
-	7550 3500 7550 3450
-Wire Wire Line
-	7550 3250 7750 3250
-Connection ~ 7750 3250
 Wire Wire Line
 	3200 4600 3150 4600
@@
 Wire Wire Line
 	10700 6200 10350 6200
-$Comp
-L CP_Small C18
-U 1 1 61DBA4EB
-P 7550 3350
-F 0 "C18" H 7560 3420 50  0000 L CNN
-F 1 "1 uF" V 7400 3250 50  0000 L CNN
-F 2 "Capacitors_THT:CP_Radial_D5.0mm_P2.50mm" H 7550 3350 50  0001 C CNN
-F 3 "" H 7550 3350 50  0001 C CNN
-	1    7550 3350
-	1    0    0    -1
-$EndComp
 Wire Notes Line
 	1250 7700 6200 7700
@@
 Wire Wire Line
 	1250 3750 1250 3850
+$Comp
+L C_Small C18
+U 1 1 61E326D6
+P 7500 3400
+F 0 "C18" H 7510 3470 50  0000 L CNN
+F 1 "NC" V 7400 3300 50  0000 L CNN
+F 2 "Capacitors_THT:C_Disc_D5.0mm_W2.5mm_P5.00mm" H 7500 3400 50  0001 C CNN
+F 3 "" H 7500 3400 50  0001 C CNN
+	1    7500 3400
+	1    0    0    -1
+$EndComp
+$Comp
+L GND #PWR34
+U 1 1 61E32AAF
+P 7500 3550
+F 0 "#PWR34" H 7500 3300 50  0001 C CNN
+F 1 "GND" H 7500 3400 50  0000 C CNN
+F 2 "" H 7500 3550 50  0001 C CNN
+F 3 "" H 7500 3550 50  0001 C CNN
+	1    7500 3550
+	1    0    0    -1
+$EndComp
+Wire Wire Line
+	7500 3500 7500 3550
+Wire Wire Line
+	7500 3300 7500 3200
+Wire Wire Line
+	7500 3200 7750 3200
+Connection ~ 7750 3200
+$Comp
+L R R?
+U 1 1 61E35D66
+P 7500 2850
+F 0 "R?" V 7580 2850 50  0000 C CNN
+F 1 "100k" V 7500 2850 50  0000 C CNN
+F 2 "Resistors_THT:R_Axial_DIN0207_L6.3mm_D2.5mm_P7.62mm_Horizontal" V 7430 2850 50  0001 C CNN
+F 3 "" H 7500 2850 50  0001 C CNN
+	1    7500 2850
+	0    -1   -1   0
+$EndComp
+Wire Wire Line
+	7750 2850 7650 2850
+Wire Wire Line
+	7350 2850 7250 2850
+$Comp
+L C_Small C?
+U 1 1 61E361F6
+P 7700 2650
+F 0 "C?" H 7710 2720 50  0000 L CNN
+F 1 "NC" V 7600 2550 50  0000 L CNN
+F 2 "Capacitors_THT:C_Disc_D5.0mm_W2.5mm_P5.00mm" H 7700 2650 50  0001 C CNN
+F 3 "" H 7700 2650 50  0001 C CNN
+	1    7700 2650
+	1    0    0    -1
+$EndComp
+Wire Wire Line
+	7700 2750 7700 2850
+Connection ~ 7700 2850
+$Comp
+L GND #PWR?
+U 1 1 61E3659E
+P 7450 2500
+F 0 "#PWR?" H 7450 2250 50  0001 C CNN
+F 1 "GND" H 7450 2350 50  0000 C CNN
+F 2 "" H 7450 2500 50  0001 C CNN
+F 3 "" H 7450 2500 50  0001 C CNN
+	1    7450 2500
+	1    0    0    -1
+$EndComp
+Wire Wire Line
+	7450 2500 7700 2500
+Wire Wire Line
+	7700 2500 7700 2550
 $EndSCHEMATC

Commit message: Added Display Board on Top
Parts:
- added J20, J21: Conn_01x01, Connectors:1pin, symbol Conn_01x01
- added J22: SPEAKER, Pin_Headers:Pin_Header_Straight_1x02_Pitch2.54mm, symbol Conn_01x02
- RV1: footprint Potentiometers:Potentiometer_WirePads -> RFBitBanger:Potentiometer_Big_Small_Combined
- gave numbers to parts that had none: 2
Connections:
- net GND: now also J20.1 (Pin_1), J21.1 (Pin_1), J22.2 (Pin_2)
- net at C19.2, J11.1 (Pin_1): now also J22.1 (Pin_1)

Commit message: Changed external connector for single 20 pin or ribbon cable
Parts:
- removed J10, J19: Conn_01x04, Pin_Headers:Pin_Header_Straight_1x04_Pitch2.54mm, symbol Conn_01x04
- removed J22: SPEAKER, Pin_Headers:Pin_Header_Straight_1x02_Pitch2.54mm, symbol Conn_01x02
- removed U5: LCD-016N002L, Pin_Headers:Pin_Header_Straight_1x16_Pitch2.54mm, symbol LCD-016N002L
- added U5: LCD1602ExtraPins, Pin_Headers:Pin_Header_Straight_1x20_Pitch2.54mm, symbol LCD1602ExtraPins
Connections:
- net +5V: now also U5.2 (VDD)
- net DB4: now also U5.11 (DB4)
- net DB5: now also U5.12 (DB5)
- net DB6: now also U5.13 (DB6)
- net DB7: now also U5.14 (DB7)
- net E: now also U5.6 (E)
- net GND: now also U5.1 (VSS), U5.17, U5.5 (R/~W)
- net RS: now also U5.4 (RS)
- net MICPADDLE: now reaches C7.2, U1.24 ((PCINT9/ADC1)PC1)
- net MICPADDLE: now also U5.18
- net SPKR: now reaches C19.2, J11.1 (Pin_1)
- net SPKR: now also U5.20
- net at R2.1: now also U5.15 (A/VEE)
- net at Q14.3 (C): now also U5.16 (K)
- net at RV3.2: now also U5.3 (VO)
- net at R76.1: now also U5.19
Other:
- moved on the sheet: Q14, R72, R76

Commit message: Added fifth button
Parts:
- added C61: 100 nF, Capacitors_THT:C_Disc_D5.0mm_W2.5mm_P2.50mm, symbol C_Small
- added R40: 10k, Resistors_THT:R_Axial_DIN0207_L6.3mm_D2.5mm_P7.62mm_Horizontal, symbol R
- added R75: 1k, Resistors_THT:R_Axial_DIN0207_L6.3mm_D2.5mm_P7.62mm_Horizontal, symbol R
- added SW6: SW_Push, Buttons_Switches_THT:SW_PUSH_6mm, symbol SW_Push
Connections:
- net +5V: now also R75.2
- net GND: now also C61.1, SW6.2
- net RS: now also R40.2
- new net: C61.2, R40.1, R75.1, SW6.1
Other:
- moved on the sheet: C10, C11, C16, C17, C42, Q14, R12, R13, R2, R29, R3, R33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

Commit message: Added extra row of ground pins for 40 pin connector
Parts:
- added J19: Conn_01x20, Pin_Headers:Pin_Header_Straight_1x20_Pitch2.54mm, symbol Conn_01x20
- C15: value NC -> 10 uF
- C53: value 100 uF -> 1000 uF; footprint Capacitors_THT:CP_Radial_D5.0mm_P2.50mm -> Capacitors_THT:CP_Radial_D8.0mm_P3.50mm
Connections:
- net GND: now also C15.2, J19.1 (Pin_1), J19.10 (Pin_10), J19.11 (Pin_11), J19.12 (Pin_12), J19.13 (Pin_13), J19.14 (Pin_14), J19.15 (Pin_15), J19.16 (Pin_16), J19.17 (Pin_17), J19.18 (Pin_18), J19.19 (Pin_19), J19.2 (Pin_2), J19.20 (Pin_20), J19.3 (Pin_3), J19.4 (Pin_4), J19.5 (Pin_5), J19.6 (Pin_6), J19.7 (Pin_7), J19.8 (Pin_8), J19.9 (Pin_9)
- net at U3.1: no longer C15.1
- net at U3.7: now also C15.1
- net at U3.8: no longer C15.2
