File: RFBitBanger/RFBitBangerRadio.sch (KiCad schematic (older format))
At the start: 137 parts, among them J12 Conn_Coaxial, Q1 2N3904, Q10 2N3904, Q11 2N3904, Q12 2N3904, Q13 2N2907, Q2 2N3904, Q3 2N2222, Q5 2N2222, Q6 2N2222, Q7 2N2222, Q8 2N2907, Q9 2N3904, T1 Trifilar, T2 Trifilar, T3 Current, U4 LM358, U6 SI5351A, Y2 7.023 MHz, Y3 27 MHz, Y4 7.023 MHz

Commit message: A few minor tweaks to layout
Parts:
- added C32: 100 pF, Capacitors_THT:C_Disc_D5.0mm_W2.5mm_P5.00mm, symbol C_Small
- added D19: LED, LEDs:LED_D3.0mm, symbol LED
- added R71: 1k, Resistors_THT:R_Axial_DIN0207_L6.3mm_D2.5mm_P7.62mm_Horizontal, symbol R
- R57: value 4k7 -> 3k3
Connections:
- net +12V: now also D19.2 (A)
- net AMPOUT: now also C32.1
- net GND: now also C32.2
- net XOSC: now also JP5.3; no longer C21.1, C22.1, Q2.1 (E), R17.2
- net at R68.2: now also C21.1, C22.1, Q2.1 (E), R17.2; no longer JP5.3
- net at D18.1 (K), Q12.3 (C), R38.1: now also R71.1
- new net: D19.1 (K), R71.2
Other:
- moved on the sheet: C20, C24, L9, R65, R68

Commit message: Before changing back to HPF
Parts:
- added C38: 100 nF, Capacitors_THT:C_Disc_D5.0mm_W2.5mm_P2.50mm, symbol C_Small
- added L11: 100 uH, Inductors_THT:L_Axial_L6.6mm_D2.7mm_P10.16mm_Horizontal_Vishay_IM-2, symbol L
- added R73: 1k, Resistors_THT:R_Axial_DIN0207_L6.3mm_D2.5mm_P7.62mm_Horizontal, symbol R
- added R74: 0R, Resistors_THT:R_Axial_DIN0207_L6.3mm_D2.5mm_P7.62mm_Horizontal, symbol R
- added RV4: 2k, Potentiometers:Potentiometer_Trimmer_Bourns_3296W, symbol POT
- C23: value 100 nF -> 10 nF
- R53: value 2k2 -> NC
- R67: value 10k -> NC
Connections:
- net +5V: now also RV4.1
- net AMPOUT: now also R74.2; no longer L6.2, Q3.3 (C), Q7.3 (C)
- net GND: now also C38.2, RV4.3
- net at C23.2, D17.1 (K), Q3.2 (B)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: now also R73.2
- new net: L6.2, Q3.3 (C), Q7.3 (C), R74.1
- new net: L11.2, RV4.2
- new net: C38.1, L11.1, R73.1
Other:
- moved on the sheet: L6, Q12, Q5, Q7, R43, R45, R53, R65

Commit message: Added common mode choke, put back LPF
Parts:
- removed L10: 1 uH, Inductors_THT:L_Axial_L6.6mm_D2.7mm_P10.16mm_Horizontal_Vishay_IM-2, symbol L
- C28, C31: value 470 pF -> 220 pF
- C29: value 100 pF -> 680 pF
- L7: value 4.7 uH -> 1.35 uH
- L8: value 1 uH -> 1.35 uH
Connections:
- net GND: now also JP6.2; no longer JP6.1
- net at C28.1, C31.1: now also C29.1, JP6.1; no longer JP6.2, L8.1
- net at C31.2, JP2.2, JP4.2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: no longer C29.1
- net at C29.2, L7.2: now also L8.1
Other:
- note added: "FOR 80 M:\nL7,L8=2.6 uH\nC28,C31=390 pF\nC29=1200 pF"
- note removed: "VALUES FOR 40 M BAND\nFOR 80 M BAND:\nL8,L10=1.2 uH, C28,C31=1500 pF\nL7=12 uH, C29=150 pF"
- moved on the sheet: C28, C31, D16, J12, JP2, L7, L8, R28, T3

Commit message: Made 3 crystals instead of 2
Parts:
- removed D4, D5: 1N4007, Diodes_THT:D_DO-41_SOD81_P7.62mm_Horizontal, symbol D
- added Y5: 7.X MHz, Crystals:Crystal_HC49-U_Vertical, symbol Crystal
- C27: footprint Capacitors_THT:C_Disc_D5.0mm_W2.5mm_P2.50mm -> Capacitors_THT:C_Disc_D5.0mm_W2.5mm_P5.00mm
- Y2, Y4: value 7.023 MHz -> 7.X MHz
- renumbered D6 to D4, D7 to D5
Connections:
- net at C12.1, C13.1, L3.1: now also R9.1; no longer R9.2
- net at C21.2, Q2.2 (B), R15.2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: now also Y5.1
- net at C48.2, D4.1 (K), D5.1 (K): now also R9.2; no longer R9.1
- net at C48.1, Y2.2, Y4.2: now also Y5.2
Other:
- moved on the sheet: C12, C13, C46, C47, D10, D14, L3, R35, R48, R49, R50, R69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

Commit message: Added overvoltage zener and extra key inputs
Parts:
- added D6: D_Zener, Diodes_THT:D_DO-41_SOD81_P7.62mm_Horizontal, symbol D_Zener
- Q3, Q5, Q6, Q7: value 2N2222 -> 2N3904
Connections:
- net AMPOUT: now also D6.1 (K)
- net GND: now also D6.2 (A)

Commit message: Added README.md
Parts:
- removed R40: NC, Resistors_THT:R_Axial_DIN0207_L6.3mm_D2.5mm_P7.62mm_Horizontal, symbol R
- R41: footprint Resistors_THT:R_Axial_DIN0207_L6.3mm_D2.5mm_P7.62mm_Horizontal -> Resistors_THT:R_Axial_DIN0309_L9.0mm_D3.2mm_P12.70mm_Horizontal

Commit message: Lots of changes...
Parts:
- removed C53: 100 uH, Capacitors_THT:CP_Radial_D5.0mm_P2.50mm, symbol CP_Small
- removed Q3, Q5, Q6, Q7, Q9: 2N3904, TO_SOT_Packages_THT:TO-92_Inline_Wide, symbol 2N3904
- added Q3, Q6, Q7, Q9: 2N7000, TO_SOT_Packages_THT:TO-92_Inline_Wide, symbol 2N7000
- added Q5: NC, TO_SOT_Packages_THT:TO-92_Inline_Wide, symbol 2N7000
- C39: value 10 uH -> 2.2 uH
- C49: value 220 uF -> 100 uF
- L4, L7, L8: footprint Inductors_THT:L_Axial_L6.6mm_D2.7mm_P10.16mm_Horizontal_Vishay_IM-2 -> RFBitBanger:SmallVerticalToroid
- L6: value 220 uH -> 22 uH; footprint Inductors_THT:L_Axial_L6.6mm_D2.7mm_P10.16mm_Horizontal_Vishay_IM-2 -> RFBitBanger:SmallVerticalToroid
- R19: value 1k -> 470R
- R20: value 1k -> 330R
- R51: value 22R -> 0R
- R54: value 10k -> 1k
- R55: value 10k -> 100k
- R62: value 100k -> 10k
- R66: value NC -> 22k
- R68: value 4k7 -> 1k
- RV2: value 50k -> 10k
Connections:
- net AMPOUT: now also Q5.3 (D), Q6.3 (D)
- net at C20.2, C24.2, L6.1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: now also Q9.3 (D)
- net at C23.2, D17.1 (K), R53.1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: now also Q3.2 (G), Q5.2 (G), Q6.2 (G), Q7.2 (G)
- net at R42.1: now also Q3.1 (S)
- net at L6.2, R74.1: now also Q3.3 (D), Q7.3 (D)
- net at C40.1, C45.1, R18.2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: now also R63.2
- net at R43.1: now also Q5.1 (S)
- net at R44.1: now also Q6.1 (S)
- net at R45.1: now also Q7.1 (S)
- net at R41.2, R51.1: now also Q9.1 (S)
- net at R20.1, R52.2, R66.1: now also Q9.2 (G)
Other:
- moved on the sheet: R63

Commit message: Implemented timers, fixed beep audio, fixed key shaping
Parts:
- removed R10: 1k, Resistors_THT:R_Axial_DIN0207_L6.3mm_D2.5mm_P7.62mm_Horizontal, symbol R
- added J17: Filt1, Pin_Headers:Pin_Header_Straight_1x02_Pitch2.54mm, symbol Conn_01x02
- added J18: Filt2, Pin_Headers:Pin_Header_Straight_1x02_Pitch2.54mm, symbol Conn_01x02
- C14: value 10 uF -> 2.2 uF
Connections:
- net GND: now also J17.1 (Pin_1), J18.1 (Pin_1)
- net at C36.1, C46.2, C55.2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: now also R8.2; no longer C14.1
- net at C20.2, C24.2, L6.1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: now also C14.2
- net at C26.2, C28.2, JP4.1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: now also J17.2 (Pin_2)
- net at R8.1: now also C14.1, Q8.2 (B), R14.1; no longer D18.2 (A)
- net at C31.2, JP2.2, JP4.2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: now also J18.2 (Pin_2)
- new net: D18.2 (A), R14.2
Other:
- moved on the sheet: C14, C20, C24, D18, D19, R14, R71, R8
