File: RFBitBanger/RFBitBangerRadio.sch (KiCad schematic (older format))
At the start: 143 parts, among them J12 Conn_Coaxial, J17 Filt1, J18 Filt2, Q1 2N3904, Q10 2N3904, Q11 2N3904, Q12 2N3904, Q13 2N2907, Q2 2N3904, Q3 2N7000, Q5 NC, Q6 2N7000, Q7 2N7000, Q8 2N2907, Q9 2N7000, T1 Trifilar, T2 Trifilar, T3 Current, U4 LM358, U6 SI5351A, Y2 7.X MHz, Y3 27 MHz, Y4 7.X MHz, Y5 7.X MHz

Commit message: Rearranged parts for better layout
Parts:
- added Q15: NC, TO_SOT_Packages_THT:TO-220-3_Vertical, symbol IRF540N
- C32: value 100 pF -> 33 pF
- R14: value 1k -> 470R
- T1, T2: footprint RFBitBanger:TripleWindingTransformer -> RFBitBanger:TripleWindingTransformerRef
Connections:
- net AMPOUT: now also L6.2, Q3.3 (D), Q7.3 (D), R74.1, Q15.2 (D)
- net GND: now also T2.2, Q15.3 (S); no longer T2.1
- net at C23.2, D17.1 (K), Q3.2 (G)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: now also Q15.1 (G)
- net at R25.2: now also T2.1; no longer T2.2
- net at D11.1 (K), D13.2 (A): now also T2.6; no longer T2.3
- net at D12.1 (K), D9.2 (A): now also T2.3; no longer T2.6
Other:
- moved on the sheet: C32, D6, Q5, Q6, Q7, R43, R44, R45, R74

Commit message: Changed DSP to higher audible frequencies
Parts:
- C33: value 100 nF -> 10 nF
- C35: value 1 nF -> 330 pF
- C45: value 100 nF -> 330 nF; footprint Capacitors_THT:C_Disc_D5.0mm_W2.5mm_P2.50mm -> Capacitors_THT:C_Disc_D5.0mm_W2.5mm_P5.00mm
- R24: value 4k7 -> 10k
Connections:
- net AUDIO: now also C35.2, R23.1, R24.2, R36.2, U4.7; no longer C39.2, R37.2, RV2.3, U4.1
- new net: C39.2, R37.2, RV2.3, U4.1
Other:
- moved on the sheet: C25, R18, R19
Changed lines of the file:
@@
 $EndComp
 $Comp
-L +5V #PWR75
+L +5V #PWR76
 U 1 1 615A5B5E
-P 5950 5750
-F 0 "#PWR75" H 5950 5600 50  0001 C CNN
-F 1 "+5V" H 5950 5890 50  0000 C CNN
-F 2 "" H 5950 5750 50  0001 C CNN
-F 3 "" H 5950 5750 50  0001 C CNN
-	1    5950 5750
+P 6150 5750
+F 0 "#PWR76" H 6150 5600 50  0001 C CNN
+F 1 "+5V" H 6150 5890 50  0000 C CNN
+F 2 "" H 6150 5750 50  0001 C CNN
+F 3 "" H 6150 5750 50  0001 C CNN
+	1    6150 5750
 	1    0    0    -1
 $EndComp
@@
 L R R18
 U 1 1 615A93FE
-P 5950 5950
-F 0 "R18" V 6030 5950 50  0000 C CNN
-F 1 "1k" V 5950 5950 50  0000 C CNN
-F 2 "Resistors_THT:R_Axial_DIN0207_L6.3mm_D2.5mm_P7.62mm_Horizontal" V 5880 5950 50  0001 C CNN
-F 3 "" H 5950 5950 50  0001 C CNN
-	1    5950 5950
+P 6150 5950
+F 0 "R18" V 6230 5950 50  0000 C CNN
+F 1 "1k" V 6150 5950 50  0000 C CNN
+F 2 "Resistors_THT:R_Axial_DIN0207_L6.3mm_D2.5mm_P7.62mm_Horizontal" V 6080 5950 50  0001 C CNN
+F 3 "" H 6150 5950 50  0001 C CNN
+	1    6150 5950
 	1    0    0    -1
 $EndComp
@@
 P 6150 6750
 F 0 "R24" V 6230 6750 50  0000 C CNN
-F 1 "4k7" V 6150 6750 50  0000 C CNN
+F 1 "10k" V 6150 6750 50  0000 C CNN
 F 2 "Resistors_THT:R_Axial_DIN0207_L6.3mm_D2.5mm_P7.62mm_Horizontal" V 6080 6750 50  0001 C CNN
 F 3 "" H 6150 6750 50  0001 C CNN
@@
 $EndComp
 $Comp
-L GND #PWR73
+L GND #PWR72
 U 1 1 615AC48C
 P 5350 6850
-F 0 "#PWR73" H 5350 6600 50  0001 C CNN
+F 0 "#PWR72" H 5350 6600 50  0001 C CNN
 F 1 "GND" H 5350 6700 50  0000 C CNN
 F 2 "" H 5350 6850 50  0001 C CNN
@@
 P 6300 7000
 F 0 "C33" H 6100 7050 50  0000 L CNN
-F 1 "100 nF" H 6000 6900 50  0000 L CNN
+F 1 "10 nF" H 6000 6900 50  0000 L CNN
 F 2 "Capacitors_THT:C_Disc_D5.0mm_W2.5mm_P2.50mm" H 6300 7000 50  0001 C CNN
 F 3 "" H 6300 7000 50  0001 C CNN
@@
 	1    0    0    -1
 $EndComp
-Text GLabel 3900 6750 1    60   Input ~ 0
+Text GLabel 5950 6600 1    60   Input ~ 0
 AUDIO
 Text Notes 1150 1150 0    60   ~ 0
@@
 L R R19
 U 1 1 615C06F9
-P 5950 6350
-F 0 "R19" V 6030 6350 50  0000 C CNN
-F 1 "470R" V 5950 6350 50  0000 C CNN
-F 2 "Resistors_THT:R_Axial_DIN0207_L6.3mm_D2.5mm_P7.62mm_Horizontal" V 5880 6350 50  0001 C CNN
-F 3 "" H 5950 6350 50  0001 C CNN
-	1    5950 6350
-	1    0    0    -1
-$EndComp
-$Comp
-L GND #PWR76
+P 6150 6350
+F 0 "R19" V 6230 6350 50  0000 C CNN
+F 1 "470R" V 6150 6350 50  0000 C CNN
+F 2 "Resistors_THT:R_Axial_DIN0207_L6.3mm_D2.5mm_P7.62mm_Horizontal" V 6080 6350 50  0001 C CNN
+F 3 "" H 6150 6350 50  0001 C CNN
+	1    6150 6350
+	1    0    0    -1
+$EndComp
+$Comp
+L GND #PWR77
 U 1 1 615C0992
-P 5950 6500
-F 0 "#PWR76" H 5950 6250 50  0001 C CNN
-F 1 "GND" H 5950 6350 50  0000 C CNN
-F 2 "" H 5950 6500 50  0001 C CNN
-F 3 "" H 5950 6500 50  0001 C CNN
-	1    5950 6500
+P 6150 6500
+F 0 "#PWR77" H 6150 6250 50  0001 C CNN
+F 1 "GND" H 6150 6350 50  0000 C CNN
+F 2 "" H 6150 6500 50  0001 C CNN
+F 3 "" H 6150 6500 50  0001 C CNN
+	1    6150 6500
 	1    0    0    -1
 $EndComp
@@
 P 5450 7200
 F 0 "C35" V 5550 7150 50  0000 L CNN
-F 1 "1 nF" V 5350 7100 50  0000 L CNN
+F 1 "330 pF" V 5350 7100 50  0000 L CNN
 F 2 "Capacitors_THT:C_Disc_D5.0mm_W2.5mm_P5.00mm" H 5450 7200 50  0001 C CNN
 F 3 "" H 5450 7200 50  0001 C CNN
@@
 $EndComp
 $Comp
-L GND #PWR77
+L GND #PWR75
 U 1 1 6160C0A3
 P 5950 7200
-F 0 "#PWR77" H 5950 6950 50  0001 C CNN
+F 0 "#PWR75" H 5950 6950 50  0001 C CNN
 F 1 "GND" H 5950 7050 50  0000 C CNN
 F 2 "" H 5950 7200 50  0001 C CNN
@@
 P 4650 6500
 F 0 "C45" H 4750 6600 50  0000 L CNN
-F 1 "100 nF" H 4750 6500 50  0000 L CNN
-F 2 "Capacitors_THT:C_Disc_D5.0mm_W2.5mm_P2.50mm" H 4650 6500 50  0001 C CNN
+F 1 "330 nF" H 4750 6500 50  0000 L CNN
+F 2 "Capacitors_THT:C_Disc_D5.0mm_W2.5mm_P5.00mm" H 4650 6500 50  0001 C CNN
 F 3 "" H 4650 6500 50  0001 C CNN
 	1    4650 6500
@@
 L C_Small C25
 U 1 1 61679E36
-P 5000 5850
-F 0 "C25" H 5100 5850 50  0000 L CNN
-F 1 "100 nF" V 4850 5750 50  0000 L CNN
-F 2 "Capacitors_THT:C_Disc_D5.0mm_W2.5mm_P2.50mm" H 5000 5850 50  0001 C CNN
-F 3 "" H 5000 5850 50  0001 C CNN
-	1    5000 5850
-	1    0    0    -1
-$EndComp
-$Comp
-L GND #PWR71
+P 5750 5900
+F 0 "C25" H 5850 5900 50  0000 L CNN
+F 1 "100 nF" V 5600 5750 50  0000 L CNN
+F 2 "Capacitors_THT:C_Disc_D5.0mm_W2.5mm_P2.50mm" H 5750 5900 50  0001 C CNN
+F 3 "" H 5750 5900 50  0001 C CNN
+	1    5750 5900
+	1    0    0    -1
+$EndComp
+$Comp
+L GND #PWR74
 U 1 1 6167A2A0
-P 5000 5950
-F 0 "#PWR71" H 5000 5700 50  0001 C CNN
-F 1 "GND" H 5000 5800 50  0000 C CNN
-F 2 "" H 5000 5950 50  0001 C CNN
-F 3 "" H 5000 5950 50  0001 C CNN
-	1    5000 5950
+P 5750 6000
+F 0 "#PWR74" H 5750 5750 50  0001 C CNN
+F 1 "GND" H 5850 6000 50  0000 C CNN
+F 2 "" H 5750 6000 50  0001 C CNN
+F 3 "" H 5750 6000 50  0001 C CNN
+	1    5750 6000
 	1    0    0    -1
 $EndComp
@@
 $EndComp
 $Comp
-L GND #PWR72
+L GND #PWR71
 U 1 1 61848EB7
 P 5300 4700
-F 0 "#PWR72" H 5300 4450 50  0001 C CNN
+F 0 "#PWR71" H 5300 4450 50  0001 C CNN
 F 1 "GND" H 5300 4550 50  0000 C CNN
 F 2 "" H 5300 4700 50  0001 C CNN
@@
 U 1 1 618BE9DA
 P 6400 6350
-F 0 "C40" V 6200 6300 50  0000 L CNN
+F 0 "C40" V 6450 6400 50  0000 L CNN
 F 1 "100 uF" V 6300 6250 50  0000 L CNN
 F 2 "Capacitors_THT:CP_Radial_D5.0mm_P2.50mm" H 6400 6350 50  0001 C CNN
@@
 $EndComp
 $Comp
-L GND #PWR74
+L GND #PWR73
 U 1 1 61B09AF1
 P 5650 2200
-F 0 "#PWR74" H 5650 1950 50  0001 C CNN
+F 0 "#PWR73" H 5650 1950 50  0001 C CNN
 F 1 "GND" H 5650 2050 50  0000 C CNN
 F 2 "" H 5650 2200 50  0001 C CNN
@@
 	8450 3300 8450 3200
 Wire Wire Line
-	5950 6100 5950 6200
-Connection ~ 5950 6150
-Wire Wire Line
 	5750 6750 6000 6750
 Connection ~ 5750 6750
 Wire Wire Line
-	5950 5750 5950 5800
-Wire Wire Line
 	6400 6150 6400 6250
 Wire Wire Line
@@
 Connection ~ 5100 6650
 Wire Wire Line
-	5000 5750 5950 5750
-Connection ~ 5350 5750
-Wire Wire Line
-	5000 5950 5000 5950
-Wire Wire Line
-	5950 6750 5950 6800
+	5350 5750 6150 5750
+Wire Wire Line
+	5950 6600 5950 6800
 Wire Wire Line
 	5750 7200 5550 7200
@@
 	5450 1600 5650 1600
 Wire Wire Line
-	3900 6750 3900 7400
+	3900 6900 3900 7400
 Wire Wire Line
 	3350 7400 3350 7250
@@
 Wire Wire Line
 	10050 2200 10100 2200
+Wire Wire Line
+	6150 6100 6150 6200
+Connection ~ 6150 6150
+Wire Wire Line
+	6150 5750 6150 5800
+Wire Wire Line
+	5750 5800 5750 5750
+Connection ~ 5750 5750
 $EndSCHEMATC
