File: RFBitBanger/RFBitBangerRadio.sch (KiCad schematic (older format))
At the start: 145 parts, among them J12 Conn_Coaxial, J17 Filt1, J18 Filt2, Q1 2N3904, Q10 2N3904, Q11 2N3904, Q12 2N3904, Q13 2N2907, Q15 NC, Q2 2N3904, Q3 2N7000, Q5 NC, Q6 2N7000, Q7 2N7000, Q8 2N2907, Q9 2N7000, T1 Trifilar, T2 Trifilar, T3 Current, U4 LM358, U6 SI5351A, Y2 7.X MHz, Y3 27 MHz, Y4 7.X MHz, Y5 7.X MHz

Commit message: JLCPCB order 2022-01-24
Parts:
- C48: footprint Capacitors_THT:C_Disc_D5.0mm_W2.5mm_P2.50mm -> Capacitors_THT:C_Disc_D5.0mm_W2.5mm_P5.00mm
- D8: value 1N4148 -> 1N4001; footprint Diodes_THT:D_DO-35_SOD27_P7.62mm_Horizontal -> Diodes_THT:D_DO-41_SOD81_P7.62mm_Horizontal
Changed lines of the file:
@@
 P 10600 1700
 F 0 "D8" H 10600 1800 50  0000 C CNN
-F 1 "1N4148" H 10600 1600 50  0000 C CNN
-F 2 "Diodes_THT:D_DO-35_SOD27_P7.62mm_Horizontal" H 10600 1700 50  0001 C CNN
+F 1 "1N4001" H 10600 1600 50  0000 C CNN
+F 2 "Diodes_THT:D_DO-41_SOD81_P7.62mm_Horizontal" H 10600 1700 50  0001 C CNN
 F 3 "" H 10600 1700 50  0001 C CNN
 	1    10600 1700
@@
 F 0 "C48" V 1900 2150 50  0000 L CNN
 F 1 "100 nF" V 2150 2050 50  0000 L CNN
-F 2 "Capacitors_THT:C_Disc_D5.0mm_W2.5mm_P2.50mm" H 2050 2200 50  0001 C CNN
+F 2 "Capacitors_THT:C_Disc_D5.0mm_W2.5mm_P5.00mm" H 2050 2200 50  0001 C CNN
 F 3 "" H 2050 2200 50  0001 C CNN
 	1    2050 2200

Commit message: Before changing si5351 code
Parts:
- C39: value 2.2 uH -> 1 uH
- C49: value 100 uF -> 22 uF
- C50: value 100 uF -> 10 uF
Changed lines of the file:
@@
 P 4150 6900
 F 0 "C39" V 4000 6850 50  0000 L CNN
-F 1 "2.2 uH" V 4250 6800 50  0000 L CNN
+F 1 "1 uH" V 4250 6800 50  0000 L CNN
 F 2 "Capacitors_THT:CP_Radial_D5.0mm_P2.50mm" H 4150 6900 50  0001 C CNN
 F 3 "" H 4150 6900 50  0001 C CNN
@@
 P 1350 6850
 F 0 "C49" V 1450 6800 50  0000 L CNN
-F 1 "100 uF" V 1250 6750 50  0000 L CNN
+F 1 "22 uF" V 1250 6750 50  0000 L CNN
 F 2 "Capacitors_THT:CP_Radial_D5.0mm_P2.50mm" H 1350 6850 50  0001 C CNN
 F 3 "" H 1350 6850 50  0001 C CNN
@@
 P 1700 7300
 F 0 "C50" V 1900 7250 50  0000 L CNN
-F 1 "100 uF" V 1800 7200 50  0000 L CNN
+F 1 "10 uF" V 1800 7200 50  0000 L CNN
 F 2 "Capacitors_THT:CP_Radial_D5.0mm_P2.50mm" H 1700 7300 50  0001 C CNN
 F 3 "" H 1700 7300 50  0001 C CNN

Commit message: Before adding SI5351 header
Parts:
- C39: value 1 uH -> 1 uF
Changed lines of the file:
@@
 P 4150 6900
 F 0 "C39" V 4000 6850 50  0000 L CNN
-F 1 "1 uH" V 4250 6800 50  0000 L CNN
+F 1 "1 uF" V 4250 6800 50  0000 L CNN
 F 2 "Capacitors_THT:CP_Radial_D5.0mm_P2.50mm" H 4150 6900 50  0001 C CNN
 F 3 "" H 4150 6900 50  0001 C CNN

Commit message: Added connector for SI5351A board
Parts:
- added J10: si5351mod, Pin_Headers:Pin_Header_Straight_1x07_Pitch2.54mm, symbol Conn_01x07
Connections:
- net +5V: now also J10.7 (Pin_7)
- net GND: now also J10.6 (Pin_6)
- net SCL: now also J10.4 (Pin_4)
- net SDA: now also J10.5 (Pin_5)
- net at R49.1, U6.10 (CLK0): now also J10.1 (Pin_1)
- net at R50.1, U6.9 (CLK1): now also J10.2 (Pin_2)

Commit message: Changed around for external filter PCB
Parts:
- removed C28, C31: 220 pF, Capacitors_THT:C_Disc_D5.0mm_W2.5mm_P5.00mm, symbol C_Small
- removed C29: 680 pF, Capacitors_THT:C_Disc_D5.0mm_W2.5mm_P5.00mm, symbol C_Small
- removed J17: Filt1, Pin_Headers:Pin_Header_Straight_1x02_Pitch2.54mm, symbol Conn_01x02
- removed J18: Filt2, Pin_Headers:Pin_Header_Straight_1x02_Pitch2.54mm, symbol Conn_01x02
- removed JP6: BYPASS, Pin_Headers:Pin_Header_Straight_1x02_Pitch2.54mm, symbol Jumper_NC_Small
- removed L7, L8: 1.35 uH, RFBitBanger:SmallVerticalToroid, symbol L
- removed R42, R43, R44, R45: 1R0, Resistors_THT:R_Axial_DIN0207_L6.3mm_D2.5mm_P7.62mm_Horizontal, symbol R
- removed R69: 330R, Resistors_THT:R_Axial_DIN0207_L6.3mm_D2.5mm_P7.62mm_Horizontal, symbol R
- added J17: Filt1, Pin_Headers:Pin_Header_Straight_1x04_Pitch2.54mm, symbol Conn_01x04
- added J18: Filt2, Pin_Headers:Pin_Header_Straight_1x04_Pitch2.54mm, symbol Conn_01x04
- C23, C26: footprint Capacitors_THT:C_Disc_D5.0mm_W2.5mm_P2.50mm -> Capacitors_THT:C_Disc_D5.0mm_W2.5mm_P5.00mm
- Q13, Q8: value 2N2907 -> SS8050
- R20: value 330R -> 100R
- R28: value 1k -> 47R
- R41: value 220R -> 150R
- R52: value 10k -> 47k
- R66: value 22k -> 470k
Connections:
- net GND: now also Q3.1 (S), Q5.1 (S), Q6.1 (S), Q7.1 (S), R28.2, J17.1 (Pin_1), J17.2 (Pin_2), J18.1 (Pin_1), J18.2 (Pin_2); no longer R28.1
- net PLLOSC: now also R49.2, R50.2
- net at C26.2, JP4.1: now also J17.3 (Pin_3), J17.4 (Pin_4)
- net at JP2.2, JP4.2, JP7.3: now also T3.1 (RF), J18.3 (Pin_3), J18.4 (Pin_4); no longer T3.2 (RF)
- net at J12.1 (In), JP2.1: now also T3.2 (RF); no longer T3.1 (RF)
- net at D16.1 (K): now also R28.1; no longer R28.2
Other:
- note removed: "FOR 80 M:\nL7,L8=2.6 uH\nC28,C31=390 pF\nC29=1200 pF"
- note removed: "OUTPUT FILTER"
- moved on the sheet: D16, JP4, R28
