File: RFBitBanger/RFBitBanger.kicad_pcb (KiCad board)
At the start: 2 copper layers, 149 x 88 mm, 223 parts, among them J1 POWER, J10 Conn_01x05, J11 SPEAKER, J12 Conn_Coaxial, J13 Conn_01x01, J2 Barrel_Jack, J3 Conn_01x01, J4 Conn_01x01, J5 Conn_01x04, J6 Conn_01x01, J7 Conn_01x01, J8 Conn_01x01, J9 ICSP, P1 Mini-DIN_6pins_ver4, Q1 2N3904, Q10 2N3904, Q11 2N3904, Q12 2N3904, Q13 2N2907, Q14 2N3904, Q2 2N3904, Q3 2N3904, Q4 2N3904, Q5 2N3904, Q6 2N3904, Q7 2N3904, Q8 2N2907, Q9 2N3904, SW1 SW_Push, SW2 SW_Push, SW3 SW_Push, SW4 SW_Push, SW5 SW_Push, T1 Trifilar, T2 Trifilar, T3 Current, T4 Common-Mode Choke, U1 ATMEGA328-PU, U2 LM7805_TO220, U3 LM386, U4 LM358, U5 LCD-016N002L, U6 SI5351A, Y1 16 MHz, Y2 7.X MHz, Y3 27 MHz, Y4 7.X MHz, Y5 7.X MHz

Commit message: Fixed overcommited MOSI pin
Parts:
- removed R75: 10k, Resistors_THT:R_Axial_DIN0207_L6.3mm_D2.5mm_P7.62mm_Horizontal
- J10: value Conn_01x05 -> Conn_01x04; footprint Pin_Headers:Pin_Header_Straight_1x05_Pitch2.54mm -> Pin_Headers:Pin_Header_Straight_1x04_Pitch2.54mm
- R76: value 10k -> 1k
- moved C1 3.97 mm to (89.4, 96.9), turned to 270 degrees
Connections:
- J10 pad 2: Net-(J10-Pad2) -> +5V
- J10 pad 3: +5V -> Net-(C7-Pad2)
- J10 pad 4: Net-(C7-Pad2) -> GND
- R76 pad 1: Net-(J10-Pad2) -> Net-(J10-Pad1)
Routing:
- net Net-(J10-Pad2): track 7.92 -> 0.00 mm
- net MOSI: track 72.8 -> 65.2 mm
- net +5V: track 357.4 -> 352.6 mm, vias 1 -> 0
- net Net-(C7-Pad2): track 8.00 -> 9.97 mm
- net Net-(J10-Pad1): track 4.84 -> 4.09 mm
Other:
- board text removed: "KY2"

Commit message: Added README.md
Parts:
- removed R40: NC, Resistors_THT:R_Axial_DIN0207_L6.3mm_D2.5mm_P7.62mm_Horizontal
- R41: footprint Resistors_THT:R_Axial_DIN0207_L6.3mm_D2.5mm_P7.62mm_Horizontal -> Resistors_THT:R_Axial_DIN0309_L9.0mm_D3.2mm_P12.70mm_Horizontal
- moved R41 18.5 mm to (177.7, 102.1), turned to 180 degrees
- moved R51 1.32 mm to (165.8, 92.4)
- moved C20 1.27 mm to (162.2, 89.6)
- moved Q9 1.21 mm to (166.9, 95.9)
- moved D6 0.82 mm to (177.2, 98.2)
- moved C23 0.77 mm to (163.2, 82.0)
- moved C32 0.55 mm to (169.2, 87.2)
- moved R74 0.51 mm to (169.2, 77.3)
- moved R44 0.44 mm to (177.2, 94.8)
Routing:
- net RF: track 13.4 -> 10.6 mm
- net Net-(Q9-Pad1): track 9.27 -> 11.1 mm
- net Net-(C23-Pad1): track 5.53 -> 3.84 mm
- net Net-(C20-Pad2): track 51.4 -> 52.7 mm
- net Net-(Q9-Pad2): track 24.6 -> 25.9 mm
- net Net-(C23-Pad2): track 83.9 -> 83.4 mm

Commit message: Lots of changes...
Parts:
- removed C57: 10 nF, Capacitors_THT:C_Disc_D5.0mm_W2.5mm_P2.50mm
- added J14: Conn_01x01, Pin_Headers:Pin_Header_Straight_1x01_Pitch2.54mm, F.Cu at (97.7, 119.6)
- added J15: Conn_01x01, Pin_Headers:Pin_Header_Straight_1x01_Pitch2.54mm, F.Cu at (164.2, 136.4)
- added J16: Conn_01x01, Pin_Headers:Pin_Header_Straight_1x01_Pitch2.54mm, F.Cu at (179.9, 58.9)
- added L10: 100 uH, Inductors_THT:L_Axial_L6.6mm_D2.7mm_P10.16mm_Horizontal_Vishay_IM-2, F.Cu at (72.6, 126.4)
- C18: value 100 nF -> 1 uF; footprint Capacitors_THT:C_Disc_D5.0mm_W2.5mm_P2.50mm -> Capacitors_THT:CP_Radial_D5.0mm_P2.50mm
- C3: value 100 uF -> 1000 uF; footprint Capacitors_THT:CP_Radial_D5.0mm_P2.50mm -> Capacitors_THT:CP_Radial_D8.0mm_P3.50mm
- C39: value 10 uH -> 2.2 uH
- C41: value 10 nF -> 100 nF
- C49: value 220 uF -> 100 uF
- C53: value 100 uH -> 100 uF
- C7: value 10 nF -> 1 nF; footprint Capacitors_THT:C_Disc_D5.0mm_W2.5mm_P2.50mm -> Capacitors_THT:C_Disc_D5.0mm_W2.5mm_P5.00mm
- L4, L7, L8: footprint Inductors_THT:L_Axial_L6.6mm_D2.7mm_P10.16mm_Horizontal_Vishay_IM-2 -> RFBitBanger:SmallVerticalToroid
- L6: value 220 uH -> 22 uH; footprint Inductors_THT:L_Axial_L6.6mm_D2.7mm_P10.16mm_Horizontal_Vishay_IM-2 -> RFBitBanger:SmallVerticalToroid
- Q3, Q6, Q7, Q9: value 2N3904 -> 2N7000
- Q5: value 2N3904 -> NC
- R11: value 10R -> 47R
- R19: value 1k -> 470R
- R20: value 1k -> 330R
- R30, R31, R62: value 100k -> 10k
- R32, R34, R54: value 10k -> 1k
- R51: value 22R -> 0R
- R55: value 10k -> 100k
- R66: value NC -> 22k
- R68: value 4k7 -> 1k
- RV2: value 50k -> 10k
- moved C53 59.2 mm to (55.9, 140.2), turned to 90 degrees
- moved R11 23.4 mm to (65.2, 129.8), turned to 0 degrees
- moved R37 18.4 mm to (112.1, 134.1), turned to 270 degrees
- moved C18 13.3 mm to (93.3, 126.0)
- moved C19 10.7 mm to (63.1, 137.6)
- moved R21 10.6 mm to (152.4, 130.5), turned to 90 degrees
- moved C41 9.90 mm to (70.6, 133.0), turned to 0 degrees
- moved R58 8.68 mm to (133.7, 141.8), turned to 90 degrees
- moved R60 7.95 mm to (136.9, 134.2)
- moved L7 7.53 mm to (177.3, 127.5)
- moved L8 7.35 mm to (162.6, 127.0)
- moved C49 7.21 mm to (147.8, 136.2)
- moved C52 7.05 mm to (135.3, 128.5)
- moved L4 7.02 mm to (103.4, 82.1), turned to 90 degrees
- moved C27 6.80 mm to (152.0, 120.1), turned to 0 degrees
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Connections:
- C18 pad 2: Net-(C18-Pad2) -> GND
- C19 pad 1: Net-(C18-Pad1) -> Net-(C19-Pad1)
- C41 pad 1: Net-(C19-Pad2) -> Net-(C19-Pad1)
- C53 pad 1: Net-(C53-Pad1) -> +12V
- Q4 pad 3: Net-(C57-Pad1) -> Net-(C18-Pad1)
- R11 pad 1: GND -> Net-(C19-Pad1)
- R11 pad 2: Net-(C18-Pad2) -> Net-(L10-Pad1)
- R32 pad 2: Net-(C57-Pad1) -> Net-(C18-Pad1)
- R34 pad 1: Net-(C57-Pad1) -> Net-(C18-Pad1)
- R63 pad 2: Net-(C53-Pad1) -> Net-(C40-Pad1)
- U3 pad 5: Net-(C18-Pad1) -> Net-(L10-Pad1)
Routing:
- net GND: track 75.6 -> 45.1 mm
- net +12V: track 235.2 -> 260.6 mm
- net Net-(C19-Pad1): track 0.00 -> 20.7 mm
- net +5V: track 352.6 -> 369.9 mm
- net Net-(C40-Pad1): track 27.2 -> 41.5 mm
- net Net-(L6-Pad2): track 42.6 -> 54.8 mm
- net Net-(L10-Pad1): track 0.00 -> 12.0 mm
- net Net-(C57-Pad1): track 10.9 -> 0.00 mm
- net Net-(C54-Pad1): track 12.6 -> 22.6 mm
- net Net-(C26-Pad2): track 26.3 -> 36.1 mm
- net AUDIOFILT: track 47.9 -> 57.2 mm
- net Net-(C53-Pad1): track 7.98 -> 0.00 mm
- net Net-(C18-Pad2): track 6.42 -> 0.00 mm
- net Net-(C23-Pad2): track 83.4 -> 89.6 mm
- net Net-(Q11-Pad1): track 11.5 -> 17.6 mm
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
Commit message: Implemented timers, fixed beep audio, fixed key shaping
Parts:
- removed R10: 1k, Resistors_THT:R_Axial_DIN0207_L6.3mm_D2.5mm_P7.62mm_Horizontal
- added J17: Filt1, Pin_Headers:Pin_Header_Straight_1x02_Pitch2.54mm, F.Cu at (161.3, 121.9)
- added J18: Filt2, Pin_Headers:Pin_Header_Straight_1x02_Pitch2.54mm, F.Cu at (161.3, 137.2)
- C14: value 10 uF -> 2.2 uF
- C15: value NC -> 10 uF
- R31: value 10k -> 220k
- moved D18 25.0 mm to (140.2, 62.5), turned to 0 degrees
- moved R14 19.0 mm to (158.0, 62.5), turned to 180 degrees
- moved Q8 14.2 mm to (143.5, 70.5), turned to 0 degrees
- moved C14 13.8 mm to (152.8, 66.5), turned to 0 degrees
- moved J8 10.9 mm to (153.0, 74.5)
- moved J15 9.75 mm to (156.2, 130.8)
- moved Q12 8.63 mm to (131.5, 67.3)
- moved C22 7.46 mm to (133.0, 76.5)
- moved C27 5.73 mm to (155.8, 124.4), turned to 90 degrees
- moved C24 4.56 mm to (157.8, 72.0), turned to 270 degrees
- moved R8 4.49 mm to (149.1, 66.2), turned to 180 degrees
- moved R67 4.24 mm to (148.4, 79.3)
- moved L8 2.94 mm to (163.3, 129.9)
- moved L7 2.76 mm to (176.6, 130.2)
- moved JP6 2.58 mm to (170.2, 119.9), turned to 90 degrees
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Connections:
- C20 pad 2: Net-(C20-Pad2) -> Net-(C14-Pad2)
- C24 pad 2: Net-(C20-Pad2) -> Net-(C14-Pad2)
- C36 pad 1: Net-(C14-Pad1) -> Net-(C36-Pad1)
- C46 pad 2: Net-(C14-Pad1) -> Net-(C36-Pad1)
- C55 pad 2: Net-(C14-Pad1) -> Net-(C36-Pad1)
- L4 pad 2: Net-(C14-Pad1) -> Net-(C36-Pad1)
- L6 pad 1: Net-(C20-Pad2) -> Net-(C14-Pad2)
- Q10 pad 3: Net-(C14-Pad1) -> Net-(C36-Pad1)
- Q13 pad 1: Net-(C14-Pad1) -> Net-(C36-Pad1)
- Q2 pad 3: Net-(C14-Pad1) -> Net-(C36-Pad1)
- Q8 pad 1: Net-(C14-Pad1) -> Net-(C36-Pad1)
- Q8 pad 2: Net-(Q8-Pad2) -> Net-(C14-Pad1)
- Q8 pad 3: Net-(C20-Pad2) -> Net-(C14-Pad2)
- Q9 pad 3: Net-(C20-Pad2) -> Net-(C14-Pad2)
- R14 pad 1: Net-(Q8-Pad2) -> Net-(C14-Pad1)
- R14 pad 2: Net-(C14-Pad2) -> Net-(D18-Pad2)
- R15 pad 1: Net-(C14-Pad1) -> Net-(C36-Pad1)
- R52 pad 1: Net-(C20-Pad2) -> Net-(C14-Pad2)
- R53 pad 2: Net-(C20-Pad2) -> Net-(C14-Pad2)
- R55 pad 1: Net-(C14-Pad1) -> Net-(C36-Pad1)
- R8 pad 1: Net-(D18-Pad2) -> Net-(C14-Pad1)
- R8 pad 2: Net-(C14-Pad2) -> Net-(C36-Pad1)
Routing:
- net Net-(C36-Pad1): track 0.00 -> 182.9 mm
- net Net-(C14-Pad1): track 161.6 -> 18.4 mm
- net Net-(C20-Pad2): track 54.9 -> 0.00 mm
- net Net-(C14-Pad2): track 13.2 -> 60.2 mm
- net Net-(Q8-Pad2): track 17.0 -> 0.00 mm
- net Net-(D18-Pad2): track 18.6 -> 2.62 mm
- net Net-(C31-Pad2): track 48.2 -> 57.7 mm
- net Net-(C26-Pad2): track 36.1 -> 43.9 mm
- net Net-(C23-Pad2): track 89.6 -> 86.7 mm
- net Net-(C28-Pad1): track 11.2 -> 13.1 mm
- net AUDIO: track 43.0 -> 41.4 mm
- net Net-(C27-Pad1): track 2.95 -> 4.59 mm
- net Net-(C21-Pad1): track 24.1 -> 25.6 mm
- net Net-(D18-Pad1): track 39.1 -> 40.4 mm
- net IF: track 30.5 -> 29.3 mm
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
Commit message: Rearranged parts for better layout
Parts:
- added C57: 100 nF, Capacitors_THT:C_Disc_D5.0mm_W2.5mm_P2.50mm, F.Cu at (89.5, 94.5)
- added J19: Conn_01x04, Pin_Headers:Pin_Header_Straight_1x04_Pitch2.54mm, F.Cu at (60.5, 84.8)
- added Q15: NC, TO_SOT_Packages_THT:TO-220-3_Vertical, F.Cu at (187.2, 82.3)
- C32: value 100 pF -> 33 pF
- R14: value 1k -> 470R
- T1, T2: footprint RFBitBanger:TripleWindingTransformer -> RFBitBanger:TripleWindingTransformerRef
- moved R61 13.8 mm to (128.5, 124.0), turned to 0 degrees
- moved R56 11.5 mm to (136.0, 115.5), turned to 180 degrees
- moved C30 9.64 mm to (140.1, 106.6)
- moved R59 8.88 mm to (130.1, 112.3), turned to 0 degrees
- moved R55 7.64 mm to (127.1, 104.1), turned to 270 degrees
- moved R5 7.48 mm to (140.5, 109.3), turned to 270 degrees
- moved D3 7.30 mm to (60.4, 97.7)
- moved R4 5.51 mm to (55.0, 99.5), turned to 90 degrees
- moved C55 2.89 mm to (133.1, 102.3), turned to 180 degrees
- moved RV3 2.78 mm to (51.2, 88.9), turned to 0 degrees
- moved C42 2.18 mm to (50.8, 77.1)
- moved Q7 2.07 mm to (180.2, 78.7)
- moved Q5 2.06 mm to (185.3, 90.8)
- moved C51 2.05 mm to (144.4, 88.2)
- moved Q6 2.02 mm to (175.6, 90.7)
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Connections:
- L6 pad 2: Net-(L6-Pad2) -> AMPOUT
- Q3 pad 3: Net-(L6-Pad2) -> AMPOUT
- Q7 pad 3: Net-(L6-Pad2) -> AMPOUT
- R74 pad 1: Net-(L6-Pad2) -> AMPOUT
- T2 pad 1: GND -> Net-(R25-Pad2)
- T2 pad 2: Net-(R25-Pad2) -> GND
- T2 pad 3: Net-(D11-Pad1) -> Net-(D12-Pad1)
- T2 pad 6: Net-(D12-Pad1) -> Net-(D11-Pad1)
- U1 pad 21: (no net) -> Net-(C57-Pad1)
Routing:
- net AMPOUT: track 41.2 -> 129.5 mm
- net GND: track 45.1 -> 108.9 mm
- net Net-(L6-Pad2): track 54.8 -> 0.00 mm
- net +5V: track 369.9 -> 406.5 mm
- net Net-(Q10-Pad2): track 20.1 -> 33.3 mm
- net Net-(RV3-Pad2): track 29.3 -> 20.2 mm
- net Net-(C52-Pad1): track 18.0 -> 9.98 mm
- net Net-(D12-Pad2): track 26.5 -> 19.1 mm
- net E: track 44.0 -> 49.4 mm
- net +12V: track 260.6 -> 265.7 mm
- net Net-(Q10-Pad1): track 18.3 -> 13.5 mm
- net Net-(C30-Pad2): track 17.5 -> 13.0 mm
- net Net-(C51-Pad1): track 12.4 -> 8.10 mm
- net IF: track 29.3 -> 33.2 mm
- net Net-(D12-Pad1): track 6.37 -> 10.2 mm
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Other:
- board text added: "FILT1"
- board text added: "FILT2"

Commit message: Changed DSP to higher audible frequencies
Parts:
- added C60: NC, Capacitors_THT:C_Disc_D5.0mm_W2.5mm_P5.00mm, F.Cu at (93.5, 133.3)
- added R10: 100k, Resistors_THT:R_Axial_DIN0207_L6.3mm_D2.5mm_P7.62mm_Horizontal, F.Cu at (78.9, 120.8)
- C15: value 10 uF -> NC
- C18: value 1 uF -> NC; footprint Capacitors_THT:CP_Radial_D5.0mm_P2.50mm -> Capacitors_THT:C_Disc_D5.0mm_W2.5mm_P5.00mm
- C33: value 100 nF -> 10 nF
- C35: value 1 nF -> 330 pF
- C45: value 100 nF -> 330 nF; footprint Capacitors_THT:C_Disc_D5.0mm_W2.5mm_P2.50mm -> Capacitors_THT:C_Disc_D5.0mm_W2.5mm_P5.00mm
- R24: value 4k7 -> 10k
- R31: value 220k -> 100k
- R32, R34: value 1k -> 100k
- moved C33 18.5 mm to (84.4, 114.2), turned to 180 degrees
- moved R31 15.4 mm to (90.2, 128.3), turned to 270 degrees
- moved R24 11.4 mm to (90.8, 116.0)
- moved J14 9.15 mm to (104.4, 113.4)
- moved R26 7.25 mm to (110.6, 124.2), turned to 180 degrees
- moved R34 7.20 mm to (96.7, 125.7)
- moved C18 6.67 mm to (99.1, 122.6), turned to 90 degrees
- moved Q4 6.60 mm to (94.7, 117.5), turned to 270 degrees
- moved R32 6.12 mm to (100.1, 133.3)
- moved C34 3.99 mm to (93.8, 136.1)
- moved R23 3.67 mm to (109.8, 127.1)
- moved C35 3.15 mm to (113.2, 125.7)
- moved C45 2.80 mm to (113.6, 117.4), turned to 270 degrees
- moved R30 2.42 mm to (86.5, 117.5)
- moved C39 2.30 mm to (106.4, 138.9), turned to 0 degrees
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Connections:
- C35 pad 2: Net-(C35-Pad2) -> AUDIO
- C39 pad 2: AUDIO -> Net-(C39-Pad2)
- R23 pad 1: Net-(C35-Pad2) -> AUDIO
- R24 pad 2: Net-(C35-Pad2) -> AUDIO
- R31 pad 1: BEEPOUT -> Net-(C60-Pad2)
- R36 pad 2: Net-(C35-Pad2) -> AUDIO
- R37 pad 2: AUDIO -> Net-(C39-Pad2)
- RV2 pad 3: AUDIO -> Net-(C39-Pad2)
- U4 pad 1: AUDIO -> Net-(C39-Pad2)
- U4 pad 7: Net-(C35-Pad2) -> AUDIO
Routing:
- net Net-(C35-Pad2): track 30.9 -> 0.00 mm
- net Net-(C39-Pad2): track 0.00 -> 30.1 mm
- net Net-(C34-Pad1): track 27.1 -> 8.19 mm
- net Net-(C60-Pad2): track 0.00 -> 13.1 mm
- net AUDIOFILT: track 57.2 -> 48.5 mm
- net Net-(C45-Pad2): track 32.8 -> 25.4 mm
- net AUDIO: track 42.0 -> 49.2 mm
- net Net-(C35-Pad1): track 14.2 -> 8.79 mm
- net TUNING: track 44.7 -> 40.1 mm
- net TRANSMIT: track 36.6 -> 32.4 mm
- net MUTEAUDIO: track 35.2 -> 31.6 mm
- net Net-(C18-Pad1): track 15.2 -> 11.8 mm
- net Net-(Q4-Pad2): track 7.03 -> 9.67 mm
- net Net-(C34-Pad2): track 8.10 -> 5.79 mm
- net BEEPOUT: track 36.2 -> 38.1 mm

Commit message: Added Display Board on Top
Parts:
- added J20: Conn_01x01, Connectors:1pin, F.Cu at (128.5, 60.5)
- added J21: Conn_01x01, Connectors:1pin, F.Cu at (128.5, 140.5)
- added J22: SPEAKER, Pin_Headers:Pin_Header_Straight_1x02_Pitch2.54mm, F.Cu at (65.5, 133.5)
- added JP8: Shutdown, Pin_Headers:Pin_Header_Straight_1x02_Pitch2.54mm, F.Cu at (133.7, 79.5)
- D15, D18, D8: value 1N4007 -> 1N4148; footprint Diodes_THT:D_DO-41_SOD81_P7.62mm_Horizontal -> Diodes_THT:D_DO-35_SOD27_P7.62mm_Horizontal
- RV1, RV2: footprint Potentiometers:Potentiometer_WirePads -> RFBitBanger:Potentiometer_Big_Small_Combined
- moved R71 24.3 mm to (161.7, 62.1)
- moved R37 20.7 mm to (94.2, 141.0), turned to 0 degrees
- moved R65 15.7 mm to (121.9, 64.4)
- moved R36 14.8 mm to (103.3, 127.1), turned to 270 degrees
- moved L11 13.5 mm to (164.3, 58.9)
- moved RV2 12.3 mm to (116.7, 142.8), turned to 0 degrees
- moved R58 10.4 mm to (129.2, 132.4), turned to 0 degrees
- moved RV1 10.3 mm to (85.7, 143.2), turned to 0 degrees
- moved D19 10.2 mm to (136.3, 60.3), turned to 270 degrees
- moved R14 9.46 mm to (151.3, 69.1), turned to 90 degrees
- moved C54 7.37 mm to (128.9, 125.5)
- moved C22 6.01 mm to (136.4, 71.5), turned to 270 degrees
- moved C52 5.18 mm to (135.0, 123.3)
- moved R60 5.03 mm to (136.8, 129.2), turned to 180 degrees
- moved C14 4.66 mm to (157.4, 67.5), turned to 270 degrees
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Routing:
- net Net-(L11-Pad2): track 27.0 -> 45.7 mm
- net Net-(L9-Pad2): track 50.0 -> 33.7 mm
- net Net-(C36-Pad1): track 183.5 -> 167.6 mm
- net Net-(D19-Pad1): track 4.58 -> 19.6 mm
- net Net-(C38-Pad1): track 35.0 -> 21.6 mm
- net +12V: track 265.7 -> 278.9 mm
- net Net-(Q12-Pad2): track 6.23 -> 19.0 mm
- net Net-(C19-Pad2): track 9.47 -> 20.7 mm
- net Net-(C50-Pad1): track 15.3 -> 24.3 mm
- net Net-(R63-Pad1): track 23.2 -> 30.7 mm
- net Net-(C34-Pad2): track 5.79 -> 12.2 mm
- net Net-(C54-Pad2): track 19.2 -> 13.8 mm
- net Net-(C21-Pad2): track 36.9 -> 41.8 mm
- net Net-(C39-Pad2): track 30.1 -> 34.6 mm
- net Net-(D18-Pad1): track 40.4 -> 36.7 mm
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
Commit message: Before trying to put everything onto a single line
Changed lines of the file:
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@@
     (links 446)
     (no_connects 0)
-    (area 40.949999 56.699999 190.100001 144.850001)
+    (area 40.490476 53.079999 194.775 149.415)
     (thickness 1.6)
     (drawings 50)
@@
   )
   (setup
-    (last_trace_width 0.5)
+    (last_trace_width 0.25)
     (user_trace_width 0.35)
     (user_trace_width 0.5)
@@
     (descr "C, Disc series, Radial, pin pitch=2.50mm, , diameter*width=5*2.5mm^2, Capacitor, http://cdn-reichelt.de/documents/datenblatt/B300/DS_KERKO_TC.pdf")
     (tags "C Disc series Radial pin pitch 2.50mm  diameter 5mm width 2.5mm Capacitor")
-    (fp_text reference C24 (at 4.83 0.16 540) (layer F.SilkS)
+    (fp_text reference C24 (at 1.04 -2.04 270) (layer F.SilkS)
       (effects (font (size 1 1) (thickness 0.15)))
     )
