File: RFBitBanger/RFBitBanger.kicad_pcb (KiCad board)
At the start: 2 copper layers, 149 x 88 mm, 234 parts, among them J1 POWER, J10 Conn_01x04, J11 SPEAKER, J12 Conn_Coaxial, J13 Conn_01x01, J14 Conn_01x01, J15 Conn_01x01, J16 Conn_01x01, J17 Filt1, J18 Filt2, J19 Conn_01x04, J2 Barrel_Jack, J20 Conn_01x01, J21 Conn_01x01, J22 SPEAKER, J3 Conn_01x01, J4 Conn_01x01, J5 Conn_01x04, J6 Conn_01x01, J7 Conn_01x01, J8 Conn_01x01, J9 ICSP, P1 Mini-DIN_6pins_ver4, Q1 2N3904, Q10 2N3904, Q11 2N3904, Q12 2N3904, Q13 2N2907, Q14 2N3904, Q15 NC, Q2 2N3904, Q3 2N7000, Q4 2N3904, Q5 NC, Q6 2N7000, Q7 2N7000, Q8 2N2907, Q9 2N7000, SW1 SW_Push, SW2 SW_Push, SW3 SW_Push, SW4 SW_Push, SW5 SW_Push, T1 Trifilar, T2 Trifilar, T3 Current, T4 Common-Mode Choke, U1 ATMEGA328-PU, U2 LM7805_TO220, U3 LM386, U4 LM358, U5 LCD-016N002L, U6 SI5351A, Y1 16 MHz, Y2 7.X MHz, Y3 27 MHz, Y4 7.X MHz, Y5 7.X MHz

Commit message: Changed external connector for single 20 pin or ribbon cable
Parts:
- removed J10, J19: Conn_01x04, Pin_Headers:Pin_Header_Straight_1x04_Pitch2.54mm
- removed J22: SPEAKER, Pin_Headers:Pin_Header_Straight_1x02_Pitch2.54mm
- U5: value LCD-016N002L -> LCD1602ExtraPins; footprint Pin_Headers:Pin_Header_Straight_1x16_Pitch2.54mm -> Pin_Headers:Pin_Header_Straight_1x20_Pitch2.54mm
- moved R76 22.1 mm to (91.8, 118.9), turned to 90 degrees
- moved Q14 9.19 mm to (50.7, 129.9)
- moved Q4 7.41 mm to (102.0, 116.6)
- moved R24 7.25 mm to (98.1, 115.7)
- moved C18 7.22 mm to (106.0, 120.4), turned to 0 degrees
- moved C41 5.19 mm to (66.0, 130.5)
- moved C37 4.89 mm to (75.6, 130.5)
- moved R11 3.79 mm to (65.0, 133.6)
- moved L10 3.43 mm to (76.0, 126.0)
- moved C42 2.04 mm to (50.0, 75.2)
- moved D1 1.13 mm to (53.3, 78.4)
- moved RV3 0.83 mm to (51.2, 88.1)
- moved J9 0.71 mm to (96.4, 108.0), turned to 180 degrees
- moved C11 0.31 mm to (62.4, 122.5)
- moved L1 0.14 mm to (65.6, 83.5)
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Connections:
- C19 pad 2: Net-(C19-Pad2) -> SPKR
- C7 pad 2: Net-(C7-Pad2) -> MICPADDLE
- J11 pad 1: Net-(C19-Pad2) -> SPKR
- R76 pad 1: Net-(J10-Pad1) -> Net-(R76-Pad1)
- U1 pad 24: Net-(C7-Pad2) -> MICPADDLE
Routing:
- net MICPADDLE: track 0.00 -> 77.7 mm
- net Net-(R76-Pad1): track 0.00 -> 70.0 mm
- net SPKR: track 0.00 -> 47.4 mm
- net GND: track 108.6 -> 132.8 mm
- net Net-(C19-Pad2): track 20.7 -> 0.00 mm
- net Net-(Q14-Pad3): track 6.17 -> 16.1 mm
- net Net-(C19-Pad1): track 24.3 -> 15.1 mm
- net Net-(C7-Pad2): track 8.89 -> 0.00 mm
- net RESET: track 79.5 -> 70.6 mm
- net MOSI: track 64.9 -> 56.2 mm
- net MISO: track 69.8 -> 61.8 mm
- net Net-(Q4-Pad2): track 9.67 -> 16.9 mm
- net Net-(J10-Pad1): track 4.68 -> 0.00 mm
- net Net-(Q14-Pad2): track 4.34 -> 8.81 mm
- net E: track 49.7 -> 45.3 mm
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Other:
- board text added: "AN"
- board text added: "KA"
- board text added: "PTT"
- board text added: "SPKR"
- board text removed: "KY1"

Commit message: JLCPCB order 2022-01-24
Parts:
- C48: footprint Capacitors_THT:C_Disc_D5.0mm_W2.5mm_P2.50mm -> Capacitors_THT:C_Disc_D5.0mm_W2.5mm_P5.00mm
- D8: value 1N4148 -> 1N4001; footprint Diodes_THT:D_DO-35_SOD27_P7.62mm_Horizontal -> Diodes_THT:D_DO-41_SOD81_P7.62mm_Horizontal
- moved R76 0.73 mm to (91.8, 119.6)
Routing:
- net Net-(C48-Pad2): track 23.6 -> 21.0 mm
- net TUNING: track 36.7 -> 37.7 mm
- net TRANSMIT: track 29.9 -> 30.7 mm
- net SCK: track 23.4 -> 24.1 mm
Other:
- board text added: "RFBITBANGER V5 BY DANIEL MARKS KW4TI CC-BY-SA 4.0"
- board text removed: "RFBITBANGER V4 BY DANIEL MARKS KW4TI CC-BY-SA 4.0"

Commit message: Before changing si5351 code
Changed lines of the file:
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@@
   )
   (setup
-    (last_trace_width 0.5)
+    (last_trace_width 0.25)
     (user_trace_width 0.35)
     (user_trace_width 0.5)
@@
     (descr "D, DO-41_SOD81 series, Axial, Horizontal, pin pitch=7.62mm, , length*diameter=5.2*2.7mm^2, , http://www.diodes.com/_files/packages/DO-41%20(Plastic).pdf")
     (tags "D DO-41_SOD81 series Axial Horizontal pin pitch 7.62mm  length 5.2mm diameter 2.7mm")
-    (fp_text reference D8 (at 3.81 -2.41) (layer F.SilkS)
+    (fp_text reference D8 (at 3.835 -0.045) (layer F.SilkS)
       (effects (font (size 1 1) (thickness 0.15)))
     )

Commit message: Added connector for SI5351A board
Parts:
- added J10: si5351mod, Pin_Headers:Pin_Header_Straight_1x07_Pitch2.54mm, F.Cu at (123.4, 108.6)
- C39: value 2.2 uH -> 1 uF
- C49: value 100 uF -> 22 uF
- C50: value 100 uF -> 10 uF
- moved R19 9.05 mm to (114.5, 114.1), turned to 180 degrees
- moved R18 8.14 mm to (124.5, 113.1), turned to 180 degrees
- moved Q4 5.40 mm to (96.6, 116.3)
- moved L3 5.23 mm to (105.1, 85.9)
- moved C18 5.13 mm to (101.0, 121.3), turned to 90 degrees
- moved C40 5.08 mm to (108.8, 118.0), turned to 270 degrees
- moved R24 5.06 mm to (93.0, 115.4)
- moved Y3 4.80 mm to (111.1, 92.5)
- moved R35 4.67 mm to (106.6, 96.8)
- moved R7 4.65 mm to (95.6, 89.6)
- moved L9 4.61 mm to (99.2, 99.0)
- moved C47 4.58 mm to (120.0, 99.8)
- moved R48 4.51 mm to (103.4, 96.8)
- moved U6 4.50 mm to (119.0, 95.0)
- moved R49 4.39 mm to (125.1, 94.7)
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Routing:
- net Net-(J10-Pad1): track 4.40 -> 21.3 mm
- net Net-(J10-Pad2): track 4.95 -> 19.2 mm
- net Net-(C47-Pad2): track 45.4 -> 32.7 mm, vias 0 -> 1
- net MISO: track 61.8 -> 70.4 mm, vias 3 -> 2
- net Net-(C40-Pad1): track 41.6 -> 34.2 mm
- net SCL: track 59.0 -> 66.2 mm, vias 0 -> 1
- net RESET: track 70.6 -> 77.5 mm, vias 2 -> 1
- net TRANSMIT: track 30.7 -> 37.0 mm
- net SDA: track 58.6 -> 64.7 mm, vias 0 -> 1
- net Net-(C36-Pad1): track 167.6 -> 162.0 mm
- net Net-(C48-Pad2): track 21.0 -> 16.5 mm
- net Net-(Q4-Pad2): track 16.9 -> 12.5 mm
- net +12V: track 277.1 -> 273.4 mm
- net Net-(R49-Pad2): track 9.47 -> 12.6 mm
- net Net-(C12-Pad1): track 12.4 -> 15.2 mm
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Other:
- board text added: "0"
- board text added: "2"
- board text added: "SI5351 MODULE"
- board text added: "VIN"

Commit message: Added fifth button
Parts:
- added C61: 100 nF, Capacitors_THT:C_Disc_D5.0mm_W2.5mm_P2.50mm, F.Cu at (49.8, 95.3)
- added R40: 10k, Resistors_THT:R_Axial_DIN0207_L6.3mm_D2.5mm_P7.62mm_Horizontal, F.Cu at (50.5, 89.0)
- added R75: 1k, Resistors_THT:R_Axial_DIN0207_L6.3mm_D2.5mm_P7.62mm_Horizontal, F.Cu at (62.5, 91.6)
- added SW6: SW_Push, Buttons_Switches_THT:SW_PUSH_6mm, F.Cu at (52.9, 91.5)
- moved D3 86.7 mm to (137.4, 137.6)
- moved R4 71.6 mm to (116.9, 135.6), turned to 0 degrees
- moved RV3 5.77 mm to (57.0, 88.2)
- moved R2 0.63 mm to (52.0, 98.9), turned to 0 degrees
- moved R63 0.50 mm to (124.6, 132.1)
Routing:
- net Net-(C61-Pad2): track 0.00 -> 17.1 mm
- net +5V: track 406.7 -> 416.4 mm, vias 0 -> 1
- net Net-(RV3-Pad2): track 17.5 -> 24.2 mm
- net MICPADDLE: track 77.7 -> 82.7 mm
- net Net-(D3-Pad2): track 6.94 -> 11.2 mm
- net E: track 45.3 -> 46.1 mm
Other:
- board text added: "RFBITBANGER V6 BY DANIEL MARKS KW4TI CC-BY-SA 4.0"
- board text removed: "RFBITBANGER V5 BY DANIEL MARKS KW4TI CC-BY-SA 4.0"

Commit message: Added extra row of ground pins for 40 pin connector
Parts:
- added J19: Conn_01x20, Pin_Headers:Pin_Header_Straight_1x20_Pitch2.54mm, F.Cu at (44.0, 72.5)
- C15: value NC -> 10 uF
- C53: value 100 uF -> 1000 uF; footprint Capacitors_THT:CP_Radial_D5.0mm_P2.50mm -> Capacitors_THT:CP_Radial_D8.0mm_P3.50mm
- moved R28 13.8 mm to (145.7, 142.1), turned to 0 degrees
- moved C15 10.1 mm to (75.1, 131.7)
- moved C37 7.27 mm to (81.5, 134.8), turned to 0 degrees
- moved D16 6.08 mm to (156.9, 140.0), turned to 270 degrees
- moved J18 3.81 mm to (161.3, 141.0)
- moved R21 3.48 mm to (152.4, 127.0)
- moved C43 3.24 mm to (152.4, 129.6)
- moved J15 3.19 mm to (155.9, 127.6)
- moved L7 2.90 mm to (176.6, 127.3)
- moved C53 2.82 mm to (53.6, 141.8)
- moved R22 2.13 mm to (145.8, 138.7)
- moved T3 2.03 mm to (176.6, 140.3)
- moved R11 1.91 mm to (63.1, 133.3), turned to 90 degrees
- moved L8 1.56 mm to (163.0, 131.4)
- moved C27 1.53 mm to (155.6, 124.4)
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Connections:
- C15 pad 2: Net-(C15-Pad2) -> GND
- U3 pad 1: Net-(C15-Pad1) -> (no net)
- U3 pad 7: (no net) -> Net-(C15-Pad1)
- U3 pad 8: Net-(C15-Pad2) -> (no net)
Routing:
- net Net-(D16-Pad2): track 9.59 -> 19.8 mm
- net Net-(C31-Pad2): track 57.7 -> 63.8 mm
- net Net-(C15-Pad2): track 5.95 -> 0.00 mm
- net Net-(RV3-Pad2): track 24.2 -> 30.1 mm
- net Net-(R2-Pad1): track 21.2 -> 27.0 mm
- net +12V: track 273.4 -> 279.1 mm
- net Net-(L10-Pad1): track 13.0 -> 18.3 mm
- net +5V: track 416.4 -> 421.3 mm
- net MICPADDLE: track 82.7 -> 87.6 mm
- net Net-(C29-Pad2): track 17.9 -> 22.3 mm
- net Net-(C26-Pad2): track 43.9 -> 40.7 mm
- net Net-(C49-Pad1): track 12.1 -> 9.77 mm
- net Net-(C43-Pad1): track 8.91 -> 6.87 mm
- net Net-(C19-Pad1): track 15.1 -> 16.8 mm
- net Net-(D16-Pad1): track 5.80 -> 4.38 mm
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Other:
- board size 149 x 88 mm -> 152 x 88 mm
- board text removed: "SPKR"

Commit message: Changed around for external filter PCB
Parts:
- removed C28, C31: 220 pF, Capacitors_THT:C_Disc_D5.0mm_W2.5mm_P5.00mm
- removed C29: 680 pF, Capacitors_THT:C_Disc_D5.0mm_W2.5mm_P5.00mm
- removed JP6: BYPASS, Pin_Headers:Pin_Header_Straight_1x02_Pitch2.54mm
- removed L7, L8: 1.35 uH, RFBitBanger:SmallVerticalToroid
- removed R42, R43, R44, R45: 1R0, Resistors_THT:R_Axial_DIN0207_L6.3mm_D2.5mm_P7.62mm_Horizontal
- removed R69: 330R, Resistors_THT:R_Axial_DIN0207_L6.3mm_D2.5mm_P7.62mm_Horizontal
- C23, C26: footprint Capacitors_THT:C_Disc_D5.0mm_W2.5mm_P2.50mm -> Capacitors_THT:C_Disc_D5.0mm_W2.5mm_P5.00mm
- J17, J18: footprint Pin_Headers:Pin_Header_Straight_1x02_Pitch2.54mm -> Pin_Headers:Pin_Header_Straight_1x04_Pitch2.54mm
- Q13, Q8: value 2N2907 -> SS8050
- R20: value 330R -> 100R
- R28: value 1k -> 47R
- R41: value 220R -> 150R
- R52: value 10k -> 47k
- R66: value 22k -> 470k
- moved R28 29.4 mm to (174.2, 134.8), turned to 180 degrees
- moved D16 22.8 mm to (177.8, 130.8)
- moved C32 12.4 mm to (176.6, 95.3), turned to 180 degrees
- moved D6 11.6 mm to (186.9, 95.3)
- moved C26 11.5 mm to (176.1, 120.6)
- moved JP4 11.2 mm to (169.7, 127.0), turned to 0 degrees
- moved R21 10.7 mm to (153.8, 137.6)
- moved JP7 9.66 mm to (176.6, 116.8), turned to 270 degrees
- moved JP2 7.32 mm to (173.4, 126.9), turned to 0 degrees
- moved C27 4.87 mm to (151.9, 127.6)
- moved C43 4.86 mm to (156.9, 131.4)
- moved J17 3.81 mm to (157.5, 120.7)
- moved J18 3.81 mm to (157.5, 141.0)
- moved C49 3.27 mm to (147.6, 138.1)
- moved L5 3.21 mm to (148.5, 122.5)
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Connections:
- J17 pad 2: Net-(C26-Pad2) -> GND
- J18 pad 2: Net-(C31-Pad2) -> GND
- JP2 pad 2: Net-(C31-Pad2) -> Net-(J18-Pad3)
- JP4 pad 2: Net-(C31-Pad2) -> Net-(J18-Pad3)
- JP7 pad 3: Net-(C31-Pad2) -> Net-(J18-Pad3)
- Q3 pad 1: Net-(Q3-Pad1) -> GND
- Q5 pad 1: Net-(Q5-Pad1) -> GND
- Q6 pad 1: Net-(Q6-Pad1) -> GND
- Q7 pad 1: Net-(Q7-Pad1) -> GND
- R28 pad 1: GND -> Net-(D16-Pad1)
- R28 pad 2: Net-(D16-Pad1) -> GND
- R49 pad 2: Net-(R49-Pad2) -> PLLOSC
- R50 pad 2: Net-(R49-Pad2) -> PLLOSC
- T3 pad 1: Net-(J12-Pad1) -> Net-(J18-Pad3)
- T3 pad 2: Net-(C31-Pad2) -> Net-(J12-Pad1)
Routing:
- net Net-(C31-Pad2): track 63.8 -> 0.00 mm
- net Net-(J18-Pad3): track 0.00 -> 41.9 mm
- net Net-(C26-Pad2): track 40.7 -> 15.7 mm
- net Net-(C29-Pad2): track 22.3 -> 0.00 mm
- net Net-(D16-Pad2): track 19.8 -> 3.57 mm
- net Net-(C23-Pad2): track 89.6 -> 75.4 mm
- net Net-(C28-Pad1): track 13.1 -> 0.00 mm
- net Net-(R49-Pad2): track 12.6 -> 0.00 mm
- net AMPOUT: track 129.5 -> 119.5 mm
- net PLLOSC: track 3.56 -> 13.2 mm
- net Net-(C43-Pad1): track 6.87 -> 12.7 mm
- net Net-(Q6-Pad1): track 5.36 -> 0.00 mm
- net Net-(Q7-Pad1): track 5.13 -> 0.00 mm
- net Net-(JP7-Pad2): track 5.17 -> 10.0 mm
- net Net-(Q3-Pad1): track 4.70 -> 0.00 mm
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Other:
- board text added: "INP"
- board text added: "OUT"
- board text added: "RFBITBANGER V8 BY DANIEL MARKS KW4TI CC-BY-SA 4.0"
- board text removed: "FILT1"
- board text removed: "FILT2"
- board text removed: "RFBITBANGER V6 BY DANIEL MARKS KW4TI CC-BY-SA 4.0"

Commit message: BandPassFilter now has six filter boards on it
Routing:
- net Net-(C23-Pad2): track 75.4 -> 84.9 mm
Changed lines of the file:
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@@
   (general
     (links 467)
-    (no_connects 1)
-    (area 37.924999 56.924999 190.075001 145.075001)
+    (no_connects 0)
+    (area 37.924999 53.079999 194.775 145.505)
     (thickness 1.6)
     (drawings 57)
-    (tracks 1608)
+    (tracks 1612)
     (zones 0)
     (modules 226)
@@
   (segment (start 121.235 72.105) (end 120.95 72.39) (width 0.5) (layer B.Cu) (net 14) (status 30))
   (segment (start 120.915 72.425) (end 120.95 72.39) (width 0.5) (layer B.Cu) (net 14) (status 30))
-  (segment (start 154.95 79.8) (end 158.19 79.8) (width 0.5) (layer B.Cu) (net 15) (status 400000))
-  (segment (start 158.19 79.8) (end 161.81 76.18) (width 0.5) (layer B.Cu) (net 15) (status 800000))
-  (segment (start 161.81 76.18) (end 161.81 75.55) (width 0.5) (layer B.Cu) (net 15) (status C00000))
-  (segment (start 161.81 75.55) (end 162.27 75.55) (width 0.5) (layer B.Cu) (net 15) (status C00000))
-  (segment (start 162.27 75.55) (end 164.4 77.68) (width 0.5) (layer B.Cu) (net 15) (status C00000))
+  (segment (start 171.83 80.915) (end 166.465 80.915) (width 0.5) (layer B.Cu) (net 15))
+  (segment (start 164.4 78.85) (end 164.4 77.68) (width 0.5) (layer B.Cu) (net 15))
+  (segment (start 166.465 80.915) (end 164.4 78.85) (width 0.5) (layer B.Cu) (net 15))
+  (segment (start 154.95 79.8) (end 158.19 79.8) (width 0.5) (layer B.Cu) (net 15))
+  (segment (start 158.19 79.8) (end 161.81 76.18) (width 0.5) (layer B.Cu) (net 15))
+  (segment (start 161.81 76.18) (end 161.81 75.55) (width 0.5) (layer B.Cu) (net 15))
+  (segment (start 161.81 75.55) (end 162.27 75.55) (width 0.5) (layer B.Cu) (net 15))
+  (segment (start 162.27 75.55) (end 164.4 77.68) (width 0.5) (layer B.Cu) (net 15))
   (segment (start 172.63 89.1) (end 172.62 89.1) (width 0.5) (layer B.Cu) (net 15))
   (segment (start 169.715 86.195) (end 169.715 80.915) (width 0.5) (layer B.Cu) (net 15))
   (segment (start 172.62 89.1) (end 169.715 86.195) (width 0.5) (layer B.Cu) (net 15))
-  (segment (start 175.18 80.915) (end 169.715 80.915) (width 0.5) (layer B.Cu) (net 15))
+  (segment (start 175.18 80.915) (end 171.83 80.915) (width 0.5) (layer B.Cu) (net 15))
+  (segment (start 171.83 80.915) (end 169.715 80.915) (width 0.5) (layer B.Cu) (net 15))
   (segment (start 173.03 79.06) (end 174.885 80.915) (width 0.5) (layer B.Cu) (net 15))
   (segment (start 181.075 80.915) (end 182.75 78.73) (width 0.5) (layer B.Cu) (net 15) (status 20))
@@
   (segment (start 133.52 90.55) (end 133.5 90.53) (width 0.5) (layer B.Cu) (net 75))
   (segment (start 133.56 90.59) (end 133.5 90.53) (width 0.5) (layer B.Cu) (net 75) (status 30))
-  (segment (start 157.78 75.84) (end 157.78 76.89) (width 0.5) (layer B.Cu) (net 76) (status 400000))
-  (segment (start 150.96 79.79) (end 150.96 85.13) (width 0.5) (layer B.Cu) (net 76) (status 800000))
+  (segment (start 157.78 75.84) (end 157.78 76.89) (width 0.5) (layer B.Cu) (net 76))
+  (segment (start 150.96 79.79) (end 150.96 85.13) (width 0.5) (layer B.Cu) (net 76))
   (segment (start 152.85 77.9) (end 150.96 79.79) (width 0.5) (layer B.Cu) (net 76))
   (segment (start 156.77 77.9) (end 152.85 77.9) (width 0.5) (layer B.Cu) (net 76))
@@
   (segment (start 176.335 111.545) (end 180.175 111.545) (width 0.5) (layer B.Cu) (net 93))
   (segment (start 174.02 113.86) (end 176.335 111.545) (width 0.5) (layer B.Cu) (net 93))
-  (segment (start 167.64 84.73) (end 167.64 87.84) (width 0.5) (layer B.Cu) (net 94) (status 400000))
-  (segment (start 167.64 87.84) (end 170.48 90.68) (width 0.5) (layer B.Cu) (net 94) (status 800000))
-  (segment (start 167.64 77.11) (end 167.64 76.78) (width 0.5) (layer B.Cu) (net 94) (status C00000))
-  (segment (start 167.64 76.78) (end 169.18 75.24) (width 0.5) (layer B.Cu) (net 94) (status 400000))
+  (segment (start 167.64 84.73) (end 167.64 87.84) (width 0.5) (layer B.Cu) (net 94))
+  (segment (start 167.64 87.84) (end 170.48 90.68) (width 0.5) (layer B.Cu) (net 94))
+  (segment (start 167.64 77.11) (end 167.64 76.78) (width 0.5) (layer B.Cu) (net 94))
+  (segment (start 167.64 76.78) (end 169.18 75.24) (width 0.5) (layer B.Cu) (net 94))
   (segment (start 169.18 75.24) (end 175.57 75.24) (width 0.5) (layer B.Cu) (net 94))
   (segment (start 161.335 82.9) (end 161.335 83.955) (width 0.5) (layer B.Cu) (net 94))
@@
   (segment (start 49.15 112.7) (end 49.15 122.05) (width 0.35) (layer B.Cu) (net 106))
   (segment (start 49.15 122.05) (end 50.72 124.84) (width 0.35) (layer B.Cu) (net 106) (status 20))
-  (segment (start 166.835 63.005) (end 165.015 63.005) (width 0.5) (layer B.Cu) (net 107) (status 400000))
-  (segment (start 161.81 66.21) (end 161.81 67.93) (width 0.5) (layer B.Cu) (net 107) (status 800000))
+  (segment (start 166.835 63.005) (end 165.015 63.005) (width 0.5) (layer B.Cu) (net 107))
+  (segment (start 161.81 66.21) (end 161.81 67.93) (width 0.5) (layer B.Cu) (net 107))
   (segment (start 165.015 63.005) (end 161.81 66.21) (width 0.5) (layer B.Cu) (net 107))
   (segment (start 164.29 58.87) (end 164.79 58.87) (width 0.5) (layer B.Cu) (net 107))
