File: RFBitBanger/RFBitBanger.kicad_pcb (KiCad board)
At the start: 2 copper layers, 152 x 88 mm, 226 parts, among them J1 POWER, J10 si5351mod, J11 SPEAKER, J12 Conn_Coaxial, J13 Conn_01x01, J14 Conn_01x01, J15 Conn_01x01, J16 Conn_01x01, J17 Filt1, J18 Filt2, J19 Conn_01x20, J2 Barrel_Jack, J20 Conn_01x01, J21 Conn_01x01, J3 Conn_01x01, J4 Conn_01x01, J5 Conn_01x04, J6 Conn_01x01, J7 Conn_01x01, J8 Conn_01x01, J9 ICSP, P1 Mini-DIN_6pins_ver4, Q1 2N3904, Q10 2N3904, Q11 2N3904, Q12 2N3904, Q13 SS8050, Q14 2N3904, Q15 NC, Q2 2N3904, Q3 2N7000, Q4 2N3904, Q5 NC, Q6 2N7000, Q7 2N7000, Q8 SS8050, Q9 2N7000, SW1 SW_Push, SW2 SW_Push, SW3 SW_Push, SW4 SW_Push, SW5 SW_Push, SW6 SW_Push, T1 Trifilar, T2 Trifilar, T3 Current, T4 Common-Mode Choke, U1 ATMEGA328-PU, U2 LM7805_TO220, U3 LM386, U4 LM358, U5 LCD1602ExtraPins, U6 SI5351A, Y1 16 MHz, Y2 7.X MHz, Y3 27 MHz, Y4 7.X MHz, Y5 7.X MHz

Commit message: Added New Documentation
Parts:
- moved R41 3.73 mm to (174.0, 101.6)
Connections:
- J17 pad 4: Net-(C26-Pad2) -> Net-(J17-Pad4)
- JP7 pad 1: Net-(C26-Pad1) -> Net-(J17-Pad4)
Routing:
- net Net-(J17-Pad4): track 0.00 -> 15.7 mm
- net Net-(JP7-Pad2): track 10.0 -> 17.5 mm
- net Net-(C26-Pad1): track 19.8 -> 13.3 mm
- net Net-(Q9-Pad1): track 10.2 -> 12.7 mm
- net Net-(C26-Pad2): track 15.7 -> 14.9 mm
Changed lines of the file:
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@@
 (kicad_pcb (version 4) (host pcbnew 4.0.7)
   (general
-    (links 467)
+    (links 466)
     (no_connects 0)
-    (area 37.924999 53.079999 194.775 145.505)
+    (area 37.924999 56.924999 190.075001 145.075001)
     (thickness 1.6)
     (drawings 57)
-    (tracks 1612)
+    (tracks 1615)
     (zones 0)
     (modules 226)
-    (nets 125)
+    (nets 126)
   )
   (page A4)
@@
   (net 123 "Net-(C61-Pad2)")
   (net 124 "Net-(J18-Pad3)")
+  (net 125 "Net-(J17-Pad4)")
   (net_class Default "This is the default net class."
     (clearance 0.2)
@@
     (add_net "Net-(J10-Pad2)")
     (add_net "Net-(J12-Pad1)")
+    (add_net "Net-(J17-Pad4)")
     (add_net "Net-(J18-Pad3)")
     (add_net "Net-(J9-Pad2)")
@@
     )
     (pad 1 thru_hole rect (at 0 0 270) (size 1.7 1.7) (drill 1) (layers *.Cu *.Mask)
-      (net 16 "Net-(C26-Pad1)"))
+      (net 125 "Net-(J17-Pad4)"))
     (pad 2 thru_hole oval (at 0 2.54 270) (size 1.7 1.7) (drill 1) (layers *.Cu *.Mask)
       (net 93 "Net-(JP7-Pad2)"))
@@
   )
   (module Resistors_THT:R_Axial_DIN0309_L9.0mm_D3.2mm_P12.70mm_Horizontal (layer F.Cu)
-    (at 177.68 102.11 180)
+    (at 173.99 101.6 180)
     (descr "Resistor, Axial_DIN0309 series, Axial, Horizontal, pin pitch=12.7mm, 0.5W = 1/2W, length*diameter=9*3.2mm^2, http://cdn-reichelt.de/documents/datenblatt/B400/1_4W%23YAG.pdf")
     (tags "Resistor Axial_DIN0309 series Axial Horizontal pin pitch 12.7mm 0.5W = 1/2W length 9mm diameter 3.2mm")
@@
       (net 17 "Net-(C26-Pad2)"))
     (pad 4 thru_hole oval (at 0 7.62 90) (size 1.7 1.7) (drill 1) (layers *.Cu *.Mask)
-      (net 17 "Net-(C26-Pad2)"))
+      (net 125 "Net-(J17-Pad4)"))
     (model ${KISYS3DMOD}/Pin_Headers.3dshapes/Pin_Header_Straight_1x04_Pitch2.54mm.wrl
       (at (xyz 0 0 0))
@@
   (segment (start 182.85 78.83) (end 182.75 78.73) (width 0.5) (layer B.Cu) (net 15) (status 30))
   (segment (start 172.9 78.92) (end 173.03 78.79) (width 0.5) (layer B.Cu) (net 15) (status 30))
-  (segment (start 180.6 119.06) (end 177.64 119.06) (width 0.5) (layer B.Cu) (net 16))
-  (segment (start 177.64 119.06) (end 176.08 120.62) (width 0.5) (layer B.Cu) (net 16))
-  (segment (start 187.775 116.625) (end 187.775 117.865) (width 0.5) (layer B.Cu) (net 16))
-  (segment (start 176.56 118) (end 176.56 116.78) (width 0.5) (layer B.Cu) (net 16))
-  (segment (start 177.62 119.06) (end 176.56 118) (width 0.5) (layer B.Cu) (net 16))
-  (segment (start 186.58 119.06) (end 180.6 119.06) (width 0.5) (layer B.Cu) (net 16))
-  (segment (start 180.6 119.06) (end 177.93 119.06) (width 0.5) (layer B.Cu) (net 16))
-  (segment (start 177.93 119.06) (end 177.62 119.06) (width 0.5) (layer B.Cu) (net 16))
-  (segment (start 187.775 117.865) (end 186.58 119.06) (width 0.5) (layer B.Cu) (net 16))
-  (segment (start 169.66 126.99) (end 169.66 122.04) (width 0.5) (layer B.Cu) (net 17))
+  (segment (start 176.08 120.62) (end 183.78 120.62) (width 0.5) (layer B.Cu) (net 16))
+  (segment (start 183.78 120.62) (end 187.775 116.625) (width 0.5) (layer B.Cu) (net 16))
+  (segment (start 162.56 120.65) (end 162.56 120.88) (width 0.5) (layer B.Cu) (net 17))
+  (segment (start 162.56 120.88) (end 164.06 122.38) (width 0.5) (layer B.Cu) (net 17))
+  (segment (start 164.06 122.38) (end 169.66 122.38) (width 0.5) (layer B.Cu) (net 17))
+  (segment (start 169.66 126.99) (end 169.66 122.38) (width 0.5) (layer B.Cu) (net 17))
+  (segment (start 169.66 122.38) (end 169.66 122.04) (width 0.5) (layer B.Cu) (net 17))
   (segment (start 169.66 122.04) (end 171.08 120.62) (width 0.5) (layer B.Cu) (net 17))
-  (segment (start 171.08 120.62) (end 165.13 120.62) (width 0.5) (layer B.Cu) (net 17) (status 20))
-  (segment (start 165.13 120.62) (end 165.1 120.65) (width 0.5) (layer B.Cu) (net 17) (status 30))
-  (segment (start 165.1 120.65) (end 162.56 120.65) (width 0.5) (layer B.Cu) (net 17) (status 30))
-  (segment (start 165.28 120.47) (end 165.1 120.65) (width 0.5) (layer B.Cu) (net 17) (status 30))
   (segment (start 96.74 133.31) (end 95.81 133.31) (width 0.5) (layer B.Cu) (net 18))
   (segment (start 95.81 133.31) (end 93.5 135.62) (width 0.5) (layer B.Cu) (net 18))
@@
   (segment (start 147.7 92.75) (end 147.69 92.76) (width 0.5) (layer B.Cu) (net 72))
   (segment (start 147.76 92.83) (end 147.69 92.76) (width 0.5) (layer B.Cu) (net 72) (status 30))
+  (segment (start 161.29 101.6) (end 163.83 101.6) (width 0.5) (layer B.Cu) (net 73))
+  (segment (start 165.24 100.19) (end 165.24 95.94) (width 0.5) (layer B.Cu) (net 73))
+  (segment (start 163.83 101.6) (end 165.24 100.19) (width 0.5) (layer B.Cu) (net 73))
   (segment (start 164.44 92.58) (end 164.44 95.14) (width 0.5) (layer B.Cu) (net 73))
   (segment (start 164.44 95.14) (end 165.24 95.94) (width 0.5) (layer B.Cu) (net 73))
-  (segment (start 165.24 95.94) (end 165.24 101.85) (width 0.5) (layer B.Cu) (net 73))
-  (segment (start 165.24 101.85) (end 164.98 102.11) (width 0.5) (layer B.Cu) (net 73))
   (segment (start 165.325 95.735) (end 165.24 95.94) (width 0.5) (layer B.Cu) (net 73) (status 30))
   (segment (start 125.6 89.06) (end 125.6 86.06) (width 0.5) (layer B.Cu) (net 74))
@@
   (segment (start 132.74 94.68) (end 132.74 97.84) (width 0.5) (layer B.Cu) (net 92))
   (segment (start 132.74 97.84) (end 132.82 97.92) (width 0.5) (layer B.Cu) (net 92))
-  (segment (start 174.02 116.78) (end 174.02 113.86) (width 0.5) (layer B.Cu) (net 93))
-  (segment (start 176.335 111.545) (end 180.175 111.545) (width 0.5) (layer B.Cu) (net 93))
-  (segment (start 174.02 113.86) (end 176.335 111.545) (width 0.5) (layer B.Cu) (net 93))
+  (segment (start 174.02 116.78) (end 174.02 117.75) (width 0.5) (layer B.Cu) (net 93))
+  (segment (start 182.58 113.95) (end 180.175 111.545) (width 0.5) (layer B.Cu) (net 93))
+  (segment (start 182.58 117.5) (end 182.58 113.95) (width 0.5) (layer B.Cu) (net 93))
+  (segment (start 181.28 118.8) (end 182.58 117.5) (width 0.5) (layer B.Cu) (net 93))
+  (segment (start 175.07 118.8) (end 181.28 118.8) (width 0.5) (layer B.Cu) (net 93))
+  (segment (start 174.02 117.75) (end 175.07 118.8) (width 0.5) (layer B.Cu) (net 93))
   (segment (start 167.64 84.73) (end 167.64 87.84) (width 0.5) (layer B.Cu) (net 94))
   (segment (start 167.64 87.84) (end 170.48 90.68) (width 0.5) (layer B.Cu) (net 94))
@@
   (segment (start 173.48 139.18) (end 174 139.7) (width 0.5) (layer B.Cu) (net 124))
   (segment (start 165.1 140.97) (end 162.56 140.97) (width 0.5) (layer B.Cu) (net 124) (status 30))
+  (segment (start 165.1 120.65) (end 165.1 119.93) (width 0.5) (layer B.Cu) (net 125))
+  (segment (start 165.1 119.93) (end 170.54 114.49) (width 0.5) (layer B.Cu) (net 125))
+  (segment (start 174.27 114.49) (end 176.56 116.78) (width 0.5) (layer B.Cu) (net 125))
+  (segment (start 170.54 114.49) (end 174.27 114.49) (width 0.5) (layer B.Cu) (net 125))
+  (segment (start 165.13 120.62) (end 165.1 120.65) (width 0.5) (layer B.Cu) (net 125) (status 30))
+  (segment (start 165.28 120.47) (end 165.1 120.65) (width 0.5) (layer B.Cu) (net 125) (status 30))
   (zone (net 0) (net_name "") (layer F.Mask) (hatch edge 0.508)
     (connect_pads (clearance 0.75))

Commit message: Increased size of heatsink pad
Parts:
- moved Q7 3.22 mm to (180.0, 75.5)
- moved Q3 3.16 mm to (170.3, 75.6)
- moved Q15 1.57 mm to (187.2, 80.8)
- moved J13 1.44 mm to (177.6, 83.2)
Routing:
- net AMPOUT: track 119.5 -> 109.2 mm
- net Net-(C23-Pad2): track 84.9 -> 91.5 mm

Commit message: Converted all Kicad projects to version 6.0.10
Routing:
- net +5V: track 421.3 -> 415.6 mm
- net Net-(C36-Pad1): track 162.0 -> 158.1 mm
- net AMPOUT: track 109.2 -> 105.7 mm
- net Net-(C14-Pad2): track 63.7 -> 60.5 mm
- net Net-(C23-Pad2): track 91.5 -> 89.2 mm
- net MICPADDLE: track 87.6 -> 85.2 mm
- net +12V: track 279.1 -> 276.8 mm
- net Net-(C19-Pad1): track 16.8 -> 14.8 mm
- net RESET: track 77.5 -> 75.9 mm
- net TXRELAY: track 44.8 -> 43.2 mm
- net SPKR: track 46.3 -> 45.0 mm
- net Net-(C50-Pad1): track 24.3 -> 23.0 mm
- net TUNING: track 40.4 -> 39.1 mm
- net Net-(C14-Pad1): track 18.6 -> 17.3 mm
- net Net-(C16-Pad2): track 29.1 -> 27.9 mm
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Other:
- net class Default removed

Commit message: Added RFBitBangerNano
Parts:
- C48: value 100 nF -> 100 pF
- Q13, Q8: value SS8050 -> SS8550
- R49, R50: value 100R -> 47R
- R73: value 1k -> 10k
Connections:
- J10 pad 3: (no net) -> unconnected-(J10-Pad3)
- J2 pad 3: (no net) -> unconnected-(J2-Pad3)
- RLY1 pad 3: (no net) -> Net-(RLY1-Pad3)
- RLY1 pad 8: (no net) -> unconnected-(RLY1-Pad8)
- U3 pad 1: (no net) -> unconnected-(U3-Pad1)
- U3 pad 8: (no net) -> unconnected-(U3-Pad8)
- U5 pad 10: (no net) -> unconnected-(U5-Pad10)
- U5 pad 7: (no net) -> unconnected-(U5-Pad7)
- U5 pad 8: (no net) -> unconnected-(U5-Pad8)
- U5 pad 9: (no net) -> unconnected-(U5-Pad9)
- U6 pad 6: (no net) -> unconnected-(U6-Pad6)

Commit message: Added two dual capacitor footprints to RFBitBanger
Parts:
- C26, C32: footprint Capacitors_THT:C_Disc_D5.0mm_W2.5mm_P5.00mm -> RFBitBanger:C_Disc_D5.0mm_W2.5mm_P5.00mm_Dual
Changed lines of the file:
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@@
     )
   )
-  (footprint "Capacitors_THT:C_Disc_D5.0mm_W2.5mm_P5.00mm" (layer "F.Cu")
+  (footprint "RFBitBanger:C_Disc_D5.0mm_W2.5mm_P5.00mm_Dual" (layer "F.Cu")
     (at 176.56 95.33 180)
     (descr "C, Disc series, Radial, pin pitch=5.00mm, , diameter*width=5*2.5mm^2, Capacitor, http://cdn-reichelt.de/documents/datenblatt/B300/DS_KERKO_TC.pdf")
@@
     (property "Sheetname" "RFBitBangerRadio")
     (attr through_hole)
-    (fp_text reference "C32" (at 2.54 0.03 180) (layer "F.SilkS")
+    (fp_text reference "C32" (at 2.49 -2.29) (layer "F.SilkS")
       (effects (font (size 1 1) (thickness 0.15)))
     )
-    (fp_text value "33 pF" (at 2.5 2.56 180) (layer "F.Fab")
-      (effects (font (size 1 1) (thickness 0.15)))
+    (fp_text value "33 pF" (at 2.54 0 270) (layer "F.Fab")
+      (effects (font (size 0.5 0.5) (thickness 0.125)))
     )
-    (fp_text user "${REFERENCE}" (at 2.5 0 180) (layer "F.Fab")
-      (effects (font (size 1 1) (thickness 0.15)))
+    (fp_text user "${REFERENCE}" (at 2.5 0 270) (layer "F.Fab")
+      (effects (font (size 0.5 0.5) (thickness 0.125)))
     )
-    (fp_line (start -0.06 0.996) (end -0.06 1.31) (layer "F.SilkS") (width 0.12))
     (fp_line (start -0.06 -1.31) (end -0.06 -0.996) (layer "F.SilkS") (width 0.12))
-    (fp_line (start -0.06 -1.31) (end 5.06 -1.31) (layer "F.SilkS") (width 0.12))
-    (fp_line (start 5.06 -1.31) (end 5.06 -0.996) (layer "F.SilkS") (width 0.12))
     (fp_line (start 5.06 0.996) (end 5.06 1.31) (layer "F.SilkS") (width 0.12))
+    (fp_line (start -0.06 -1.31) (end 5.06 -1.31) (layer "F.SilkS") (width 0.12))
     (fp_line (start -0.06 1.31) (end 5.06 1.31) (layer "F.SilkS") (width 0.12))
+    (fp_line (start 5.06 -1.31) (end 5.06 -0.996) (layer "F.SilkS") (width 0.12))
+    (fp_line (start -0.06 0.996) (end -0.06 1.31) (layer "F.SilkS") (width 0.12))
     (fp_line (start -1.05 -1.6) (end -1.05 1.6) (layer "F.CrtYd") (width 0.05))
-    (fp_line (start -1.05 1.6) (end 6.05 1.6) (layer "F.CrtYd") (width 0.05))
-    (fp_line (start 6.05 -1.6) (end -1.05 -1.6) (layer "F.CrtYd") (width 0.05))
     (fp_line (start 6.05 1.6) (end 6.05 -1.6) (layer "F.CrtYd") (width 0.05))
+    (fp_line (start 6.05 -1.6) (end -1.05 -1.6) (layer "F.CrtYd") (width 0.05))
+    (fp_line (start -1.05 1.6) (end 6.05 1.6) (layer "F.CrtYd") (width 0.05))
     (fp_line (start 0 1.25) (end 5 1.25) (layer "F.Fab") (width 0.1))
-    (fp_line (start 5 1.25) (end 5 -1.25) (layer "F.Fab") (width 0.1))
     (fp_line (start 5 -1.25) (end 0 -1.25) (layer "F.Fab") (width 0.1))
     (fp_line (start 0 -1.25) (end 0 1.25) (layer "F.Fab") (width 0.1))
-    (pad "1" thru_hole circle locked (at 0 0 180) (size 1.6 1.6) (drill 0.8) (layers *.Cu *.Mask)
+    (fp_line (start 5 1.25) (end 5 -1.25) (layer "F.Fab") (width 0.1))
+    (pad "1" smd rect (at 1.4 0 180) (size 1.524 1.524) (layers "F.Cu" "F.Paste" "F.Mask")
+      (net 94 "AMPOUT") (pintype "passive"))
+    (pad "1" thru_hole circle (at 0 0 180) (size 1.6 1.6) (drill 0.8) (layers *.Cu *.Mask)
       (net 94 "AMPOUT") (pintype "passive"))
-    (pad "2" thru_hole circle locked (at 5 0 180) (size 1.6 1.6) (drill 0.8) (layers *.Cu *.Mask)
+    (pad "2" thru_hole circle (at 5 0 180) (size 1.6 1.6) (drill 0.8) (layers *.Cu *.Mask)
+      (net 2 "GND") (pintype "passive"))
+    (pad "2" smd rect (at 3.6 0 180) (size 1.524 1.524) (layers "F.Cu" "F.Paste" "F.Mask")
       (net 2 "GND") (pintype "passive"))
     (model "${KISYS3DMOD}/Capacitors_THT.3dshapes/C_Disc_D5.0mm_W2.5mm_P5.00mm.wrl"
@@
     )
   )
-  (footprint "Capacitors_THT:C_Disc_D5.0mm_W2.5mm_P5.00mm" (layer "F.Cu")
+  (footprint "RFBitBanger:C_Disc_D5.0mm_W2.5mm_P5.00mm_Dual" (layer "F.Cu")
     (at 176.08 120.62 180)
     (descr "C, Disc series, Radial, pin pitch=5.00mm, , diameter*width=5*2.5mm^2, Capacitor, http://cdn-reichelt.de/documents/datenblatt/B300/DS_KERKO_TC.pdf")
@@
     (property "Sheetname" "RFBitBangerRadio")
     (attr through_hole)
-    (fp_text reference "C26" (at 2.49 0 180) (layer "F.SilkS")
+    (fp_text reference "C26" (at 2.56 -2.32) (layer "F.SilkS")
       (effects (font (size 1 1) (thickness 0.15)))
     )
-    (fp_text value "10 nF" (at 2.5 2.56 180) (layer "F.Fab")
-      (effects (font (size 1 1) (thickness 0.15)))
+    (fp_text value "10 nF" (at 2.54 0 270) (layer "F.Fab")
+      (effects (font (size 0.5 0.5) (thickness 0.125)))
     )
-    (fp_text user "${REFERENCE}" (at 2.5 0 180) (layer "F.Fab")
-      (effects (font (size 1 1) (thickness 0.15)))
+    (fp_text user "${REFERENCE}" (at 2.5 0 270) (layer "F.Fab")
+      (effects (font (size 0.5 0.5) (thickness 0.125)))
     )
     (fp_line (start -0.06 -1.31) (end 5.06 -1.31) (layer "F.SilkS") (width 0.12))
-    (fp_line (start 5.06 0.996) (end 5.06 1.31) (layer "F.SilkS") (width 0.12))
-    (fp_line (start -0.06 0.996) (end -0.06 1.31) (layer "F.SilkS") (width 0.12))
+    (fp_line (start -0.06 -1.31) (end -0.06 -0.996) (layer "F.SilkS") (width 0.12))
     (fp_line (start -0.06 1.31) (end 5.06 1.31) (layer "F.SilkS") (width 0.12))
+    (fp_line (start -0.06 0.996) (end -0.06 1.31) (layer "F.SilkS") (width 0.12))
+    (fp_line (start 5.06 0.996) (end 5.06 1.31) (layer "F.SilkS") (width 0.12))
     (fp_line (start 5.06 -1.31) (end 5.06 -0.996) (layer "F.SilkS") (width 0.12))
-    (fp_line (start -0.06 -1.31) (end -0.06 -0.996) (layer "F.SilkS") (width 0.12))
-    (fp_line (start -1.05 1.6) (end 6.05 1.6) (layer "F.CrtYd") (width 0.05))
-    (fp_line (start 6.05 1.6) (end 6.05 -1.6) (layer "F.CrtYd") (width 0.05))
     (fp_line (start 6.05 -1.6) (end -1.05 -1.6) (layer "F.CrtYd") (width 0.05))
     (fp_line (start -1.05 -1.6) (end -1.05 1.6) (layer "F.CrtYd") (width 0.05))
-    (fp_line (start 5 1.25) (end 5 -1.25) (layer "F.Fab") (width 0.1))
-    (fp_line (start 5 -1.25) (end 0 -1.25) (layer "F.Fab") (width 0.1))
+    (fp_line (start -1.05 1.6) (end 6.05 1.6) (layer "F.CrtYd") (width 0.05))
+    (fp_line (start 6.05 1.6) (end 6.05 -1.6) (layer "F.CrtYd") (width 0.05))
     (fp_line (start 0 -1.25) (end 0 1.25) (layer "F.Fab") (width 0.1))
+    (fp_line (start 5 1.25) (end 5 -1.25) (layer "F.Fab") (width 0.1))
     (fp_line (start 0 1.25) (end 5 1.25) (layer "F.Fab") (width 0.1))
-    (pad "1" thru_hole circle locked (at 0 0 180) (size 1.6 1.6) (drill 0.8) (layers *.Cu *.Mask)
+    (fp_line (start 5 -1.25) (end 0 -1.25) (layer "F.Fab") (width 0.1))
+    (pad "1" smd rect (at 1.4 0 180) (size 1.524 1.524) (layers "F.Cu" "F.Paste" "F.Mask")
       (net 16 "Net-(C26-Pad1)") (pintype "passive"))
-    (pad "2" thru_hole circle locked (at 5 0 180) (size 1.6 1.6) (drill 0.8) (layers *.Cu *.Mask)
+    (pad "1" thru_hole circle (at 0 0 180) (size 1.6 1.6) (drill 0.8) (layers *.Cu *.Mask)
+      (net 16 "Net-(C26-Pad1)") (pintype "passive"))
+    (pad "2" smd rect (at 3.6 0 180) (size 1.524 1.524) (layers "F.Cu" "F.Paste" "F.Mask")
+      (net 17 "Net-(C26-Pad2)") (pintype "passive"))
+    (pad "2" thru_hole circle (at 5 0 180) (size 1.6 1.6) (drill 0.8) (layers *.Cu *.Mask)
       (net 17 "Net-(C26-Pad2)") (pintype "passive"))
     (model "${KISYS3DMOD}/Capacitors_THT.3dshapes/C_Disc_D5.0mm_W2.5mm_P5.00mm.wrl"
@@
   (segment (start 171.83 129.45) (end 171.18 129.45) (width 0.5) (layer "B.Cu") (net 124))
   (segment (start 171.83 137.53) (end 174 139.7) (width 0.5) (layer "B.Cu") (net 124))
-  (segment (start 171.48 117.86) (end 173.2 119.58) (width 0.5) (layer "B.Cu") (net 124))
-  (segment (start 173.2 119.58) (end 173.2 122.32) (width 0.5) (layer "B.Cu") (net 124))
-  (segment (start 173.2 122.32) (end 171.55 123.97) (width 0.5) (layer "B.Cu") (net 124))
-  (segment (start 171.55 123.97) (end 171.55 129.08) (width 0.5) (layer "B.Cu") (net 124))
-  (segment (start 171.55 129.08) (end 171.18 129.45) (width 0.5) (layer "B.Cu") (net 124))
   (segment (start 171.18 129.45) (end 169.74 129.45) (width 0.5) (layer "B.Cu") (net 124))
   (segment (start 172.73 140.97) (end 174 139.7) (width 0.5) (layer "B.Cu") (net 124))
   (segment (start 171.83 129.45) (end 171.83 137.53) (width 0.5) (layer "B.Cu") (net 124))
-  (segment (start 171.48 116.78) (end 171.48 117.86) (width 0.5) (layer "B.Cu") (net 124))
+  (segment (start 171.48 117.86) (end 173.52 119.9) (width 0.5) (layer "B.Cu") (net 124))
+  (segment (start 171.55 129.08) (end 171.18 129.45) (width 0.5) (layer "B.Cu") (net 124))
+  (segment (start 173.52 122) (end 171.55 123.97) (width 0.5) (layer "B.Cu") (net 124))
+  (segment (start 171.55 123.97) (end 171.55 129.08) (width 0.5) (layer "B.Cu") (net 124))
   (segment (start 165.1 140.97) (end 172.73 140.97) (width 0.5) (layer "B.Cu") (net 124))
   (segment (start 173.43 129.45) (end 171.83 129.45) (width 0.5) (layer "B.Cu") (net 124))
+  (segment (start 173.52 119.9) (end 173.52 122) (width 0.5) (layer "B.Cu") (net 124))
   (segment (start 165.1 140.97) (end 162.56 140.97) (width 0.5) (layer "B.Cu") (net 124))
+  (segment (start 171.48 116.78) (end 171.48 117.86) (width 0.5) (layer "B.Cu") (net 124))
   (segment (start 165.1 119.93) (end 170.54 114.49) (width 0.5) (layer "B.Cu") (net 125))
   (segment (start 170.54 114.49) (end 174.27 114.49) (width 0.5) (layer "B.Cu") (net 125))
