File: RFBitBanger/RFBitBangerRadio.kicad_sch (KiCad schematic)
At the start: 135 parts, among them J10 si5351mod, J12 Conn_Coaxial, J17 Filt1, J18 Filt2, Q1 2N3904, Q10 2N3904, Q11 2N3904, Q12 2N3904, Q13 SS8550, Q15 NC, Q2 2N3904, Q3 2N7000, Q5 NC, Q6 2N7000, Q7 2N7000, Q8 SS8550, Q9 2N7000, T1 Trifilar, T2 Trifilar, T3 Current, U4 LM358, U6 SI5351A, Y2 7.X MHz, Y3 27 MHz, Y4 7.X MHz, Y5 7.X MHz

Commit message: Added two dual capacitor footprints to RFBitBanger
Parts:
- C26, C32: footprint Capacitors_THT:C_Disc_D5.0mm_W2.5mm_P5.00mm -> RFBitBanger:C_Disc_D5.0mm_W2.5mm_P5.00mm_Dual
Changed lines of the file:
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@@
       (effects (font (size 1.27 1.27)) (justify left))
     )
-    (property "Footprint" "Capacitors_THT:C_Disc_D5.0mm_W2.5mm_P5.00mm" (id 2) (at 213.36 132.08 0)
+    (property "Footprint" "RFBitBanger:C_Disc_D5.0mm_W2.5mm_P5.00mm_Dual" (id 2) (at 213.36 132.08 0)
       (effects (font (size 1.27 1.27)) hide)
     )
@@
       (effects (font (size 1.27 1.27)) (justify left))
     )
-    (property "Footprint" "Capacitors_THT:C_Disc_D5.0mm_W2.5mm_P5.00mm" (id 2) (at 262.89 66.04 0)
-      (effects (font (size 1.27 1.27)) hide)
-    )
+    (property "Footprint" "RFBitBanger:C_Disc_D5.0mm_W2.5mm_P5.00mm_Dual" (id 2) (at 262.89 66.04 0)
+      (effects (font (size 1.27 1.27)) hide)
+    )

Commit message: Fixed problems with manual, added filters
Parts:
- R38: value 33R -> 2R2
Changed lines of the file:
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@@
     (in_bom yes) (on_board yes)
     (property "Reference" "R38" (id 0) (at 248.92 43.18 90))
-    (property "Value" "33R" (id 1) (at 246.38 43.18 90))
+    (property "Value" "2R2" (id 1) (at 246.38 43.18 90))
     (property "Footprint" "Resistors_THT:R_Axial_DIN0207_L6.3mm_D2.5mm_P7.62mm_Horizontal" (id 2) (at 248.158 43.18 90)
       (effects (font (size 1.27 1.27)) hide)

Commit message: Added TCXO option to RFBitBanger SMT
Parts:
- Y3: value 27 MHz -> 25 MHz
Changed lines of the file:
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@@
     (in_bom yes) (on_board yes)
     (property "Reference" "Y3" (id 0) (at 106.68 53.34 0))
-    (property "Value" "27 MHz" (id 1) (at 100.33 46.99 90))
+    (property "Value" "25 MHz" (id 1) (at 100.33 46.99 90))
     (property "Footprint" "Crystals:Crystal_HC49-U_Vertical" (id 2) (at 102.87 53.34 0)
       (effects (font (size 1.27 1.27)) hide)
