File: PortableTerminal/PortableTerminal.kicad_pcb (KiCad board)
At the start: 2 copper layers, 64 x 75 mm, 54 parts, among them J1 Barrel_Jack, J10 RCAJack, J11 Conn_01x02, J2 Conn_01x01, J3 Conn_01x01, J4 ICSP, J5 Conn_01x01, J6 Conn_01x01, J7 Conn_01x04, J8 Conn_01x04, J9 RCAJack, P1 Mini-DIN_6pins_ver4, Q1 2N3904, SW1 SW_Push, U1 LM7805_TO220, U2 ATMEGA328P-PU, U3 LCD-016N002L, U4 MicroSD_SPI_CD, Y1 Crystal

Commit message: Added CW decode
Changed lines of the file:
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@@
   )
   (setup
-    (last_trace_width 0.35)
+    (last_trace_width 0.25)
     (user_trace_width 0.35)
     (user_trace_width 0.5)
@@
     (effects (font (size 1 1) (thickness 0.15)))
   )
-  (gr_text 1 (at 74 124) (layer F.SilkS)
+  (gr_text 1 (at 74.168 119.634) (layer F.SilkS)
     (effects (font (size 1 1) (thickness 0.15)))
   )
@@
   (gr_line (start 116 63) (end 116 138) (angle 90) (layer Edge.Cuts) (width 0.15))
   (gr_line (start 52 63) (end 116 63) (angle 90) (layer Edge.Cuts) (width 0.15))
-  (gr_text RESET (at 64.262 71.882) (layer F.SilkS)
+  (gr_text RESET (at 64.516 72.644) (layer F.SilkS)
     (effects (font (size 1 1) (thickness 0.15)))
   )
@@
   (segment (start 91.492 119.618) (end 91.77 119.34) (width 0.35) (layer F.Cu) (net 2))
   (segment (start 72.092 81.686) (end 72.086 81.68) (width 0.35) (layer B.Cu) (net 2) (status 30))
-  (segment (start 67.818 66.112) (end 68 66.112) (width 0.35) (layer B.Cu) (net 3) (status C00000))
-  (segment (start 68 66.112) (end 69.342 64.77) (width 0.35) (layer B.Cu) (net 3) (status 400000))
-  (segment (start 75.17 66.026) (end 75.17 66.9) (width 0.35) (layer B.Cu) (net 3) (status 800000))
+  (segment (start 67.818 66.112) (end 68 66.112) (width 0.35) (layer B.Cu) (net 3))
+  (segment (start 68 66.112) (end 69.342 64.77) (width 0.35) (layer B.Cu) (net 3))
+  (segment (start 75.17 66.026) (end 75.17 66.9) (width 0.35) (layer B.Cu) (net 3))
   (segment (start 73.914 64.77) (end 75.17 66.026) (width 0.35) (layer B.Cu) (net 3))
   (segment (start 69.342 64.77) (end 73.914 64.77) (width 0.35) (layer B.Cu) (net 3))
@@
   (segment (start 73.406 76.2) (end 76.708 79.502) (width 0.35) (layer B.Cu) (net 18))
   (segment (start 78.232 79.502) (end 78.486 79.756) (width 0.35) (layer B.Cu) (net 18))
-  (segment (start 62.34 111.42) (end 65.03 111.42) (width 0.35) (layer B.Cu) (net 19) (status 400000))
-  (segment (start 65.03 111.42) (end 66.03 110.42) (width 0.35) (layer B.Cu) (net 19) (status 800000))
+  (segment (start 62.34 111.42) (end 65.03 111.42) (width 0.35) (layer B.Cu) (net 19))
+  (segment (start 65.03 111.42) (end 66.03 110.42) (width 0.35) (layer B.Cu) (net 19))
   (segment (start 64.262 105.372) (end 65.99 107.1) (width 0.35) (layer B.Cu) (net 19))
   (segment (start 64.262 104.394) (end 64.262 105.372) (width 0.35) (layer B.Cu) (net 19))

Commit message: Completely remade board with common base input
Parts:
- added Q2: 2N3904, TO_SOT_Packages_THT:TO-92_Inline_Wide, F.Cu at (104.1, 88.9)
- added R21: 10k, Resistors_THT:R_Axial_DIN0207_L6.3mm_D2.5mm_P7.62mm_Horizontal, F.Cu at (95.5, 112.5)
- moved J4 3.17 mm to (98.5, 97.2)
- moved C7 2.74 mm to (96.2, 115.3)
- moved RV1 2.54 mm to (95.0, 85.9)
- moved R9 2.16 mm to (92.3, 107.0)
- moved JP1 1.82 mm to (95.5, 91.1)
Connections:
- U3 pad 16: GND -> Net-(Q2-Pad3)
Routing:
- net Net-(Q2-Pad3): track 0.00 -> 29.7 mm
- net Net-(Q2-Pad2): track 0.00 -> 27.7 mm, vias 0 -> 2
- net Net-(R21-Pad1): track 18.8 -> 29.3 mm, vias 0 -> 1
- net MOSI: track 53.5 -> 59.2 mm
- net +5V: track 278.3 -> 281.0 mm
- net SCK: track 22.7 -> 25.4 mm
- net RS: track 45.5 -> 43.4 mm
- net RESET: track 88.6 -> 90.7 mm, vias 1 -> 2
- net Net-(RV1-Pad2): track 37.9 -> 36.6 mm
- net DB4: track 36.2 -> 37.5 mm
- net MISO: track 77.2 -> 78.0 mm
- net DB5: track 34.9 -> 35.6 mm
Other:
- board text added: "PORTABLE SERIAL TERMINAL V2 BY DANIEL MARKS KW4TI CC-BY-SA 4.0"
- board text removed: "HD44780 DISPLAY"
- board text removed: "PORTABLE SERIAL TERMINAL BY DANIEL MARKS KW4TI CC-BY-SA 4.0"

Commit message: Added frequency counter and power measurement circuitry to PortableTerminal
Parts:
- added C10: 100 nF, Capacitors_THT:C_Disc_D5.0mm_W2.5mm_P2.50mm, F.Cu at (116.2, 117.1)
- added C11: 10 nF, Capacitors_THT:C_Disc_D5.0mm_W2.5mm_P2.50mm, F.Cu at (111.0, 106.0)
- added C9: 100 nF, Capacitors_THT:C_Disc_D5.0mm_W2.5mm_P2.50mm, F.Cu at (107.1, 129.5)
- added D5: 1N4148, Diodes_THT:D_DO-35_SOD27_P7.62mm_Horizontal, F.Cu at (109.8, 119.4)
- added D6: 1N4148, Diodes_THT:D_DO-35_SOD27_P7.62mm_Horizontal, F.Cu at (129.1, 116.9)
- added D7: 1N4148, Diodes_THT:D_DO-35_SOD27_P7.62mm_Horizontal, F.Cu at (106.9, 119.0)
- added J12: Conn_Coaxial, PortableTerminal:bnc_90_1-1337543-0_pad_combo, F.Cu at (116.3, 142.4)
- added R22: 100R, Resistors_THT:R_Axial_DIN0309_L9.0mm_D3.2mm_P12.70mm_Horizontal, F.Cu at (128.6, 125.9)
- added R23: 100R, Resistors_THT:R_Axial_DIN0309_L9.0mm_D3.2mm_P12.70mm_Horizontal, F.Cu at (128.5, 121.9)
- added R24: 10k, Resistors_THT:R_Axial_DIN0207_L6.3mm_D2.5mm_P7.62mm_Horizontal, F.Cu at (113.0, 108.9)
- added R25: 470R, Resistors_THT:R_Axial_DIN0207_L6.3mm_D2.5mm_P7.62mm_Horizontal, F.Cu at (75.2, 105.2)
- added R26: 470R, Resistors_THT:R_Axial_DIN0207_L6.3mm_D2.5mm_P7.62mm_Horizontal, F.Cu at (112.8, 119.4)
- added R27: 1k, Resistors_THT:R_Axial_DIN0207_L6.3mm_D2.5mm_P7.62mm_Horizontal, F.Cu at (109.7, 109.0)
- added R28: 100k, Resistors_THT:R_Axial_DIN0207_L6.3mm_D2.5mm_P7.62mm_Horizontal, F.Cu at (124.5, 86.7)
- added R29: 10k, Resistors_THT:R_Axial_DIN0207_L6.3mm_D2.5mm_P7.62mm_Horizontal, F.Cu at (114.3, 89.7)
- added U5: 74HC74, Housings_DIP:DIP-14_W7.62mm_Socket, F.Cu at (123.8, 113.7)
- moved R11 40.1 mm to (120.4, 78.9), turned to 270 degrees
- moved R14 37.1 mm to (106.8, 89.0), turned to 270 degrees
- moved R10 33.0 mm to (117.2, 86.5), turned to 90 degrees
- moved R15 26.2 mm to (110.0, 96.7), turned to 90 degrees
- moved R13 25.4 mm to (113.9, 78.9)
- moved R12 25.4 mm to (110.5, 86.5)
- moved R5 21.2 mm to (53.7, 117.7), turned to 0 degrees
- moved J5 15.0 mm to (128.0, 135.0)
- moved U3 15.0 mm to (128.0, 110.0)
- moved J2 15.0 mm to (128.0, 66.0)
- moved Q2 6.72 mm to (105.5, 82.3)
- moved R7 1.32 mm to (64.7, 116.9)
- moved R8 1.31 mm to (64.7, 113.7)
- moved J9 1.11 mm to (58.3, 110.3)
- moved R4 1.10 mm to (64.9, 107.4)
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Connections:
- J1 pad 3: Net-(J1-Pad3) -> (no net)
- P1 pad 2: Net-(P1-Pad2) -> (no net)
- P1 pad 6: Net-(P1-Pad6) -> (no net)
- U2 pad 21: Net-(U2-Pad21) -> (no net)
- U3 pad 10: Net-(U3-Pad10) -> (no net)
- U3 pad 7: Net-(U3-Pad7) -> (no net)
- U3 pad 8: Net-(U3-Pad8) -> (no net)
- U3 pad 9: Net-(U3-Pad9) -> (no net)
- U4 pad 9: Net-(U4-Pad9) -> (no net)
Routing:
- net +5V: track 281.0 -> 370.9 mm
- net Net-(R25-Pad2): track 0.00 -> 66.9 mm
- net RS: track 43.4 -> 80.1 mm
- net Net-(C9-Pad2): track 0.00 -> 30.2 mm
- net Net-(RV1-Pad2): track 36.6 -> 66.4 mm
- net Net-(D5-Pad1): track 0.00 -> 28.8 mm
- net Net-(C11-Pad1): track 0.00 -> 26.1 mm
- net E: track 48.8 -> 74.1 mm
- net DB4: track 37.5 -> 62.7 mm
- net Net-(R10-Pad1): track 36.8 -> 59.1 mm
- net Net-(R14-Pad1): track 24.5 -> 45.8 mm
- net MOSI: track 59.2 -> 78.5 mm
- net GND: track 4.77 -> 23.2 mm
- net Net-(Q2-Pad3): track 29.7 -> 46.2 mm
- net DB7: track 30.9 -> 47.3 mm
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Other:
- board size 64 x 75 mm -> 79 x 75 mm
- board text added: "74HC74"
- board text added: "FREQ CTR"
- board text added: "PORTABLE SERIAL TERMINAL V3 BY DANIEL MARKS KW4TI CC-BY-SA 4.0"
- board text removed: "PORTABLE SERIAL TERMINAL V2 BY DANIEL MARKS KW4TI CC-BY-SA 4.0"

Commit message: Added common mode choke to PortableTerminal
Parts:
- added C12: 100 nF, Capacitors_THT:C_Disc_D5.0mm_W2.5mm_P2.50mm, F.Cu at (83.1, 126.9)
- added C13: 100 nF, Capacitors_THT:C_Disc_D5.0mm_W2.5mm_P2.50mm, F.Cu at (80.0, 127.0)
- added T1: Common-Mode Choke, PortableTerminal:DoubleWindingTransformer, F.Cu at (70.6, 123.6)
- R27: value 1k -> 100R
- moved C1 9.16 mm to (78.5, 121.2), turned to 270 degrees
- moved C8 3.72 mm to (85.5, 122.3), turned to 180 degrees
- moved U1 2.94 mm to (79.6, 116.8)
- moved J1 1.95 mm to (68.6, 129.5)
- moved U4 1.58 mm to (96.3, 120.7)
Connections:
- J1 pad 1: +12V -> Net-(C12-Pad1)
- J1 pad 2: GND -> Net-(C12-Pad2)
- J11 pad 1: +12V -> Net-(C12-Pad1)
- J11 pad 2: GND -> Net-(C12-Pad2)
Routing:
- net Net-(C12-Pad2): track 0.00 -> 36.8 mm
- net Net-(C12-Pad1): track 0.00 -> 31.8 mm
- net GND: track 23.2 -> 31.6 mm
- net +5V: track 370.9 -> 364.7 mm
- net MISO: track 77.9 -> 80.1 mm
- net Net-(R10-Pad1): track 59.1 -> 57.5 mm
- net +12V: track 29.2 -> 27.8 mm
- net Net-(R12-Pad1): track 55.8 -> 54.4 mm
- net Net-(R25-Pad2): track 66.9 -> 65.7 mm
- net Net-(C7-Pad1): track 16.9 -> 15.8 mm
- net Net-(R14-Pad1): track 45.8 -> 44.7 mm
- net Net-(J10-Pad2): track 12.8 -> 12.2 mm

Commit message: Added README.md
Connections:
- U5 pad 13: +5V -> RS
Routing:
- net +5V: track 364.7 -> 338.2 mm
- net RS: track 80.1 -> 98.5 mm
Changed lines of the file:
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@@
     (links 163)
     (no_connects 0)
-    (area 51.924999 62.924999 131.075001 138.075001)
+    (area 50.252381 61.977 134.009524 143.685001)
     (thickness 1.6)
     (drawings 33)
-    (tracks 757)
+    (tracks 756)
     (zones 0)
     (modules 75)
@@
   )
   (setup
-    (last_trace_width 0.5)
+    (last_trace_width 0.35)
     (user_trace_width 0.35)
     (user_trace_width 0.5)
@@
       (net 47 "Net-(U5-Pad2)"))
     (pad 13 thru_hole oval (at 7.62 2.54 180) (size 1.6 1.6) (drill 0.8) (layers *.Cu *.Mask)
-      (net 5 +5V))
+      (net 33 RS))
     (pad 7 thru_hole oval (at 0 15.24 180) (size 1.6 1.6) (drill 0.8) (layers *.Cu *.Mask)
       (net 2 GND))
@@
   (segment (start 72.67 73.126) (end 72.136 73.66) (width 0.35) (layer B.Cu) (net 4))
   (segment (start 72.036 73.56) (end 72.136 73.66) (width 0.35) (layer B.Cu) (net 4) (status 30))
+  (segment (start 88.297118 125.822589) (end 99.657411 125.822589) (width 0.5) (layer B.Cu) (net 5))
+  (segment (start 100.3 125.18) (end 100.3 125.2) (width 0.5) (layer B.Cu) (net 5))
+  (segment (start 99.657411 125.822589) (end 100.3 125.18) (width 0.5) (layer B.Cu) (net 5))
+  (segment (start 103.5 121.54) (end 113.49 121.54) (width 0.5) (layer B.Cu) (net 5))
+  (segment (start 125.71 120.28) (end 129.05 116.94) (width 0.5) (layer B.Cu) (net 5))
+  (segment (start 114.75 120.28) (end 125.71 120.28) (width 0.5) (layer B.Cu) (net 5))
+  (segment (start 113.49 121.54) (end 114.75 120.28) (width 0.5) (layer B.Cu) (net 5))
+  (segment (start 123.77 106.04) (end 122.56 106.04) (width 0.5) (layer B.Cu) (net 5))
+  (segment (start 122.66 113.66) (end 123.77 113.66) (width 0.5) (layer B.Cu) (net 5))
+  (segment (start 121.85 112.85) (end 122.66 113.66) (width 0.5) (layer B.Cu) (net 5))
+  (segment (start 121.85 106.75) (end 121.85 112.85) (width 0.5) (layer B.Cu) (net 5))
+  (segment (start 122.56 106.04) (end 121.85 106.75) (width 0.5) (layer B.Cu) (net 5))
+  (segment (start 114.79 114.75) (end 116.15 113.66) (width 0.5) (layer B.Cu) (net 5))
+  (segment (start 105.98 114.75) (end 114.79 114.75) (width 0.5) (layer B.Cu) (net 5))
+  (segment (start 103.5 117.5) (end 105.98 114.75) (width 0.5) (layer B.Cu) (net 5))
+  (segment (start 103.5 122) (end 103.5 121.54) (width 0.5) (layer B.Cu) (net 5))
+  (segment (start 103.5 121.54) (end 103.5 117.5) (width 0.5) (layer B.Cu) (net 5))
+  (segment (start 100.3 125.2) (end 103.5 122) (width 0.5) (layer B.Cu) (net 5))
   (segment (start 84.68 116.85) (end 85.09 116.85) (width 0.5) (layer B.Cu) (net 5))
   (segment (start 85.09 116.85) (end 85.52 117.28) (width 0.5) (layer B.Cu) (net 5))
   (segment (start 85.52 117.28) (end 85.52 122.35) (width 0.5) (layer B.Cu) (net 5))
   (segment (start 85.52 122.35) (end 85.52 123.03) (width 0.5) (layer B.Cu) (net 5) (status 30))
-  (segment (start 85.52 123.03) (end 89.11 126.64) (width 0.5) (layer B.Cu) (net 5) (status 10))
-  (segment (start 93.95 135.48) (end 95.67 137.2) (width 0.5) (layer B.Cu) (net 5))
-  (segment (start 93.95 129.04) (end 93.95 135.48) (width 0.5) (layer B.Cu) (net 5))
-  (segment (start 91.55 126.64) (end 93.95 129.04) (width 0.5) (layer B.Cu) (net 5))
-  (segment (start 89.11 126.64) (end 91.55 126.64) (width 0.5) (layer B.Cu) (net 5))
+  (segment (start 85.52 123.03) (end 88.297118 125.822589) (width 0.5) (layer B.Cu) (net 5) (status 10))
   (segment (start 69.719 118.741) (end 69.901 118.741) (width 0.5) (layer B.Cu) (net 5))
   (segment (start 83.58 114.92) (end 84.68 116.02) (width 0.5) (layer B.Cu) (net 5))
@@
   (segment (start 62.732 103.13) (end 62.738 103.124) (width 0.35) (layer B.Cu) (net 5))
   (segment (start 116.15 103.5) (end 116.84 103.5) (width 0.35) (layer B.Cu) (net 5))
-  (segment (start 116.84 103.5) (end 117.68 102.66) (width 0.35) (layer B.Cu) (net 5))
-  (segment (start 125.43 105.59) (end 124.98 106.04) (width 0.35) (layer B.Cu) (net 5))
-  (segment (start 125.43 97.22) (end 125.43 105.59) (width 0.35) (layer B.Cu) (net 5))
-  (segment (start 124.74 96.53) (end 125.43 97.22) (width 0.35) (layer B.Cu) (net 5))
-  (segment (start 115.08 96.53) (end 124.74 96.53) (width 0.35) (layer B.Cu) (net 5))
-  (segment (start 114.59 97.02) (end 115.08 96.53) (width 0.35) (layer B.Cu) (net 5))
-  (segment (start 114.59 98.97) (end 114.59 97.02) (width 0.35) (layer B.Cu) (net 5))
-  (segment (start 115.29 99.67) (end 114.59 98.97) (width 0.35) (layer B.Cu) (net 5))
-  (segment (start 117 99.67) (end 115.29 99.67) (width 0.35) (layer B.Cu) (net 5))
-  (segment (start 117.68 100.35) (end 117 99.67) (width 0.35) (layer B.Cu) (net 5))
-  (segment (start 117.68 102.66) (end 117.68 100.35) (width 0.35) (layer B.Cu) (net 5))
   (segment (start 116.15 113.66) (end 115.14 113.66) (width 0.5) (layer B.Cu) (net 5))
-  (segment (start 115.14 113.66) (end 114.39 112.91) (width 0.5) (layer B.Cu) (net 5))
-  (segment (start 114.39 112.91) (end 114.39 105.26) (width 0.5) (layer B.Cu) (net 5))
   (segment (start 114.39 105.26) (end 116.15 103.5) (width 0.5) (layer B.Cu) (net 5))
+  (segment (start 114.39 112.91) (end 114.39 105.26) (width 0.5) (layer B.Cu) (net 5))
+  (segment (start 115.14 113.66) (end 114.39 112.91) (width 0.5) (layer B.Cu) (net 5))
   (segment (start 116.15 113.66) (end 116.15 116.98) (width 0.5) (layer B.Cu) (net 5))
   (segment (start 116.15 116.98) (end 116.25 117.08) (width 0.5) (layer B.Cu) (net 5))
@@
   (segment (start 123.77 113.66) (end 116.15 113.66) (width 0.5) (layer B.Cu) (net 5))
   (segment (start 115.97 116.8) (end 116.25 117.08) (width 0.5) (layer B.Cu) (net 5) (status 30))
-  (segment (start 116.15 111.12) (end 116.15 113.66) (width 0.5) (layer B.Cu) (net 5))
-  (segment (start 120.36 137.2) (end 123.03 137.2) (width 0.5) (layer B.Cu) (net 5))
-  (segment (start 124.47 132.71) (end 124.43 132.71) (width 0.5) (layer B.Cu) (net 5))
-  (segment (start 124.47 135.76) (end 124.47 132.71) (width 0.5) (layer B.Cu) (net 5))
-  (segment (start 123.03 137.2) (end 124.47 135.76) (width 0.5) (layer B.Cu) (net 5))
   (segment (start 129.93 107.46) (end 128 107.46) (width 0.5) (layer B.Cu) (net 5))
   (segment (start 130.34 107.87) (end 129.93 107.46) (width 0.5) (layer B.Cu) (net 5))
-  (segment (start 130.34 127.59) (end 130.34 116.76) (width 0.5) (layer B.Cu) (net 5))
   (segment (start 130.34 116.76) (end 130.34 107.87) (width 0.5) (layer B.Cu) (net 5))
-  (segment (start 128.35 129.58) (end 130.34 127.59) (width 0.5) (layer B.Cu) (net 5))
-  (segment (start 126.11 129.58) (end 128.35 129.58) (width 0.5) (layer B.Cu) (net 5))
-  (segment (start 124.43 131.26) (end 126.11 129.58) (width 0.5) (layer B.Cu) (net 5))
-  (segment (start 124.43 132.71) (end 124.43 131.26) (width 0.5) (layer B.Cu) (net 5))
-  (segment (start 95.67 137.2) (end 120.36 137.2) (width 0.5) (layer B.Cu) (net 5))
   (segment (start 89.34 94.98) (end 89.34 93.37) (width 0.5) (layer B.Cu) (net 5))
   (segment (start 91.57 91.14) (end 95.48 91.14) (width 0.5) (layer B.Cu) (net 5))
@@
   (segment (start 96.25 75.996) (end 100.13 75.996) (width 0.35) (layer B.Cu) (net 32))
   (segment (start 87.664 84.836) (end 96.25 75.996) (width 0.35) (layer B.Cu) (net 32))
+  (segment (start 116.15 111.12) (end 118.35 111.12) (width 0.35) (layer B.Cu) (net 33))
+  (segment (start 122.53 102.22) (end 127.84 102.22) (width 0.35) (layer B.Cu) (net 33))
+  (segment (start 120.84 103.91) (end 122.53 102.22) (width 0.35) (layer B.Cu) (net 33))
+  (segment (start 120.84 108.63) (end 120.84 103.91) (width 0.35) (layer B.Cu) (net 33))
+  (segment (start 118.35 111.12) (end 120.84 108.63) (width 0.35) (layer B.Cu) (net 33))
+  (segment (start 127.84 102.22) (end 128 102.38) (width 0.35) (layer B.Cu) (net 33))
   (segment (start 124.26 92.68) (end 125.2 92.68) (width 0.35) (layer B.Cu) (net 33))
   (segment (start 126.47 100.85) (end 128 102.38) (width 0.35) (layer B.Cu) (net 33))
@@
   (segment (start 118.3 99.29) (end 118.3 107.78) (width 0.35) (layer B.Cu) (net 46))
   (segment (start 117.43 98.42) (end 118.3 99.29) (width 0.35) (layer B.Cu) (net 46))
+  (segment (start 123.77 100.96) (end 124.45 100.96) (width 0.35) (layer F.Cu) (net 47))
+  (segment (start 124.45 100.96) (end 125.31 101.82) (width 0.35) (layer F.Cu) (net 47))
+  (segment (start 124.69 111.12) (end 123.77 111.12) (width 0.35) (layer F.Cu) (net 47))
+  (segment (start 125.31 110.5) (end 124.69 111.12) (width 0.35) (layer F.Cu) (net 47))
+  (segment (start 125.31 101.82) (end 125.31 110.5) (width 0.35) (layer F.Cu) (net 47))
   (segment (start 123.77 100.96) (end 123.77 101.17) (width 0.35) (layer B.Cu) (net 47))
-  (segment (start 123.77 101.17) (end 122.07 102.87) (width 0.35) (layer B.Cu) (net 47))
-  (segment (start 122.07 102.87) (end 122.07 110.49) (width 0.35) (layer B.Cu) (net 47))
-  (segment (start 122.07 110.49) (end 122.7 111.12) (width 0.35) (layer B.Cu) (net 47))
-  (segment (start 122.7 111.12) (end 123.77 111.12) (width 0.35) (layer B.Cu) (net 47))
   (segment (start 123.77 103.5) (end 121.9 103.5) (width 0.35) (layer F.Cu) (net 48))
   (segment (start 119.36 106.04) (end 116.15 106.04) (width 0.35) (layer F.Cu) (net 48))

Commit message: Lots of changes...
Parts:
- added JP3: Load, Pin_Headers:Pin_Header_Straight_1x02_Pitch2.54mm, F.Cu at (128.6, 127.9)
- moved J2 73.0 mm to (55.0, 66.0)
- moved J6 73.0 mm to (128.0, 135.0)
- moved J3 69.0 mm to (55.0, 135.0)
- moved J5 69.0 mm to (128.0, 66.0)
- moved R22 12.2 mm to (116.5, 124.2), turned to 0 degrees
- moved R23 12.1 mm to (116.5, 120.3), turned to 0 degrees
- moved D6 0.51 mm to (129.5, 116.7)
- moved C10 0.48 mm to (116.7, 116.9)
- moved R24 0.30 mm to (112.7, 109.0)
- moved R27 0.22 mm to (109.5, 109.0)
Connections:
- R22 pad 2: Net-(C9-Pad2) -> Net-(JP3-Pad1)
- R23 pad 2: Net-(C9-Pad2) -> Net-(JP3-Pad1)
Routing:
- net Net-(JP3-Pad1): track 0.00 -> 7.85 mm
- net Net-(D5-Pad1): track 28.8 -> 29.9 mm
- net +5V: track 338.2 -> 339.0 mm
- net Net-(U5-Pad2): track 12.6 -> 13.4 mm

Commit message: Implemented timers, fixed beep audio, fixed key shaping
Connections:
- P1 pad 7: Net-(P1-Pad7) -> GND
Routing:
- net Net-(P1-Pad7): track 14.4 -> 0.00 mm
- net GND: track 31.6 -> 45.9 mm
