File: PortableTerminal/PortableTerminal.kicad_pcb (KiCad board)
At the start: 2 copper layers, 79 x 75 mm, 76 parts, among them J1 Barrel_Jack, J10 RCAJack, J11 Conn_01x02, J12 Conn_Coaxial, J2 Conn_01x01, J3 Conn_01x01, J4 ICSP, J5 Conn_01x01, J6 Conn_01x01, J7 Conn_01x04, J8 Conn_01x04, J9 RCAJack, P1 Mini-DIN_6pins_ver4, Q1 2N3904, Q2 2N3904, SW1 SW_Push, T1 Common-Mode Choke, U1 LM7805_TO220, U2 ATMEGA328P-PU, U3 LCD-016N002L, U4 MicroSD_SPI_CD, U5 74HC74, Y1 Crystal

Commit message: Converted all Kicad projects to version 6.0.10
Connections:
- J1 pad 3: (no net) -> unconnected-(J1-Pad3)
- P1 pad 2: (no net) -> unconnected-(P1-Pad2)
- P1 pad 6: (no net) -> unconnected-(P1-Pad6)
- U2 pad 21: (no net) -> unconnected-(U2-Pad21)
- U3 pad 10: (no net) -> unconnected-(U3-Pad10)
- U3 pad 7: (no net) -> unconnected-(U3-Pad7)
- U3 pad 8: (no net) -> unconnected-(U3-Pad8)
- U3 pad 9: (no net) -> unconnected-(U3-Pad9)
- U4 pad 9: (no net) -> unconnected-(U4-Pad9)
Routing:
- net RS: track 98.5 -> 92.2 mm
- net +5V: track 339.0 -> 336.4 mm
- net GND: track 45.9 -> 43.7 mm
- net MOSI: track 78.5 -> 76.8 mm
- net Net-(R9-Pad2): track 15.8 -> 14.2 mm
- net Net-(R8-Pad2): track 11.9 -> 10.6 mm
- net +12V: track 27.8 -> 26.5 mm
- net Net-(U4-Pad2): track 44.7 -> 43.6 mm
- net RESET: track 90.7 -> 89.6 mm
- net Net-(J11-Pad1): track 31.8 -> 30.8 mm
- net Net-(RV1-Pad2): track 66.4 -> 65.3 mm
- net Net-(J4-Pad2): track 8.78 -> 8.02 mm
- net DB7: track 47.3 -> 46.6 mm
- net Net-(R6-Pad2): track 23.9 -> 23.2 mm
- net TX: track 8.53 -> 7.82 mm
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Other:
- net class Default removed
