File: BitBangDisplay/BitBangDisplayRadio.sch (KiCad schematic (older format))
At the start: 145 parts, among them J12 Conn_Coaxial, J17 Filt1, J18 Filt2, Q1 2N3904, Q10 2N3904, Q11 2N3904, Q12 2N3904, Q13 2N2907, Q15 NC, Q2 2N3904, Q3 2N7000, Q5 NC, Q6 2N7000, Q7 2N7000, Q8 2N2907, Q9 2N7000, T1 Trifilar, T2 Trifilar, T3 Current, U4 LM358, U6 SI5351A, Y2 7.X MHz, Y3 27 MHz, Y4 7.X MHz, Y5 7.X MHz

Commit message: Added Display Board on Top
Parts:
- D15, D18, D8: value 1N4148 -> 1N4007; footprint Diodes_THT:D_DO-35_SOD27_P7.62mm_Horizontal -> Diodes_THT:D_DO-41_SOD81_P7.62mm_Horizontal
- J12: footprint RFBitBanger:bnc_90_1-1337543-0_pad_combo -> BitBangDisplay:bnc_90_1-1337543-0_pad_combo
- L4, L6, L7, L8: footprint RFBitBanger:SmallVerticalToroid -> BitBangDisplay:SmallVerticalToroid
- RLY1: footprint RFBitBanger:G2VRelay -> BitBangDisplay:G2VRelay
- RV2: footprint RFBitBanger:Potentiometer_Big_Small_Combined -> Potentiometers:Potentiometer_WirePads
- T1, T2: footprint RFBitBanger:TripleWindingTransformerRef -> BitBangDisplay:TripleWindingTransformerRef
- T3: footprint RFBitBanger:SamplingTransformer -> BitBangDisplay:SamplingTransformer
Connections:
- wire segments 309 -> 310
