File: BitBangDisplay/BitBangDisplay.sch (KiCad schematic (older format))
At the start: 72 parts, among them J1 Conn_01x04, J10 Conn_01x04, J11 Conn_01x01, J12 Conn_01x01, J13 KeyerJack, J14 KeyerJack, J15 KeyerJack, J19 Conn_01x04, J2 Audio-Jack-3, J20 Conn_01x01, J21 Conn_01x01, J22 SPEAKER, J3 Conn_01x01, J4 Conn_01x01, J5 Conn_01x01, J6 Conn_01x01, J7 Conn_01x01, J8 Conn_01x01, J9 Conn_01x01, SW2 SW_Push, SW3 SW_Push, SW4 SW_Push, SW5 SW_Push, U1 LCD-016N002L, U2 LM358, U5 LCD-016N002L

Commit message: Before trying to put everything onto a single line
Parts:
- removed J2: Audio-Jack-3, BitBangDisplay:PJ-3240-35mm-stereo, symbol Audio-Jack-3
- added J16: SPEAKER, Connectors_Terminal_Blocks:TerminalBlock_bornier-2_P5.08mm, symbol Conn_01x02
- added J2: Audio-Jack-3_2Switches, BitBangDisplay:PJ-3240-35mm-stereo, symbol Audio-Jack-3_2Switches
Connections:
- net at C1.1, J22.1 (Pin_1): now also J2.1, J2.2
- net at C1.2, J22.2 (Pin_2): now also J16.2 (Pin_2), J2.3
- new net: J16.1 (Pin_1), J2.4
Other:
- moved on the sheet: C1, J22
Changed lines of the file:
@@
 L Conn_01x02 J22
 U 1 1 61E72EDE
-P 6000 900
-F 0 "J22" H 6000 1000 50  0000 C CNN
-F 1 "SPEAKER" H 6000 700 50  0000 C CNN
-F 2 "Pin_Headers:Pin_Header_Straight_1x02_Pitch2.54mm" H 6000 900 50  0001 C CNN
-F 3 "" H 6000 900 50  0001 C CNN
-	1    6000 900
+P 4550 1200
+F 0 "J22" H 4550 1300 50  0000 C CNN
+F 1 "SPEAKER" H 4550 1000 50  0000 C CNN
+F 2 "Pin_Headers:Pin_Header_Straight_1x02_Pitch2.54mm" H 4550 1200 50  0001 C CNN
+F 3 "" H 4550 1200 50  0001 C CNN
+	1    4550 1200
 	1    0    0    -1
 $EndComp
@@
 RW
 $Comp
-L Audio-Jack-3 J2
-U 1 1 61E88BBE
-P 5100 1000
-F 0 "J2" H 5050 1175 50  0000 C CNN
-F 1 "Audio-Jack-3" H 5200 930 50  0000 C CNN
-F 2 "BitBangDisplay:PJ-3240-35mm-stereo" H 5350 1100 50  0001 C CNN
-F 3 "" H 5350 1100 50  0001 C CNN
-	1    5100 1000
-	1    0    0    -1
-$EndComp
-$Comp
 L Conn_01x01 J4
 U 1 1 61E88E38
@@
 L C_Small C1
 U 1 1 61E8A31F
-P 5550 1150
-F 0 "C1" H 5560 1220 50  0000 L CNN
-F 1 "10 nF" H 5560 1070 50  0000 L CNN
-F 2 "Capacitors_THT:C_Disc_D5.0mm_W2.5mm_P2.50mm" H 5550 1150 50  0001 C CNN
-F 3 "" H 5550 1150 50  0001 C CNN
-	1    5550 1150
-	1    0    0    -1
+P 3700 1600
+F 0 "C1" H 3710 1670 50  0000 L CNN
+F 1 "10 nF" H 3710 1520 50  0000 L CNN
+F 2 "Capacitors_THT:C_Disc_D5.0mm_W2.5mm_P2.50mm" H 3700 1600 50  0001 C CNN
+F 3 "" H 3700 1600 50  0001 C CNN
+	1    3700 1600
+	0    1    1    0
 $EndComp
 $Comp
@@
 	2800 4000 2650 4000
 Wire Wire Line
-	5800 1300 5800 1000
-Wire Wire Line
-	4900 1100 4900 1300
-Wire Wire Line
-	5300 1000 5600 1000
-Wire Wire Line
-	5600 1000 5600 900
-Wire Wire Line
-	5600 900  5800 900
-Wire Wire Line
 	6950 2250 6950 2200
 Wire Wire Line
@@
 Wire Wire Line
 	6950 2000 7150 2000
-Wire Wire Line
-	4900 1300 5800 1300
-Wire Wire Line
-	5550 1050 5550 1000
-Connection ~ 5550 1000
-Wire Wire Line
-	5550 1250 5550 1300
-Connection ~ 5550 1300
 Wire Wire Line
 	4900 2100 4900 2550
@@
 Connection ~ 7700 3450
 Wire Wire Line
-	8450 3450 8450 3050
-Wire Wire Line
-	8200 3450 8450 3450
+	8450 3050 8450 3450
+Wire Wire Line
+	8450 3450 8200 3450
 $Comp
 L C_Small C12
@@
 Wire Wire Line
 	4250 3350 4350 3350
+$Comp
+L Audio-Jack-3_2Switches J2
+U 1 1 61E9A48E
+P 3550 1200
+F 0 "J2" H 3550 1490 50  0000 C CNN
+F 1 "Audio-Jack-3_2Switches" H 3400 1000 50  0000 L CNN
+F 2 "BitBangDisplay:PJ-3240-35mm-stereo" H 3800 1300 50  0001 C CNN
+F 3 "" H 3800 1300 50  0001 C CNN
+	1    3550 1200
+	1    0    0    -1
+$EndComp
+Wire Wire Line
+	3350 1400 3350 1950
+Wire Wire Line
+	3350 1600 3600 1600
+Wire Wire Line
+	3750 1200 4350 1200
+Wire Wire Line
+	3900 1100 3900 1600
+Wire Wire Line
+	3900 1600 3800 1600
+Connection ~ 3900 1200
+Wire Wire Line
+	4350 1300 4350 1950
+Wire Wire Line
+	4350 1950 3350 1950
+Connection ~ 3350 1600
+$Comp
+L Conn_01x02 J16
+U 1 1 61E9B47A
+P 4550 700
+F 0 "J16" H 4550 800 50  0000 C CNN
+F 1 "SPEAKER" H 4550 500 50  0000 C CNN
+F 2 "Connectors_Terminal_Blocks:TerminalBlock_bornier-2_P5.08mm" H 4550 700 50  0001 C CNN
+F 3 "" H 4550 700 50  0001 C CNN
+	1    4550 700
+	1    0    0    -1
+$EndComp
+Wire Wire Line
+	3750 1300 3850 1300
+Wire Wire Line
+	3850 1300 3850 700
+Wire Wire Line
+	3850 700  4350 700
+Wire Wire Line
+	4350 800  4100 800
+Wire Wire Line
+	4100 800  4100 1300
+Wire Wire Line
+	4100 1300 4350 1300
+Wire Wire Line
+	3900 1100 3750 1100
 $EndSCHEMATC

Commit message: Changed external connector for single 20 pin or ribbon cable
Parts:
- removed J10, J19: Conn_01x04, Pin_Headers:Pin_Header_Straight_1x04_Pitch2.54mm, symbol Conn_01x04
- removed J22: SPEAKER, Pin_Headers:Pin_Header_Straight_1x02_Pitch2.54mm, symbol Conn_01x02
- removed U1, U5: LCD-016N002L, Pin_Headers:Pin_Header_Straight_1x16_Pitch2.54mm, symbol LCD-016N002L
- added C13: 100 nF, Capacitors_THT:C_Disc_D5.0mm_W2.5mm_P2.50mm, symbol C_Small
- added L4: 100 uH, Inductors_THT:L_Axial_L6.6mm_D2.7mm_P10.16mm_Horizontal_Vishay_IM-2, symbol L_Small
- added R22: 47R, Resistors_THT:R_Axial_DIN0207_L6.3mm_D2.5mm_P7.62mm_Horizontal, symbol R
- added U1: LCD1602ExtraPins, Pin_Headers:Pin_Header_Straight_1x16_Pitch2.54mm, symbol LCD1602ExtraPins
- added U5: LCD1602ExtraPins, Pin_Headers:Pin_Header_Straight_1x20_Pitch2.54mm, symbol LCD1602ExtraPins
Connections:
- net +5VP is gone; now on net +5V: C7.1, R11.1, R4.1, R5.2, U2.8 (V+)
- net +5V: now also C13.1, U1.2 (VDD), U5.2 (VDD)
- net AVEE: now also U1.15 (A/VEE), U5.15 (A/VEE)
- net DB4: now also U1.11 (DB4), U5.11 (DB4)
- net DB5: now also U1.12 (DB5), U5.12 (DB5)
- net DB6: now also U1.13 (DB6), U5.13 (DB6)
- net DB7: now also U1.14 (DB7), U5.14 (DB7)
- net E: now also U1.6 (E), U5.6 (E)
- net GND: now also C1.2, J16.2 (Pin_2), J2.3, C13.2, U1.1 (VSS), U5.1 (VSS), U5.17
- net K: now also U1.16 (K), U5.16 (K)
- net RS: now also U1.4 (RS), U5.4 (RS)
- net RW: now also U1.5 (R/~W), U5.5 (R/~W)
- net VO: now also U1.3 (VO), U5.3 (VO)
- net PTT: now reaches R1.1, R4.2
- net PTT: now also U5.19
- net MIC: now reaches R2.1, R20.2
- net MIC: now also U5.18
- net at C1.1, J2.1, J2.2: now also L4.1, R22.1
- new net SPKR: L4.2, R22.2, U5.20

Commit message: Added fifth button
Parts:
- added C14: 100 nF, Capacitors_THT:C_Disc_D5.0mm_W2.5mm_P2.50mm, symbol C_Small
- added R23: 10k, Resistors_THT:R_Axial_DIN0207_L6.3mm_D2.5mm_P7.62mm_Horizontal, symbol R
- added R24: 1k, Resistors_THT:R_Axial_DIN0207_L6.3mm_D2.5mm_P7.62mm_Horizontal, symbol R
- added SW1: SW_Push, Buttons_Switches_THT:SW_PUSH_6mm, symbol SW_Push
Connections:
- net +5V: now also R24.2
- net GND: now also C14.1, SW1.2
- net RS: now also R23.2
- new net: C14.2, R23.1, R24.1, SW1.1
Other:
- moved on the sheet: C10, C11, C16, C17, R12, R13, R29, R3, R33, R46, R47, R6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

Commit message: Added extra row of ground pins for 40 pin connector
Parts:
- added J10: Conn_01x20, Pin_Headers:Pin_Header_Straight_1x20_Pitch2.54mm, symbol Conn_01x20
Connections:
- net GND: now also J10.1 (Pin_1), J10.10 (Pin_10), J10.11 (Pin_11), J10.12 (Pin_12), J10.13 (Pin_13), J10.14 (Pin_14), J10.15 (Pin_15), J10.16 (Pin_16), J10.17 (Pin_17), J10.18 (Pin_18), J10.19 (Pin_19), J10.2 (Pin_2), J10.20 (Pin_20), J10.3 (Pin_3), J10.4 (Pin_4), J10.5 (Pin_5), J10.6 (Pin_6), J10.7 (Pin_7), J10.8 (Pin_8), J10.9 (Pin_9)
Changed lines of the file:
@@
 $EndComp
 $Comp
-L GND #PWR8
+L GND #PWR01
 U 1 1 615D1E98
 P 3950 6300
-F 0 "#PWR8" H 3950 6050 50  0001 C CNN
+F 0 "#PWR01" H 3950 6050 50  0001 C CNN
 F 1 "GND" H 3950 6150 50  0000 C CNN
 F 2 "" H 3950 6300 50  0001 C CNN
@@
 $EndComp
 $Comp
-L GND #PWR5
+L GND #PWR02
 U 1 1 615D2C34
 P 3500 6300
-F 0 "#PWR5" H 3500 6050 50  0001 C CNN
+F 0 "#PWR02" H 3500 6050 50  0001 C CNN
 F 1 "GND" H 3500 6150 50  0000 C CNN
 F 2 "" H 3500 6300 50  0001 C CNN
@@
 $EndComp
 $Comp
-L GND #PWR16
+L GND #PWR03
 U 1 1 615D3831
 P 5150 6300
-F 0 "#PWR16" H 5150 6050 50  0001 C CNN
+F 0 "#PWR03" H 5150 6050 50  0001 C CNN
 F 1 "GND" H 5150 6150 50  0000 C CNN
 F 2 "" H 5150 6300 50  0001 C CNN
@@
 $EndComp
 $Comp
-L GND #PWR13
+L GND #PWR04
 U 1 1 615D3842
 P 4700 6300
-F 0 "#PWR13" H 4700 6050 50  0001 C CNN
+F 0 "#PWR04" H 4700 6050 50  0001 C CNN
 F 1 "GND" H 4700 6150 50  0000 C CNN
 F 2 "" H 4700 6300 50  0001 C CNN
@@
 $EndComp
 $Comp
-L GND #PWR17
+L GND #PWR05
 U 1 1 615D3B9E
 P 5150 7200
-F 0 "#PWR17" H 5150 6950 50  0001 C CNN
+F 0 "#PWR05" H 5150 6950 50  0001 C CNN
 F 1 "GND" H 5150 7050 50  0000 C CNN
 F 2 "" H 5150 7200 50  0001 C CNN
@@
 $EndComp
 $Comp
-L GND #PWR14
+L GND #PWR06
 U 1 1 615D3BAF
 P 4700 7250
-F 0 "#PWR14" H 4700 7000 50  0001 C CNN
+F 0 "#PWR06" H 4700 7000 50  0001 C CNN
 F 1 "GND" H 4700 7100 50  0000 C CNN
 F 2 "" H 4700 7250 50  0001 C CNN
@@
 $EndComp
 $Comp
-L GND #PWR9
+L GND #PWR07
 U 1 1 615E0B59
 P 3950 7150
-F 0 "#PWR9" H 3950 6900 50  0001 C CNN
+F 0 "#PWR07" H 3950 6900 50  0001 C CNN
 F 1 "GND" H 3950 7000 50  0000 C CNN
 F 2 "" H 3950 7150 50  0001 C CNN
@@
 $EndComp
 $Comp
-L GND #PWR6
+L GND #PWR08
 U 1 1 615E0B65
 P 3500 7200
-F 0 "#PWR6" H 3500 6950 50  0001 C CNN
+F 0 "#PWR08" H 3500 6950 50  0001 C CNN
 F 1 "GND" H 3500 7050 50  0000 C CNN
 F 2 "" H 3500 7200 50  0001 C CNN
@@
 $EndComp
 $Comp
-L GND #PWR2
+L GND #PWR09
 U 1 1 6163A158
 P 1600 7300
-F 0 "#PWR2" H 1600 7050 50  0001 C CNN
+F 0 "#PWR09" H 1600 7050 50  0001 C CNN
 F 1 "GND" H 1600 7150 50  0000 C CNN
 F 2 "" H 1600 7300 50  0001 C CNN
@@
 $EndComp
 $Comp
-L +5V #PWR1
+L +5V #PWR010
 U 1 1 6163A550
 P 1600 5650
-F 0 "#PWR1" H 1600 5500 50  0001 C CNN
+F 0 "#PWR010" H 1600 5500 50  0001 C CNN
 F 1 "+5V" H 1600 5790 50  0000 C CNN
 F 2 "" H 1600 5650 50  0001 C CNN
@@
 DB4
 $Comp
-L +5V #PWR11
+L +5V #PWR011
 U 1 1 61649A09
 P 4350 5650
-F 0 "#PWR11" H 4350 5500 50  0001 C CNN
+F 0 "#PWR011" H 4350 5500 50  0001 C CNN
 F 1 "+5V" H 4350 5790 50  0000 C CNN
 F 2 "" H 4350 5650 50  0001 C CNN
@@
 RS
 $Comp
-L GND #PWR26
+L GND #PWR012
 U 1 1 61C9A041
 P 10500 6150
-F 0 "#PWR26" H 10500 5900 50  0001 C CNN
+F 0 "#PWR012" H 10500 5900 50  0001 C CNN
 F 1 "GND" H 10500 6000 50  0000 C CNN
 F 2 "" H 10500 6150 50  0001 C CNN
@@
 RW
 $Comp
-L GND #PWR4
+L GND #PWR013
 U 1 1 61E7CC06
 P 1700 2600
-F 0 "#PWR4" H 1700 2350 50  0001 C CNN
+F 0 "#PWR013" H 1700 2350 50  0001 C CNN
 F 1 "GND" H 1700 2450 50  0000 C CNN
 F 2 "" H 1700 2600 50  0001 C CNN
@@
 $EndComp
 $Comp
-L +5V #PWR3
+L +5V #PWR014
 U 1 1 61E7CC0C
 P 1700 950
-F 0 "#PWR3" H 1700 800 50  0001 C CNN
+F 0 "#PWR014" H 1700 800 50  0001 C CNN
 F 1 "+5V" H 1700 1090 50  0000 C CNN
 F 2 "" H 1700 950 50  0001 C CNN
@@
 $EndComp
 $Comp
-L GND #PWR15
+L GND #PWR015
 U 1 1 61E8AAB8
 P 4900 2550
-F 0 "#PWR15" H 4900 2300 50  0001 C CNN
+F 0 "#PWR015" H 4900 2300 50  0001 C CNN
 F 1 "GND" H 4900 2400 50  0000 C CNN
 F 2 "" H 4900 2550 50  0001 C CNN
@@
 $EndComp
 $Comp
-L GND #PWR7
+L GND #PWR016
 U 1 1 61E8F430
 P 3850 3600
-F 0 "#PWR7" H 3850 3350 50  0001 C CNN
+F 0 "#PWR016" H 3850 3350 50  0001 C CNN
 F 1 "GND" H 3850 3450 50  0000 C CNN
 F 2 "" H 3850 3600 50  0001 C CNN
@@
 $EndComp
 $Comp
-L GND #PWR22
+L GND #PWR017
 U 1 1 61E904B7
 P 6600 3650
-F 0 "#PWR22" H 6600 3400 50  0001 C CNN
+F 0 "#PWR017" H 6600 3400 50  0001 C CNN
 F 1 "GND" H 6600 3500 50  0000 C CNN
 F 2 "" H 6600 3650 50  0001 C CNN
@@
 $EndComp
 $Comp
-L GND #PWR19
+L GND #PWR018
 U 1 1 61E90B59
 P 5900 2900
-F 0 "#PWR19" H 5900 2650 50  0001 C CNN
+F 0 "#PWR018" H 5900 2650 50  0001 C CNN
 F 1 "GND" H 5900 2750 50  0000 C CNN
 F 2 "" H 5900 2900 50  0001 C CNN
@@
 $EndComp
 $Comp
-L GND #PWR25
+L GND #PWR019
 U 1 1 61E954D7
 P 8600 3750
-F 0 "#PWR25" H 8600 3500 50  0001 C CNN
+F 0 "#PWR019" H 8600 3500 50  0001 C CNN
 F 1 "GND" H 8600 3600 50  0000 C CNN
 F 2 "" H 8600 3750 50  0001 C CNN
@@
 Connection ~ 7000 3350
 $Comp
-L GND #PWR24
+L GND #PWR020
 U 1 1 61E9593A
 P 7200 3800
-F 0 "#PWR24" H 7200 3550 50  0001 C CNN
+F 0 "#PWR020" H 7200 3550 50  0001 C CNN
 F 1 "GND" H 7200 3650 50  0000 C CNN
 F 2 "" H 7200 3800 50  0001 C CNN
@@
 SPKR
 $Comp
-L GND #PWR12
+L GND #PWR021
 U 1 1 61ECE877
 P 4500 1400
-F 0 "#PWR12" H 4500 1150 50  0001 C CNN
+F 0 "#PWR021" H 4500 1150 50  0001 C CNN
 F 1 "GND" H 4500 1250 50  0000 C CNN
 F 2 "" H 4500 1400 50  0001 C CNN
@@
 Connection ~ 4350 1300
 $Comp
-L +5V #PWR21
+L +5V #PWR022
 U 1 1 61ECEE17
 P 6600 2450
-F 0 "#PWR21" H 6600 2300 50  0001 C CNN
+F 0 "#PWR022" H 6600 2300 50  0001 C CNN
 F 1 "+5V" H 6600 2590 50  0000 C CNN
 F 2 "" H 6600 2450 50  0001 C CNN
@@
 $EndComp
 $Comp
-L +5V #PWR23
+L +5V #PWR023
 U 1 1 61ECF2E6
 P 6950 1350
-F 0 "#PWR23" H 6950 1200 50  0001 C CNN
+F 0 "#PWR023" H 6950 1200 50  0001 C CNN
 F 1 "+5V" H 6950 1490 50  0000 C CNN
 F 2 "" H 6950 1350 50  0001 C CNN
@@
 $EndComp
 Wire Wire Line
-	4700 1200 4400 1200
+	4400 1200 4700 1200
 $Comp
 L R R22
@@
 $EndComp
 $Comp
-L GND #PWR10
+L GND #PWR024
 U 1 1 61ED1FD3
 P 4150 2850
-F 0 "#PWR10" H 4150 2600 50  0001 C CNN
+F 0 "#PWR024" H 4150 2600 50  0001 C CNN
 F 1 "GND" H 4150 2700 50  0000 C CNN
 F 2 "" H 4150 2850 50  0001 C CNN
@@
 $EndComp
 $Comp
-L GND #PWR20
+L GND #PWR025
 U 1 1 6219F5CD
 P 6300 7200
-F 0 "#PWR20" H 6300 6950 50  0001 C CNN
+F 0 "#PWR025" H 6300 6950 50  0001 C CNN
 F 1 "GND" H 6300 7050 50  0000 C CNN
 F 2 "" H 6300 7200 50  0001 C CNN
@@
 $EndComp
 $Comp
-L GND #PWR18
+L GND #PWR026
 U 1 1 6219F5D9
 P 5850 7250
-F 0 "#PWR18" H 5850 7000 50  0001 C CNN
+F 0 "#PWR026" H 5850 7000 50  0001 C CNN
 F 1 "GND" H 5850 7100 50  0000 C CNN
 F 2 "" H 5850 7250 50  0001 C CNN
@@
 Wire Notes Line
 	6550 5300 6550 7550
+$Comp
+L Conn_01x20 J10
+U 1 1 625E2ED6
+P 2250 4450
+F 0 "J10" H 2250 5450 50  0000 C CNN
+F 1 "Conn_01x20" H 2250 3350 50  0000 C CNN
+F 2 "Pin_Headers:Pin_Header_Straight_1x20_Pitch2.54mm" H 2250 4450 50  0001 C CNN
+F 3 "" H 2250 4450 50  0001 C CNN
+	1    2250 4450
+	0    -1   -1   0
+$EndComp
+Wire Wire Line
+	1350 4650 3250 4650
+Connection ~ 3150 4650
+Connection ~ 3050 4650
+Connection ~ 2950 4650
+Connection ~ 2850 4650
+Connection ~ 2750 4650
+Connection ~ 2650 4650
+Connection ~ 2550 4650
+Connection ~ 2450 4650
+Connection ~ 2350 4650
+Connection ~ 2250 4650
+Connection ~ 2150 4650
+Connection ~ 2050 4650
+Connection ~ 1950 4650
+Connection ~ 1850 4650
+Connection ~ 1750 4650
+Connection ~ 1650 4650
+Connection ~ 1550 4650
+Connection ~ 1450 4650
+$Comp
+L GND #PWR027
+U 1 1 625E4A8D
+P 1350 4700
+F 0 "#PWR027" H 1350 4450 50  0001 C CNN
+F 1 "GND" H 1350 4550 50  0000 C CNN
+F 2 "" H 1350 4700 50  0001 C CNN
+F 3 "" H 1350 4700 50  0001 C CNN
+	1    1350 4700
+	1    0    0    -1
+$EndComp
+Wire Wire Line
+	1350 4700 1350 4650
+Wire Notes Line
+	1150 4250 3500 4250
+Wire Notes Line
+	3500 4250 3500 4950
+Wire Notes Line
+	3500 4950 1150 4950
+Wire Notes Line
+	1150 4950 1150 4250
 $EndSCHEMATC

Commit message: Changed bitbang display values
Parts:
- C12, C9: value 1 nF -> 100 pF
Changed lines of the file:
@@
 P 6750 4200
 F 0 "C9" V 6800 4250 50  0000 L CNN
-F 1 "1 nF" V 6600 4150 50  0000 L CNN
+F 1 "100 pF" V 6600 4150 50  0000 L CNN
 F 2 "Capacitors_THT:C_Disc_D5.0mm_W2.5mm_P5.00mm" H 6750 4200 50  0001 C CNN
 F 3 "" H 6750 4200 50  0001 C CNN
@@
 P 8050 3700
 F 0 "C12" V 8100 3750 50  0000 L CNN
-F 1 "1 nF" V 7900 3650 50  0000 L CNN
+F 1 "100 pF" V 7900 3650 50  0000 L CNN
 F 2 "Capacitors_THT:C_Disc_D5.0mm_W2.5mm_P5.00mm" H 8050 3700 50  0001 C CNN
 F 3 "" H 8050 3700 50  0001 C CNN
