File: BitBangDisplay/BitBangDisplay.kicad_pcb (KiCad board)
At the start: 2 copper layers, 100 x 88 mm, 72 parts, among them J1 Conn_01x04, J10 Conn_01x04, J11 Conn_01x01, J12 Conn_01x01, J13 KeyerJack, J14 KeyerJack, J15 KeyerJack, J19 Conn_01x04, J2 Audio-Jack-3, J20 Conn_01x01, J21 Conn_01x01, J22 SPEAKER, J3 Conn_01x01, J4 Conn_01x01, J5 Conn_01x01, J6 Conn_01x01, J7 Conn_01x01, J8 Conn_01x01, J9 Conn_01x01, SW2 SW_Push, SW3 SW_Push, SW4 SW_Push, SW5 SW_Push, U1 LCD-016N002L, U2 LM358, U5 LCD-016N002L

Commit message: Before trying to put everything onto a single line
Parts:
- added J16: SPEAKER, Connectors_Terminal_Blocks:TerminalBlock_bornier-2_P5.08mm, F.Cu at (128.0, 128.9)
- J2: value Audio-Jack-3 -> Audio-Jack-3_2Switches
- moved C4 18.1 mm to (106.6, 129.6)
Connections:
- J2 pad 2: (no net) -> Net-(C1-Pad1)
- J2 pad 4: (no net) -> Net-(J16-Pad1)
Routing:
- net Net-(J16-Pad1): track 0.00 -> 41.4 mm
- net Net-(C1-Pad2): track 49.9 -> 77.0 mm
- net Net-(C4-Pad2): track 19.6 -> 29.2 mm
- net Net-(C1-Pad1): track 46.6 -> 51.0 mm
Other:
- board text added: "INTERNAL SPEAKER"
Changed lines of the file:
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@@
 (kicad_pcb (version 4) (host pcbnew 4.0.7)
   (general
-    (links 123)
+    (links 126)
     (no_connects 0)
     (area 31.924999 56.924999 132.075001 145.075001)
     (thickness 1.6)
-    (drawings 32)
-    (tracks 365)
+    (drawings 33)
+    (tracks 385)
     (zones 0)
-    (modules 72)
-    (nets 44)
+    (modules 73)
+    (nets 45)
   )
   (page A4)
@@
   (net 42 "Net-(JP3-Pad1)")
   (net 43 "Net-(JP4-Pad1)")
+  (net 44 "Net-(J16-Pad1)")
   (net_class Default "This is the default net class."
     (clearance 0.2)
@@
     (add_net "Net-(J14-Pad1)")
     (add_net "Net-(J14-Pad2)")
+    (add_net "Net-(J16-Pad1)")
     (add_net "Net-(JP1-Pad2)")
     (add_net "Net-(JP2-Pad2)")
@@
       (effects (font (size 1 1) (thickness 0.15)))
     )
-    (fp_text value Audio-Jack-3 (at 0 -0.5 180) (layer F.Fab)
+    (fp_text value Audio-Jack-3_2Switches (at 0 -0.5 180) (layer F.Fab)
       (effects (font (size 1 1) (thickness 0.15)))
     )
@@
     (pad 1 thru_hole oval (at -4.8 6.1 180) (size 1 2) (drill oval 0.75 1.5) (layers *.Cu *.Mask)
       (net 22 "Net-(C1-Pad1)"))
-    (pad 2 thru_hole oval (at 5.2 9.6 180) (size 1 2) (drill oval 0.75 1.5) (layers *.Cu *.Mask))
-    (pad 4 thru_hole oval (at -4.3 13 180) (size 2 1.5) (drill oval 1.5 1) (layers *.Cu *.Mask))
+    (pad 2 thru_hole oval (at 5.2 9.6 180) (size 1 2) (drill oval 0.75 1.5) (layers *.Cu *.Mask)
+      (net 22 "Net-(C1-Pad1)"))
+    (pad 4 thru_hole oval (at -4.3 13 180) (size 2 1.5) (drill oval 1.5 1) (layers *.Cu *.Mask)
+      (net 44 "Net-(J16-Pad1)"))
     (pad 5 thru_hole oval (at 2.6 8.6 180) (size 1.5 2) (drill oval 1 1.5) (layers *.Cu *.Mask))
   )
@@
   )
   (module Capacitors_THT:C_Disc_D5.0mm_W2.5mm_P5.00mm (layer B.Cu)
-    (at 124.63 130.87 270)
+    (at 106.6 129.58 270)
     (descr "C, Disc series, Radial, pin pitch=5.00mm, , diameter*width=5*2.5mm^2, Capacitor, http://cdn-reichelt.de/documents/datenblatt/B300/DS_KERKO_TC.pdf")
     (tags "C Disc series Radial pin pitch 5.00mm  diameter 5mm width 2.5mm Capacitor")
@@
     )
   )
+  (module Connectors_Terminal_Blocks:TerminalBlock_bornier-2_P5.08mm (layer F.Cu)
+    (at 128.02 128.93 270)
+    (descr "simple 2-pin terminal block, pitch 5.08mm, revamped version of bornier2")
+    (tags "terminal block bornier2")
+    (fp_text reference J16 (at 2.54 -5.08 270) (layer F.SilkS)
+      (effects (font (size 1 1) (thickness 0.15)))
+    )
+    (fp_text value SPEAKER (at 2.54 5.08 270) (layer F.Fab)
+      (effects (font (size 1 1) (thickness 0.15)))
+    )
+    (fp_text user %R (at 2.54 0 270) (layer F.Fab)
+      (effects (font (size 1 1) (thickness 0.15)))
+    )
+    (fp_line (start -2.41 2.55) (end 7.49 2.55) (layer F.Fab) (width 0.1))
+    (fp_line (start -2.46 -3.75) (end -2.46 3.75) (layer F.Fab) (width 0.1))
+    (fp_line (start -2.46 3.75) (end 7.54 3.75) (layer F.Fab) (width 0.1))
+    (fp_line (start 7.54 3.75) (end 7.54 -3.75) (layer F.Fab) (width 0.1))
+    (fp_line (start 7.54 -3.75) (end -2.46 -3.75) (layer F.Fab) (width 0.1))
+    (fp_line (start 7.62 2.54) (end -2.54 2.54) (layer F.SilkS) (width 0.12))
+    (fp_line (start 7.62 3.81) (end 7.62 -3.81) (layer F.SilkS) (width 0.12))
+    (fp_line (start 7.62 -3.81) (end -2.54 -3.81) (layer F.SilkS) (width 0.12))
+    (fp_line (start -2.54 -3.81) (end -2.54 3.81) (layer F.SilkS) (width 0.12))
+    (fp_line (start -2.54 3.81) (end 7.62 3.81) (layer F.SilkS) (width 0.12))
+    (fp_line (start -2.71 -4) (end 7.79 -4) (layer F.CrtYd) (width 0.05))
+    (fp_line (start -2.71 -4) (end -2.71 4) (layer F.CrtYd) (width 0.05))
+    (fp_line (start 7.79 4) (end 7.79 -4) (layer F.CrtYd) (width 0.05))
+    (fp_line (start 7.79 4) (end -2.71 4) (layer F.CrtYd) (width 0.05))
+    (pad 1 thru_hole rect (at 0 0 270) (size 3 3) (drill 1.52) (layers *.Cu *.Mask)
+      (net 44 "Net-(J16-Pad1)"))
+    (pad 2 thru_hole circle (at 5.08 0 270) (size 3 3) (drill 1.52) (layers *.Cu *.Mask)
+      (net 23 "Net-(C1-Pad2)"))
+    (model ${KISYS3DMOD}/Terminal_Blocks.3dshapes/TerminalBlock_bornier-2_P5.08mm.wrl
+      (at (xyz 0.1 0 0))
+      (scale (xyz 1 1 1))
+      (rotate (xyz 0 0 0))
+    )
+  )
+  (gr_text "INTERNAL\nSPEAKER" (at 128.09 124.82) (layer F.SilkS)
+    (effects (font (size 1 1) (thickness 0.15)))
+  )
   (gr_text 1 (at 79.96 105.05) (layer B.SilkS)
     (effects (font (size 1 1) (thickness 0.15)) (justify mirror))
@@
   (segment (start 93.392 87.456) (end 93.472 87.376) (width 0.5) (layer B.Cu) (net 21) (status 30))
   (segment (start 93.472 87.376) (end 93.642 87.376) (width 0.5) (layer F.Cu) (net 21) (status 30))
+  (segment (start 93.3 134.95) (end 93.3 137.95) (width 0.5) (layer B.Cu) (net 22))
+  (segment (start 93.3 137.95) (end 94.265 138.915) (width 0.5) (layer B.Cu) (net 22))
   (segment (start 65.5 133.5) (end 65.83 133.5) (width 0.5) (layer B.Cu) (net 22))
   (segment (start 65.83 133.5) (end 68.01 135.68) (width 0.5) (layer B.Cu) (net 22))
@@
   (segment (start 78.73 139.08) (end 80.36 140.71) (width 0.5) (layer B.Cu) (net 22))
   (segment (start 80.36 140.71) (end 92.47 140.71) (width 0.5) (layer B.Cu) (net 22))
-  (segment (start 92.47 140.71) (end 94.73 138.45) (width 0.5) (layer B.Cu) (net 22))
+  (segment (start 92.47 140.71) (end 94.265 138.915) (width 0.5) (layer B.Cu) (net 22))
+  (segment (start 94.265 138.915) (end 94.73 138.45) (width 0.5) (layer B.Cu) (net 22))
   (segment (start 94.73 138.45) (end 103.3 138.45) (width 0.5) (layer B.Cu) (net 22))
   (segment (start 103.3 138.45) (end 105.76 138.45) (width 0.5) (layer B.Cu) (net 22))
   (segment (start 105.76 138.45) (end 106.51 139.2) (width 0.5) (layer B.Cu) (net 22))
+  (segment (start 106.51 141.7) (end 124.32 141.7) (width 0.5) (layer B.Cu) (net 23))
+  (segment (start 125.2 136.83) (end 128.02 134.01) (width 0.5) (layer B.Cu) (net 23))
+  (segment (start 125.2 140.82) (end 125.2 136.83) (width 0.5) (layer B.Cu) (net 23))
+  (segment (start 124.32 141.7) (end 125.2 140.82) (width 0.5) (layer B.Cu) (net 23))
   (segment (start 62.96 133.5) (end 62.96 133.6) (width 0.5) (layer B.Cu) (net 23))
   (segment (start 62.96 133.6) (end 65.93 136.57) (width 0.5) (layer B.Cu) (net 23))
@@
   (segment (start 111.25 81.03) (end 111.25 81.63) (width 0.35) (layer B.Cu) (net 32))
   (segment (start 111.25 81.63) (end 107.96 84.92) (width 0.35) (layer B.Cu) (net 32))
+  (segment (start 120.85 138.57) (end 119.52 138.57) (width 0.35) (layer B.Cu) (net 33))
+  (segment (start 119.52 138.57) (end 119.25 138.3) (width 0.35) (layer B.Cu) (net 33))
+  (segment (start 107.8 134.58) (end 106.6 134.58) (width 0.35) (layer B.Cu) (net 33))
+  (segment (start 111.52 138.3) (end 107.8 134.58) (width 0.35) (layer B.Cu) (net 33))
+  (segment (start 119.25 138.3) (end 111.52 138.3) (width 0.35) (layer B.Cu) (net 33))
   (segment (start 121.08 128.05) (end 119.64 128.05) (width 0.35) (layer B.Cu) (net 33))
-  (segment (start 119.52 138.57) (end 120.85 138.57) (width 0.35) (layer B.Cu) (net 33))
   (segment (start 117.92 136.97) (end 119.52 138.57) (width 0.35) (layer B.Cu) (net 33))
   (segment (start 117.92 129.77) (end 117.92 136.97) (width 0.35) (layer B.Cu) (net 33))
   (segment (start 119.64 128.05) (end 117.92 129.77) (width 0.35) (layer B.Cu) (net 33))
-  (segment (start 124.63 135.87) (end 123.55 135.87) (width 0.35) (layer B.Cu) (net 33))
-  (segment (start 123.55 135.87) (end 120.85 138.57) (width 0.35) (layer B.Cu) (net 33))
   (segment (start 110.92 128.05) (end 93.65 128.05) (width 0.35) (layer B.Cu) (net 34))
   (segment (start 90.81 125.21) (end 90.81 111.09) (width 0.35) (layer B.Cu) (net 34))
@@
   (segment (start 62.25 100.11) (end 62.25 97.12) (width 0.35) (layer B.Cu) (net 43))
   (segment (start 65.62 103.48) (end 62.25 100.11) (width 0.35) (layer B.Cu) (net 43))
+  (segment (start 102.8 131.55) (end 102.8 134.45) (width 0.5) (layer B.Cu) (net 44))
+  (segment (start 125.6 128.93) (end 128.02 128.93) (width 0.5) (layer B.Cu) (net 44))
+  (segment (start 123.55 130.98) (end 125.6 128.93) (width 0.5) (layer B.Cu) (net 44))
+  (segment (start 123.55 139.92) (end 123.55 130.98) (width 0.5) (layer B.Cu) (net 44))
+  (segment (start 122.76 140.71) (end 123.55 139.92) (width 0.5) (layer B.Cu) (net 44))
+  (segment (start 110.87 140.71) (end 122.76 140.71) (width 0.5) (layer B.Cu) (net 44))
+  (segment (start 108.63 138.47) (end 110.87 140.71) (width 0.5) (layer B.Cu) (net 44))
+  (segment (start 108.63 137.55) (end 108.63 138.47) (width 0.5) (layer B.Cu) (net 44))
+  (segment (start 107.93 136.85) (end 108.63 137.55) (width 0.5) (layer B.Cu) (net 44))
+  (segment (start 105.2 136.85) (end 107.93 136.85) (width 0.5) (layer B.Cu) (net 44))
+  (segment (start 102.8 134.45) (end 105.2 136.85) (width 0.5) (layer B.Cu) (net 44))
   (zone (net 2) (net_name GND) (layer F.Cu) (hatch edge 0.508)
     (connect_pads (clearance 1))

Commit message: Changed external connector for single 20 pin or ribbon cable
Parts:
- removed J10, J19: Conn_01x04, Pin_Headers:Pin_Header_Straight_1x04_Pitch2.54mm
- removed J22: SPEAKER, Pin_Headers:Pin_Header_Straight_1x02_Pitch2.54mm
- added C13: 100 nF, Capacitors_THT:C_Disc_D5.0mm_W2.5mm_P2.50mm, B.Cu at (97.5, 97.2)
- added L4: 100 uH, Inductors_THT:L_Axial_L6.6mm_D2.7mm_P10.16mm_Horizontal_Vishay_IM-2, B.Cu at (101.7, 121.4)
- added R22: 47R, Resistors_THT:R_Axial_DIN0207_L6.3mm_D2.5mm_P7.62mm_Horizontal, B.Cu at (101.7, 124.8)
- R9: moved to B.Cu
- U1: value LCD-016N002L -> LCD1602ExtraPins
- U5: value LCD-016N002L -> LCD1602ExtraPins; footprint Pin_Headers:Pin_Header_Straight_1x16_Pitch2.54mm -> Pin_Headers:Pin_Header_Straight_1x20_Pitch2.54mm
- moved L3 23.0 mm to (101.7, 115.7)
- moved R1 21.1 mm to (90.4, 89.8), turned to 0 degrees
- moved R2 18.7 mm to (90.2, 86.6), turned to 0 degrees
- moved R4 17.3 mm to (87.5, 93.8)
- moved R5 8.59 mm to (94.1, 104.8)
- moved R13 7.85 mm to (65.2, 134.2)
- moved R46 7.85 mm to (61.9, 134.2)
- moved R12 7.83 mm to (58.7, 134.2)
- moved R47 7.79 mm to (55.5, 134.2)
- moved R33 7.77 mm to (52.2, 134.2)
- moved R29 7.75 mm to (42.3, 134.1)
- moved R3 7.75 mm to (48.9, 134.2)
- moved R6 7.73 mm to (45.6, 134.2)
- moved L2 3.61 mm to (101.0, 77.4)
- moved L1 3.42 mm to (100.9, 80.9)
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Connections:
- C1 pad 2: Net-(C1-Pad2) -> GND
- C7 pad 1: +5VP -> +5V
- J16 pad 2: Net-(C1-Pad2) -> GND
- J2 pad 3: Net-(C1-Pad2) -> GND
- R1 pad 1: Net-(J10-Pad1) -> PTT
- R11 pad 1: +5VP -> +5V
- R2 pad 1: Net-(J10-Pad3) -> MIC
- R20 pad 2: Net-(J10-Pad3) -> MIC
- R4 pad 1: +5VP -> +5V
- R4 pad 2: Net-(J10-Pad1) -> PTT
- R5 pad 2: +5VP -> +5V
- U2 pad 8: +5VP -> +5V
Routing:
- net +5V: track 98.3 -> 200.7 mm
- net Net-(C1-Pad2): track 77.0 -> 0.00 mm
- net PTT: track 0.00 -> 70.7 mm
- net MIC: track 0.00 -> 68.1 mm
- net SPKR: track 0.00 -> 49.8 mm
- net Net-(C5-Pad1): track 53.8 -> 12.6 mm
- net +5VP: track 36.6 -> 0.00 mm
- net GND: track 0.00 -> 36.0 mm
- net Net-(J10-Pad1): track 30.3 -> 0.00 mm
- net Net-(J10-Pad3): track 28.9 -> 0.00 mm
- net Net-(C1-Pad1): track 51.0 -> 36.3 mm
- net DB6: track 88.0 -> 100.5 mm
- net Net-(L2-Pad2): track 5.25 -> 17.1 mm
- net DB7: track 95.2 -> 106.9 mm
- net DB4: track 74.7 -> 86.0 mm
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Other:
- board text added: "AN"
- board text added: "KA"
- board text added: "PTT"
- board text added: "SPKR"
- board text removed: "KY1"

Commit message: Before adding SI5351 header
Parts:
- moved J13 18.2 mm to (119.1, 57.1)
- moved J14 13.1 mm to (101.3, 57.1)
- moved L1 12.7 mm to (113.5, 80.9)
- moved L2 12.6 mm to (113.6, 77.4)
- moved C3 11.5 mm to (109.6, 76.6)
- moved C2 9.84 mm to (123.9, 74.0)
- moved U1 1.75 mm to (42.8, 66.0)
Routing:
- net Net-(L2-Pad2): track 17.1 -> 32.5 mm
- net Net-(L1-Pad2): track 16.7 -> 31.0 mm
- net Net-(J1-Pad1): track 35.7 -> 48.0 mm
- net Net-(J14-Pad2): track 23.2 -> 35.2 mm
- net Net-(J14-Pad1): track 20.9 -> 29.5 mm
- net Net-(C3-Pad2): track 22.9 -> 27.2 mm
- net K: track 72.4 -> 74.5 mm
- net DB5: track 92.3 -> 94.3 mm
- net DB4: track 86.0 -> 87.9 mm
- net AVEE: track 70.1 -> 72.0 mm
- net +5V: track 200.7 -> 199.1 mm
- net RW: track 19.4 -> 21.1 mm
- net VO: track 16.4 -> 14.8 mm
- net Net-(C2-Pad2): track 17.9 -> 16.5 mm
- net DB7: track 106.9 -> 107.8 mm
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Other:
- board text added: "RFBitBanger Display V2 BY DANIEL MARKS KW4TI CC-BY-SA 4.0"
- board text removed: "RFBitBanger Display BY DANIEL MARKS KW4TI CC-BY-SA 4.0"

Commit message: Added fifth button
Parts:
- added C14: 100 nF, Capacitors_THT:C_Disc_D5.0mm_W2.5mm_P2.50mm, B.Cu at (36.1, 137.7)
- added R23: 10k, Resistors_THT:R_Axial_DIN0207_L6.3mm_D2.5mm_P7.62mm_Horizontal, B.Cu at (35.8, 134.1)
- added R24: 1k, Resistors_THT:R_Axial_DIN0207_L6.3mm_D2.5mm_P7.62mm_Horizontal, B.Cu at (39.0, 134.1)
- added SW1: SW_Push, Buttons_Switches_THT:SW_PUSH_6mm, F.Cu at (53.4, 138.6)
- moved C16 12.1 mm to (70.1, 135.6)
- moved C11 2.46 mm to (70.1, 130.0)
Routing:
- net RS: track 16.7 -> 69.0 mm
- net Net-(C14-Pad2): track 0.00 -> 29.8 mm
- net +5V: track 199.1 -> 212.2 mm
- net Net-(C16-Pad2): track 20.6 -> 31.1 mm
- net Net-(C11-Pad2): track 37.4 -> 42.9 mm
- net DB5: track 94.3 -> 89.1 mm
- net DB6: track 101.2 -> 96.3 mm
- net GND: track 36.0 -> 40.4 mm
- net DB4: track 87.9 -> 83.6 mm
- net DB7: track 107.8 -> 103.9 mm
- net Net-(C17-Pad2): track 38.5 -> 40.5 mm
- net Net-(C10-Pad2): track 48.2 -> 49.3 mm

Commit message: Added extra row of ground pins for 40 pin connector
Parts:
- added J10: Conn_01x20, Pin_Headers:Pin_Header_Straight_1x20_Pitch2.54mm, B.Cu at (49.0, 72.5)
- U5: moved to B.Cu
- turned U5 to 180 degrees
Routing:
- net VO: track 14.8 -> 18.5 mm
- net AVEE: track 72.0 -> 68.5 mm
- net DB7: track 103.9 -> 100.5 mm
- net K: track 74.5 -> 71.1 mm
- net DB6: track 96.3 -> 93.6 mm
- net DB5: track 89.1 -> 87.1 mm
- net RS: track 69.0 -> 70.9 mm
- net PTT: track 70.7 -> 68.8 mm
- net DB4: track 83.6 -> 82.0 mm
- net Net-(C9-Pad2): track 44.6 -> 43.1 mm
- net MIC: track 68.1 -> 66.8 mm
- net SPKR: track 49.8 -> 51.0 mm
- net E: track 25.2 -> 24.7 mm
Other:
- board text added: "SPK"
- board text removed: "SPKR"

Commit message: Modified FSK SLOW mode, added section back about +- filters
Parts:
- moved J12 1.00 mm to (36.5, 97.0)
- moved J8 1.00 mm to (111.5, 97.0)
Routing:
- net DB4: track 82.0 -> 81.2 mm
- net RS: track 70.9 -> 71.4 mm
Changed lines of the file:
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@@
   )
   (setup
-    (last_trace_width 0.35)
+    (last_trace_width 0.25)
     (user_trace_width 0.35)
     (user_trace_width 0.5)
@@
   )
   (module BitBangDisplay:SimpleHole (layer F.Cu)
-    (at 110.5 97)
+    (at 111.5 97)
     (fp_text reference J8 (at 0 0.5) (layer F.SilkS) hide
       (effects (font (size 1 1) (thickness 0.15)))
@@
   )
   (module BitBangDisplay:SimpleHole (layer F.Cu)
-    (at 35.5 97)
+    (at 36.5 97)
     (fp_text reference J12 (at 0 0.5) (layer F.SilkS) hide
       (effects (font (size 1 1) (thickness 0.15)))
@@
   (segment (start 45.4 128.8) (end 38.26 128.8) (width 0.5) (layer B.Cu) (net 1))
   (segment (start 38.26 128.8) (end 34.31 128.8) (width 0.5) (layer B.Cu) (net 1))
-  (segment (start 37.17 123.63) (end 38.61 122.19) (width 0.5) (layer B.Cu) (net 1))
-  (segment (start 34.23 123.63) (end 37.17 123.63) (width 0.5) (layer B.Cu) (net 1))
-  (segment (start 33.42 124.44) (end 34.23 123.63) (width 0.5) (layer B.Cu) (net 1))
-  (segment (start 33.42 127.91) (end 33.42 124.44) (width 0.5) (layer B.Cu) (net 1))
+  (segment (start 37.46 123.79) (end 40.48 122.71) (width 0.5) (layer B.Cu) (net 1))
+  (segment (start 34.23 124.87) (end 37.46 123.79) (width 0.5) (layer B.Cu) (net 1))
+  (segment (start 33.42 125.68) (end 34.23 124.87) (width 0.5) (layer B.Cu) (net 1))
+  (segment (start 33.42 127.91) (end 33.42 125.68) (width 0.5) (layer B.Cu) (net 1))
   (segment (start 34.31 128.8) (end 33.42 127.91) (width 0.5) (layer B.Cu) (net 1))
   (segment (start 46.5 75.04) (end 45.59 75.04) (width 0.35) (layer B.Cu) (net 1))
@@
   (segment (start 58.68 127.37) (end 57.25 128.8) (width 0.35) (layer B.Cu) (net 1))
   (segment (start 65.21 126.57) (end 65.21 127.4) (width 0.5) (layer B.Cu) (net 1))
-  (segment (start 38.61 82.93) (end 46.5 75.04) (width 0.5) (layer B.Cu) (net 1))
-  (segment (start 38.61 122.19) (end 38.61 82.93) (width 0.5) (layer B.Cu) (net 1))
+  (segment (start 40.48 82.62) (end 46.5 75.04) (width 0.5) (layer B.Cu) (net 1))
+  (segment (start 40.48 122.71) (end 40.48 82.62) (width 0.5) (layer B.Cu) (net 1))
   (segment (start 63.81 128.8) (end 59.74 128.8) (width 0.5) (layer B.Cu) (net 1))
   (segment (start 59.74 128.8) (end 57.25 128.8) (width 0.5) (layer B.Cu) (net 1))
@@
   (segment (start 47.65 124.89) (end 44.77 124.89) (width 0.35) (layer B.Cu) (net 6))
   (segment (start 44.95 100.44) (end 46.5 100.44) (width 0.35) (layer B.Cu) (net 6))
-  (segment (start 42.48 102.91) (end 44.95 100.44) (width 0.35) (layer B.Cu) (net 6))
-  (segment (start 42.48 122.6) (end 42.48 102.91) (width 0.35) (layer B.Cu) (net 6))
-  (segment (start 44.77 124.89) (end 42.48 122.6) (width 0.35) (layer B.Cu) (net 6))
+  (segment (start 42.82 102.91) (end 44.95 100.44) (width 0.35) (layer B.Cu) (net 6))
+  (segment (start 42.82 122.6) (end 42.82 102.91) (width 0.35) (layer B.Cu) (net 6))
+  (segment (start 44.77 124.89) (end 42.82 122.6) (width 0.35) (layer B.Cu) (net 6))
   (segment (start 48.93 126.55) (end 48.93 126.17) (width 0.35) (layer B.Cu) (net 6))
   (segment (start 48.93 126.17) (end 47.65 124.89) (width 0.35) (layer B.Cu) (net 6))
@@
   (segment (start 47.9 96.61) (end 50.67 96.61) (width 0.35) (layer B.Cu) (net 7))
   (segment (start 42.33 126.51) (end 42.33 124.69) (width 0.35) (layer B.Cu) (net 7))
-  (segment (start 41.46 102.49) (end 46.05 97.9) (width 0.35) (layer B.Cu) (net 7))
-  (segment (start 41.46 123.82) (end 41.46 102.49) (width 0.35) (layer B.Cu) (net 7))
-  (segment (start 42.33 124.69) (end 41.46 123.82) (width 0.35) (layer B.Cu) (net 7))
+  (segment (start 42.1 102.49) (end 46.05 97.9) (width 0.35) (layer B.Cu) (net 7))
+  (segment (start 42.1 123.82) (end 42.1 102.49) (width 0.35) (layer B.Cu) (net 7))
+  (segment (start 42.33 124.69) (end 42.1 123.82) (width 0.35) (layer B.Cu) (net 7))
   (segment (start 46.05 97.9) (end 46.5 97.9) (width 0.35) (layer B.Cu) (net 7))
   (segment (start 42.06 126.51) (end 42.33 126.51) (width 0.35) (layer B.Cu) (net 7))
@@
   (segment (start 47.96 101.69) (end 50.98 101.69) (width 0.35) (layer B.Cu) (net 9))
   (segment (start 51.47 124.22) (end 45.54 124.22) (width 0.35) (layer B.Cu) (net 9))
-  (segment (start 43.36 105.39) (end 45.77 102.98) (width 0.35) (layer B.Cu) (net 9))
-  (segment (start 43.36 122.04) (end 43.36 105.39) (width 0.35) (layer B.Cu) (net 9))
-  (segment (start 45.54 124.22) (end 43.36 122.04) (width 0.35) (layer B.Cu) (net 9))
+  (segment (start 43.56 105.39) (end 45.77 102.98) (width 0.35) (layer B.Cu) (net 9))
+  (segment (start 43.56 122.04) (end 43.56 105.39) (width 0.35) (layer B.Cu) (net 9))
+  (segment (start 45.54 124.22) (end 43.56 122.04) (width 0.35) (layer B.Cu) (net 9))
   (segment (start 45.77 102.98) (end 46.5 102.98) (width 0.35) (layer B.Cu) (net 9))
   (segment (start 55.47 126.55) (end 55.47 125.77) (width 0.35) (layer B.Cu) (net 9))
@@
   (segment (start 50.3 78.84) (end 51.61 77.53) (width 0.35) (layer B.Cu) (net 11))
   (segment (start 47.25 78.84) (end 50.3 78.84) (width 0.35) (layer B.Cu) (net 11))
-  (segment (start 40.29 122.57) (end 40.29 123.28) (width 0.35) (layer B.Cu) (net 11))
+  (segment (start 41.38 122.55) (end 41.36 123.46) (width 0.35) (layer B.Cu) (net 11))
   (segment (start 37.7 124.55) (end 35.76 126.49) (width 0.35) (layer B.Cu) (net 11))
-  (segment (start 39.02 124.55) (end 37.7 124.55) (width 0.35) (layer B.Cu) (net 11))
-  (segment (start 40.29 123.28) (end 39.02 124.55) (width 0.35) (layer B.Cu) (net 11))
+  (segment (start 40.58 124.54) (end 37.7 124.55) (width 0.35) (layer B.Cu) (net 11))
+  (segment (start 41.36 123.46) (end 40.58 124.54) (width 0.35) (layer B.Cu) (net 11))
   (segment (start 35.76 126.49) (end 35.76 126.23) (width 0.35) (layer B.Cu) (net 11) (status 30))
-  (segment (start 40.29 122.57) (end 40.29 101.48) (width 0.35) (layer B.Cu) (net 11))
-  (segment (start 40.29 101.48) (end 43.73 98.04) (width 0.35) (layer B.Cu) (net 11))
+  (segment (start 41.38 122.55) (end 41.38 101.46) (width 0.35) (layer B.Cu) (net 11))
+  (segment (start 41.38 101.46) (end 43.73 98.04) (width 0.35) (layer B.Cu) (net 11))
   (segment (start 43.73 98.04) (end 43.73 82.08) (width 0.35) (layer B.Cu) (net 11))
   (segment (start 43.73 82.08) (end 45.69 80.12) (width 0.35) (layer B.Cu) (net 11))

Commit message: Converted all Kicad projects to version 6.0.10
Parts:
- C12, C9: value 1 nF -> 100 pF
Connections:
- C8 pad 2: Net-(C8-Pad2) -> +5V
- J1 pad 4: (no net) -> unconnected-(J1-Pad4)
- J15 pad 2: (no net) -> unconnected-(J15-Pad2)
- J2 pad 5: (no net) -> unconnected-(J2-Pad5)
- R11 pad 2: Net-(C8-Pad2) -> +5V
- R14 pad 1: Net-(C8-Pad2) -> +5V
- U1 pad 10: (no net) -> unconnected-(U1-Pad10)
- U1 pad 7: (no net) -> unconnected-(U1-Pad7)
- U1 pad 8: (no net) -> unconnected-(U1-Pad8)
- U1 pad 9: (no net) -> unconnected-(U1-Pad9)
- U2 pad 3: Net-(C8-Pad2) -> +5V
- U2 pad 5: Net-(C8-Pad2) -> +5V
- U5 pad 10: (no net) -> unconnected-(U5-Pad10)
- U5 pad 7: (no net) -> unconnected-(U5-Pad7)
- U5 pad 8: (no net) -> unconnected-(U5-Pad8)
- U5 pad 9: (no net) -> unconnected-(U5-Pad9)
Routing:
- net Net-(C8-Pad2): track 30.2 -> 0.00 mm
- net +5V: track 212.0 -> 242.1 mm
- net Net-(C11-Pad2): track 42.9 -> 41.1 mm
- net DB4: track 81.2 -> 80.3 mm
- net Net-(R46-Pad1): track 40.5 -> 39.8 mm
- net Net-(C9-Pad1): track 18.9 -> 18.2 mm
- net Net-(JP2-Pad1): track 29.5 -> 28.9 mm
- net RW: track 21.3 -> 20.7 mm
- net DB7: track 100.5 -> 99.9 mm
- net GND: track 40.4 -> 39.9 mm
Other:
- net class Default removed
