File: BitBangDisplay/BitBangDisplay.kicad_pcb (KiCad board)
At the start: 2 copper layers, 100 x 88 mm, 78 parts, among them J1 Conn_01x04, J10 Conn_01x20, J11 Conn_01x01, J12 Conn_01x01, J13 KeyerJack, J14 KeyerJack, J15 KeyerJack, J16 SPEAKER, J2 Audio-Jack-3_2Switches, J20 Conn_01x01, J21 Conn_01x01, J3 Conn_01x01, J4 Conn_01x01, J5 Conn_01x01, J6 Conn_01x01, J7 Conn_01x01, J8 Conn_01x01, J9 Conn_01x01, SW1 SW_Push, SW2 SW_Push, SW3 SW_Push, SW4 SW_Push, SW5 SW_Push, U1 LCD1602ExtraPins, U2 LM358, U5 LCD1602ExtraPins

Commit message: Added provisional iambic paddle state machine documentation
Connections:
- C8 pad 2: +5V -> Net-(C8-Pad2)
- R11 pad 2: +5V -> Net-(C8-Pad2)
- R14 pad 1: +5V -> Net-(C8-Pad2)
- U2 pad 3: +5V -> Net-(C8-Pad2)
- U2 pad 5: +5V -> Net-(C8-Pad2)
Routing:
- net +5V: track 242.1 -> 211.9 mm
- net Net-(C8-Pad2): track 0.00 -> 30.2 mm

Commit message: Aligned mounting holes to new display for BitBangDisplay
Parts:
- moved J13 15.8 mm to (103.4, 57.4)
- moved L2 11.8 mm to (101.8, 76.7)
- moved L1 11.7 mm to (101.9, 80.3)
- moved C2 11.4 mm to (114.8, 80.9), turned to 90 degrees
- moved C3 10.6 mm to (99.1, 75.7)
- moved J14 10.4 mm to (90.9, 57.4)
- moved J6 1.73 mm to (112.2, 66.0)
- moved J4 1.26 mm to (41.3, 65.0)
- moved J8 0.72 mm to (112.2, 97.0)
- moved J12 0.70 mm to (37.2, 97.0)
Routing:
- net Net-(L2-Pad2): track 32.5 -> 18.2 mm
- net Net-(L1-Pad2): track 31.0 -> 17.9 mm
- net Net-(J1-Pad1): track 48.0 -> 35.7 mm
- net Net-(J14-Pad2): track 35.2 -> 23.2 mm
- net Net-(J14-Pad1): track 28.9 -> 20.2 mm
- net Net-(C2-Pad2): track 16.5 -> 21.3 mm
Other:
- board text added: "RFBitBanger Display V3 BY DANIEL MARKS KW4TI CC-BY-SA 4.0"
- board text removed: "RFBitBanger Display V2 BY DANIEL MARKS KW4TI CC-BY-SA 4.0"

Commit message: Swapped UART and PADDLE jacks
Parts:
- moved J13 13.0 mm to (90.3, 57.4)
- moved J14 11.9 mm to (102.8, 57.4)
Routing:
- net Net-(J14-Pad2): track 23.2 -> 59.5 mm
- net Net-(J14-Pad1): track 20.2 -> 39.4 mm
- net Net-(J1-Pad1): track 35.7 -> 51.3 mm
- net Net-(C2-Pad2): track 21.3 -> 29.5 mm
