File: BitBangDisplay/BitBangDisplay.kicad_sch (KiCad schematic)
At the start: 78 parts, among them J1 Conn_01x04, J10 Conn_01x20, J11 Conn_01x01, J12 Conn_01x01, J13 KeyerJack, J14 KeyerJack, J15 KeyerJack, J16 SPEAKER, J2 Audio-Jack-3_2Switches, J20 Conn_01x01, J21 Conn_01x01, J3 Conn_01x01, J4 Conn_01x01, J5 Conn_01x01, J6 Conn_01x01, J7 Conn_01x01, J8 Conn_01x01, J9 Conn_01x01, SW1 SW_Push, SW2 SW_Push, SW3 SW_Push, SW4 SW_Push, SW5 SW_Push, U1 LCD1602ExtraPins, U2 LM358, U5 LCD1602ExtraPins

Commit message: Added provisional iambic paddle state machine documentation
Connections:
- net +5V: no longer C8.2, R11.2, R14.1, U2.3 (+), U2.5 (+)
- new net: C8.2, R11.2, R14.1, U2.3 (+), U2.5 (+)
Changed lines of the file:
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@@
   (junction (at 209.55 87.63) (diameter 0) (color 0 0 0 0)
   )
-  (junction (at 167.64 72.39) (diameter 0) (color 0 0 0 0)
-  )
   (junction (at 165.1 100.33) (diameter 0) (color 0 0 0 0)
   )
@@
     (stroke (width 0) (type default) (color 0 0 0 0))
   )
-  (wire (pts (xy 161.29 72.39) (xy 167.64 72.39))
-    (stroke (width 0) (type default) (color 0 0 0 0))
-  )
   (wire (pts (xy 218.44 66.04) (xy 218.44 67.31))
     (stroke (width 0) (type default) (color 0 0 0 0))
@@
     (stroke (width 0) (type default) (color 0 0 0 0))
   )
-  (wire (pts (xy 167.64 72.39) (xy 199.39 72.39))
-    (stroke (width 0) (type default) (color 0 0 0 0))
-  )
   (wire (pts (xy 102.87 148.59) (xy 102.87 170.18))
     (stroke (width 0) (type default) (color 0 0 0 0))
   )
-  (wire (pts (xy 199.39 72.39) (xy 199.39 74.93))
+  (wire (pts (xy 199.39 71.12) (xy 199.39 74.93))
     (stroke (width 0) (type default) (color 0 0 0 0))
   )
@@
     (stroke (width 0) (type default) (color 0 0 0 0))
   )
-  (wire (pts (xy 161.29 77.47) (xy 161.29 72.39))
+  (wire (pts (xy 161.29 71.12) (xy 161.29 77.47))
     (stroke (width 0) (type default) (color 0 0 0 0))
   )
@@
     (stroke (width 0) (type default) (color 0 0 0 0))
   )
+  (wire (pts (xy 161.29 71.12) (xy 199.39 71.12))
+    (stroke (width 0) (type default) (color 0 0 0 0))
+  )
