File: BandPassFilter/BandPassFilter.sch (KiCad schematic (older format))
At the start: 11 parts, among them J1 OUT, J2 INP

Commit message: BandPassFilter now has six filter boards on it
Parts:
- added C10, C16, C24, C29, C36: C3, Capacitors_THT:C_Disc_D5.0mm_W2.5mm_P5.00mm, symbol C_Small
- added C11, C18, C25, C30, C37: C4, Capacitors_THT:C_Disc_D5.0mm_W2.5mm_P5.00mm, symbol C_Small
- added C12, C19, C33, C38: C7, Capacitors_THT:C_Disc_D5.0mm_W2.5mm_P5.00mm, symbol C_Small
- added C13, C20, C26, C31, C39: C5, Capacitors_THT:C_Disc_D5.0mm_W2.5mm_P5.00mm, symbol C_Small
- added C14, C21, C32, C40: C6, Capacitors_THT:C_Disc_D5.0mm_W2.5mm_P5.00mm, symbol C_Small
- added C15, C22, C27, C34, C8: C1, Capacitors_THT:C_Disc_D5.0mm_W2.5mm_P5.00mm, symbol C_Small
- added C17, C23, C28, C35, C9: C2, Capacitors_THT:C_Disc_D5.0mm_W2.5mm_P5.00mm, symbol C_Small
- added C41: C8, Capacitors_THT:C_Disc_D5.0mm_W2.5mm_P5.00mm, symbol C_Small
- added C42: C9, Capacitors_THT:C_Disc_D5.0mm_W2.5mm_P5.00mm, symbol C_Small
- added J10, J12, J15, J4, J6, J8: OUT, Pin_Headers:Pin_Header_Straight_1x04_Pitch2.54mm, symbol Conn_01x04
- added J11, J14, J3, J5, J7, J9: INP, Pin_Headers:Pin_Header_Straight_1x04_Pitch2.54mm, symbol Conn_01x04
- added J13, J16: Conn_Coaxial, BandPassFilter:Amphenol_RF_SMA_132289, symbol Conn_Coaxial
- added L1, L10, L12, L5, L8: L2, BandPassFilter:L_Toroid_Horizontal_D12.7mm_Compact, symbol L_Small
- added L11, L13, L4, L6: L3, BandPassFilter:L_Toroid_Horizontal_D12.7mm_Compact, symbol L_Small
- added L14: L4, BandPassFilter:L_Toroid_Horizontal_D12.7mm_Compact, symbol L_Small
- added L7, L9: L1, BandPassFilter:L_Toroid_Horizontal_D12.7mm_Compact, symbol L_Small
Connections:
- net GND: now also C11.1, C14.1, C15.1, C18.1, C21.1, C22.1, C24.1, C26.1, C27.1, C29.1, C31.1, C34.1, C37.1, C40.1, C8.1, J10.1 (Pin_1), J10.2 (Pin_2), J11.1 (Pin_1), J11.2 (Pin_2), J12.1 (Pin_1), J12.2 (Pin_2), J13.2 (Ext), J14.1 (Pin_1), J14.2 (Pin_2), J15.1 (Pin_1), J15.2 (Pin_2), J16.2 (Ext), J3.1 (Pin_1), J3.2 (Pin_2), J4.1 (Pin_1), J4.2 (Pin_2), J5.1 (Pin_1), J5.2 (Pin_2), J6.1 (Pin_1), J6.2 (Pin_2), J7.1 (Pin_1), J7.2 (Pin_2), J8.1 (Pin_1), J8.2 (Pin_2), J9.1 (Pin_1), J9.2 (Pin_2), L11.2, L14.2
- new net: C8.2, J3.3 (Pin_3), J3.4 (Pin_4), L1.1
- new net: C9.1, L1.2
- new net: C10.1, C9.2
- new net: C10.2, C11.2, C12.1, C13.1, L4.1
- new net: C12.2, C13.2, C14.2, J4.3 (Pin_3), J4.4 (Pin_4), L4.2
- new net: C15.2, J5.3 (Pin_3), J5.4 (Pin_4), L5.1
- new net: C16.1, C17.1, L5.2
- new net: C16.2, C17.2, C18.2, C19.1, C20.1, L6.1
- new net: C19.2, C20.2, C21.2, J6.3 (Pin_3), J6.4 (Pin_4), L6.2
- new net: C22.2, C23.1, J7.3 (Pin_3), J7.4 (Pin_4), L7.1
- new net: C23.2, C24.2, C25.1, L7.2, L8.1
- new net: C25.2, C26.2, J8.3 (Pin_3), J8.4 (Pin_4), L8.2
- new net: C27.2, C28.1, J9.3 (Pin_3), J9.4 (Pin_4), L9.1
- new net: C28.2, C29.2, C30.1, L10.1, L9.2
- new net: C30.2, C31.2, C32.1, L10.2
- new net: C33.2, J10.3 (Pin_3), J10.4 (Pin_4)
- new net: C32.2, C33.1, L11.1
- new net: J13.1 (In), J14.3 (Pin_3), J14.4 (Pin_4)
- new net: J15.3 (Pin_3), J15.4 (Pin_4), J16.1 (In)
- new net: C34.2, J11.3 (Pin_3), J11.4 (Pin_4), L12.1
- new net: C35.1, L12.2
- new net: C35.2, C36.1
- new net: C36.2, C37.2, C38.1, C39.1, L13.1
- new net: C38.2, C39.2, C40.2, C41.1, L13.2
- new net: C42.2, J12.3 (Pin_3), J12.4 (Pin_4)
- new net: C41.2, C42.1, L14.1
Other:
- moved on the sheet: C1, C2, C3, C4, C5, C6, C7, J1, J2, L2, L3

Commit message: Modified BandPass Filter, Documentation
Connections:
- net at C2.1, L2.2: now also C3.1
- net at C2.2: now also C3.2, C4.2, C5.1, C7.1, L3.1; no longer C3.1
- net at C9.1, L1.2: now also C10.1
- net at C9.2: now also C10.2, C11.2, C12.1, C13.1, L4.1; no longer C10.1
- net at C35.1, L12.2: now also C36.1
- net at C35.2: now also C36.2, C37.2, C38.1, C39.1, L13.1; no longer C36.1
Other:
- moved on the sheet: C10, C2, C3, C35, C36, C9
Changed lines of the file:
@@
 L C_Small C2
 U 1 1 63AA7B73
-P 2700 1150
-F 0 "C2" H 2710 1220 50  0000 L CNN
-F 1 "C2" H 2710 1070 50  0000 L CNN
-F 2 "Capacitors_THT:C_Disc_D5.0mm_W2.5mm_P5.00mm" H 2700 1150 50  0001 C CNN
-F 3 "" H 2700 1150 50  0001 C CNN
-	1    2700 1150
+P 2850 1150
+F 0 "C2" H 2860 1220 50  0000 L CNN
+F 1 "C2" H 2860 1070 50  0000 L CNN
+F 2 "Capacitors_THT:C_Disc_D5.0mm_W2.5mm_P5.00mm" H 2850 1150 50  0001 C CNN
+F 3 "" H 2850 1150 50  0001 C CNN
+	1    2850 1150
 	0    -1   -1   0
 $EndComp
@@
 L C_Small C3
 U 1 1 63AA7C3C
-P 3050 1150
-F 0 "C3" H 3060 1220 50  0000 L CNN
-F 1 "C3" H 3060 1070 50  0000 L CNN
-F 2 "Capacitors_THT:C_Disc_D5.0mm_W2.5mm_P5.00mm" H 3050 1150 50  0001 C CNN
-F 3 "" H 3050 1150 50  0001 C CNN
-	1    3050 1150
+P 2850 900
+F 0 "C3" H 2860 970 50  0000 L CNN
+F 1 "C3" H 2860 820 50  0000 L CNN
+F 2 "Capacitors_THT:C_Disc_D5.0mm_W2.5mm_P5.00mm" H 2850 900 50  0001 C CNN
+F 3 "" H 2850 900 50  0001 C CNN
+	1    2850 900
 	0    -1   -1   0
 $EndComp
@@
 L C_Small C9
 U 1 1 63AE0261
-P 2700 2400
-F 0 "C9" H 2710 2470 50  0000 L CNN
-F 1 "C2" H 2710 2320 50  0000 L CNN
-F 2 "Capacitors_THT:C_Disc_D5.0mm_W2.5mm_P5.00mm" H 2700 2400 50  0001 C CNN
-F 3 "" H 2700 2400 50  0001 C CNN
-	1    2700 2400
+P 2850 2400
+F 0 "C9" H 2860 2470 50  0000 L CNN
+F 1 "C2" H 2860 2320 50  0000 L CNN
+F 2 "Capacitors_THT:C_Disc_D5.0mm_W2.5mm_P5.00mm" H 2850 2400 50  0001 C CNN
+F 3 "" H 2850 2400 50  0001 C CNN
+	1    2850 2400
 	0    -1   -1   0
 $EndComp
@@
 L C_Small C10
 U 1 1 63AE0267
-P 3050 2400
-F 0 "C10" H 3060 2470 50  0000 L CNN
-F 1 "C3" H 3060 2320 50  0000 L CNN
-F 2 "Capacitors_THT:C_Disc_D5.0mm_W2.5mm_P5.00mm" H 3050 2400 50  0001 C CNN
-F 3 "" H 3050 2400 50  0001 C CNN
-	1    3050 2400
+P 2850 2150
+F 0 "C10" H 2860 2220 50  0000 L CNN
+F 1 "C3" H 2860 2070 50  0000 L CNN
+F 2 "Capacitors_THT:C_Disc_D5.0mm_W2.5mm_P5.00mm" H 2850 2150 50  0001 C CNN
+F 3 "" H 2850 2150 50  0001 C CNN
+	1    2850 2150
 	0    -1   -1   0
 $EndComp
@@
 L C_Small C35
 U 1 1 63AE4A98
-P 6200 1100
-F 0 "C35" H 6210 1170 50  0000 L CNN
-F 1 "C2" H 6210 1020 50  0000 L CNN
-F 2 "Capacitors_THT:C_Disc_D5.0mm_W2.5mm_P5.00mm" H 6200 1100 50  0001 C CNN
-F 3 "" H 6200 1100 50  0001 C CNN
-	1    6200 1100
+P 6350 1100
+F 0 "C35" H 6360 1170 50  0000 L CNN
+F 1 "C2" H 6360 1020 50  0000 L CNN
+F 2 "Capacitors_THT:C_Disc_D5.0mm_W2.5mm_P5.00mm" H 6350 1100 50  0001 C CNN
+F 3 "" H 6350 1100 50  0001 C CNN
+	1    6350 1100
 	0    -1   -1   0
 $EndComp
@@
 L C_Small C36
 U 1 1 63AE4A9E
-P 6550 1100
-F 0 "C36" H 6560 1170 50  0000 L CNN
-F 1 "C3" H 6560 1020 50  0000 L CNN
-F 2 "Capacitors_THT:C_Disc_D5.0mm_W2.5mm_P5.00mm" H 6550 1100 50  0001 C CNN
-F 3 "" H 6550 1100 50  0001 C CNN
-	1    6550 1100
+P 6350 850
+F 0 "C36" H 6360 920 50  0000 L CNN
+F 1 "C3" H 6360 770 50  0000 L CNN
+F 2 "Capacitors_THT:C_Disc_D5.0mm_W2.5mm_P5.00mm" H 6350 850 50  0001 C CNN
+F 3 "" H 6350 850 50  0001 C CNN
+	1    6350 850
 	0    -1   -1   0
 $EndComp
@@
 	3250 1100 3450 1100
 Wire Wire Line
-	3150 1150 3250 1150
+	2950 1150 3250 1150
 Wire Wire Line
 	3250 1150 3250 1100
 Wire Wire Line
-	2950 1150 2800 1150
-Wire Wire Line
-	2600 1150 2550 1150
+	2550 1150 2750 1150
 Wire Wire Line
 	3450 750  3500 750
@@
 	3250 2350 3450 2350
 Wire Wire Line
-	3150 2400 3250 2400
+	2950 2400 3250 2400
 Wire Wire Line
 	3250 2400 3250 2350
 Wire Wire Line
-	2950 2400 2800 2400
-Wire Wire Line
-	2600 2400 2550 2400
+	2550 2400 2750 2400
 Wire Wire Line
 	3450 2000 3500 2000
@@
 	6750 1050 6950 1050
 Wire Wire Line
-	6650 1100 6750 1100
+	6450 1100 6750 1100
 Wire Wire Line
 	6750 1100 6750 1050
 Wire Wire Line
-	6450 1100 6300 1100
-Wire Wire Line
-	6100 1100 6050 1100
+	6250 1100 6050 1100
 Wire Wire Line
 	6950 700  7000 700
@@
 	6900 2700 6900 2950
 Connection ~ 6900 2800
+Wire Wire Line
+	2650 2400 2650 2150
+Wire Wire Line
+	2650 2150 2750 2150
+Connection ~ 2650 2400
+Wire Wire Line
+	2950 2150 3050 2150
+Wire Wire Line
+	3050 2150 3050 2400
+Connection ~ 3050 2400
+Wire Wire Line
+	2650 1150 2650 900
+Wire Wire Line
+	2650 900  2750 900
+Connection ~ 2650 1150
+Wire Wire Line
+	2950 900  3050 900
+Wire Wire Line
+	3050 900  3050 1150
+Connection ~ 3050 1150
+Wire Wire Line
+	6150 1100 6150 850
+Wire Wire Line
+	6150 850  6250 850
+Connection ~ 6150 1100
+Wire Wire Line
+	6600 1100 6600 850
+Wire Wire Line
+	6600 850  6450 850
+Connection ~ 6600 1100
 $EndSCHEMATC
