File: RFBitBangerNano/RFBitBangerNano.kicad_pcb (KiCad board)
At the start: 2 copper layers, 152 x 88 mm, 209 parts, among them J1 POWER, J10 si5351mod, J11 SPEAKER, J12 Conn_Coaxial, J13 Conn_01x01, J15 Conn_01x01, J16 Conn_01x01, J17 Filt1, J18 Filt2, J19 Conn_01x20, J2 Barrel_Jack, J20 Conn_01x01, J21 Conn_01x01, J3 Conn_01x01, J4 Conn_01x01, J6 Conn_01x01, J7 Conn_01x01, J8 Conn_01x01, P1 Mini-DIN_6pins_ver4, Q1 2N3904, Q10 2N3904, Q11 2N3904, Q12 2N3904, Q13 SS8550, Q14 2N3904, Q15 NC, Q2 2N3904, Q3 2N7000, Q4 2N3904, Q5 NC, Q6 2N7000, Q7 2N7000, Q8 SS8550, Q9 2N7000, SW2 SW_Push, SW3 SW_Push, SW4 SW_Push, SW5 SW_Push, SW6 SW_Push, T1 Trifilar, T2 Trifilar, T3 Current, T4 Common-Mode Choke, U2 LM7805_TO220, U3 LM386, U4 LM358, U5 LCD1602ExtraPins, U6 SI5351A, Y2 7.X MHz, Y3 27 MHz, Y4 7.X MHz, Y5 7.X MHz

Commit message: Added RFBitBangerNano gerbers
Other:
- board text removed: "ICSP"
Changed lines of the file:
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@@
-    (effects (font (size 1 1) (thickness 0.15)))
-  )
-  (gr_text "1" (at 64.655 73.875) (layer "F.SilkS")
-    (effects (font (size 1 1) (thickness 0.15)))
-  )
-  (gr_text "1" (at 98.53 107.94) (layer "F.SilkS")
     (effects (font (size 1 1) (thickness 0.15)))
   )
@@
     (effects (font (size 1 1) (thickness 0.15)))
   )
-  (gr_text "ICSP" (at 95.11 100.56) (layer "F.SilkS")
-    (effects (font (size 1 1) (thickness 0.15)))
-  )
