File: RFBitBangerNano/RFBitBangerNano.kicad_sch (KiCad schematic)
At the start: 91 parts, among them J1 POWER, J11 SPEAKER, J13 Conn_01x01, J14 Conn_01x01, J15 Conn_01x01, J16 Conn_01x01, J19 Conn_01x20, J2 Barrel_Jack, J20 Conn_01x01, J21 Conn_01x01, J3 Conn_01x01, J4 Conn_01x01, J5 Conn_01x04, J6 Conn_01x01, J7 Conn_01x01, J8 Conn_01x01, J9 ICSP, P1 Mini-DIN_6pins_ver4, Q14 2N3904, Q4 2N3904, SW1 SW_Push, SW2 SW_Push, SW3 SW_Push, SW4 SW_Push, SW5 SW_Push, SW6 SW_Push, T4 Common-Mode Choke, U1 ATMEGA328-PU, U2 LM7805_TO220, U3 LM386, U5 LCD1602ExtraPins, Y1 16 MHz

Commit message: Added RFBitBangerNano
Parts:
- removed C1, C2, C59: 100 nF, Capacitors_THT:C_Disc_D5.0mm_W2.5mm_P2.50mm, symbol RFBitBanger-rescue:C_Small
- removed C4, C5: 100 pF, Capacitors_THT:C_Disc_D5.0mm_W2.5mm_P5.00mm, symbol RFBitBanger-rescue:C_Small
- removed C8, C9: 20 pF, Capacitors_THT:C_Disc_D5.0mm_W2.5mm_P5.00mm, symbol RFBitBanger-rescue:C_Small
- removed D2: 1N4148, Diodes_THT:D_DO-35_SOD27_P7.62mm_Horizontal, symbol RFBitBanger-rescue:D
- removed J14: Conn_01x01, Pin_Headers:Pin_Header_Straight_1x01_Pitch2.54mm, symbol RFBitBanger-rescue:Conn_01x01
- removed J5: Conn_01x04, Pin_Headers:Pin_Header_Straight_1x04_Pitch2.54mm, symbol RFBitBanger-rescue:Conn_01x04
- removed J9: ICSP, Pin_Headers:Pin_Header_Straight_2x03_Pitch2.54mm, symbol RFBitBanger-rescue:Conn_02x03_Odd_Even
- removed JP3: 5VDC, Pin_Headers:Pin_Header_Straight_1x02_Pitch2.54mm, symbol RFBitBanger-rescue:Jumper_NO_Small
- removed L1, L2: 10 uH, Inductors_THT:L_Axial_L6.6mm_D2.7mm_P10.16mm_Horizontal_Vishay_IM-2, symbol RFBitBanger-rescue:L
- removed R1: 10k, Resistors_THT:R_Axial_DIN0207_L6.3mm_D2.5mm_P7.62mm_Horizontal, symbol RFBitBanger-rescue:R
- removed SW1: SW_Push, Buttons_Switches_THT:SW_PUSH_6mm, symbol RFBitBanger-rescue:SW_Push
- removed U1: ATMEGA328-PU, Housings_DIP:DIP-28_W7.62mm_Socket, symbol RFBitBanger-rescue:ATMEGA328-PU
- removed Y1: 16 MHz, Crystals:Crystal_HC49-U_Vertical, symbol RFBitBanger-rescue:Crystal
- added A1: Arduino_Nano_v3.x, Module:Arduino_Nano, symbol MCU_Module:Arduino_Nano_v3.x
- C10, C11, C16, C17, C18, C34, C37, C41, C42, C44, C57, C58, C60, C61, C7: symbol RFBitBanger-rescue:C_Small -> RFBitBangerNano-rescue:C_Small
- C15, C19, C3, C53, C6: symbol RFBitBanger-rescue:CP_Small -> RFBitBangerNano-rescue:CP_Small
- D1: symbol RFBitBanger-rescue:D -> RFBitBangerNano-rescue:D
- D3: symbol RFBitBanger-rescue:LED -> RFBitBangerNano-rescue:LED
- J1, J11: symbol RFBitBanger-rescue:Conn_01x02 -> RFBitBangerNano-rescue:Conn_01x02
- J13, J15, J16, J20, J21, J3, J4, J6, J7, J8: symbol RFBitBanger-rescue:Conn_01x01 -> RFBitBangerNano-rescue:Conn_01x01
- J19: symbol RFBitBanger-rescue:Conn_01x20 -> RFBitBangerNano-rescue:Conn_01x20
- J2: symbol RFBitBanger-rescue:Barrel_Jack -> RFBitBangerNano-rescue:Barrel_Jack
- L10: symbol RFBitBanger-rescue:L -> RFBitBangerNano-rescue:L
- Q14, Q4: symbol RFBitBanger-rescue:2N3904 -> RFBitBangerNano-rescue:2N3904
- R10, R11, R12, R13, R2, R29, R3, R30, R31, R32, R33, R34, R4, R40, R46, R47, R6, R64, R70, R72, R75, R76: symbol RFBitBanger-rescue:R -> RFBitBangerNano-rescue:R
- RV1: footprint RFBitBanger:Potentiometer_Big_Small_Combined -> RFBitBangerNano:Potentiometer_Big_Small_Combined; symbol RFBitBanger-rescue:POT -> RFBitBangerNano-rescue:POT
- RV3: symbol RFBitBanger-rescue:POT -> RFBitBangerNano-rescue:POT
- SW2, SW3, SW4, SW5, SW6: symbol RFBitBanger-rescue:SW_Push -> RFBitBangerNano-rescue:SW_Push
- T4: footprint RFBitBanger:DoubleWindingTransformer -> RFBitBangerNano:DoubleWindingTransformer
- U2: symbol RFBitBanger-rescue:LM7805_TO220 -> RFBitBangerNano-rescue:LM7805_TO220
- U3: symbol RFBitBanger-rescue:LM386 -> RFBitBangerNano-rescue:LM386
Connections:
- net +5V: now also A1.27 (+5V)
- net AUDIOFILT: now also A1.19 (A0)
- net BEEPOUT: now also A1.6 (D3)
- net DB4: now also A1.8 (D5)
- net DB5: now also A1.9 (D6)
- net DB6: now also A1.10 (D7)
- net DB7: now also A1.11 (D8)
- net E: now also A1.21 (A2)
- net GND: now also A1.29 (GND), A1.4 (GND)
- net MICPADDLE: now also A1.20 (A1)
- net MISO: now also A1.15 (D12)
- net MOSI: now also A1.14 (D11)
- net MUTEAUDIO: now also A1.7 (D4)
- net PS2CLK: now also A1.5 (D2)
- net RESET: now also A1.28 (~{RESET})
- net RS: now also A1.22 (A3)
- net RXD: now also A1.2 (D0/RX)
- net SCK: now also A1.16 (D13)
- net SCL: now also A1.24 (A5)
- net SDA: now also A1.23 (A4)
- net TRANSMIT: now also A1.12 (D9)
- net TUNING: now also A1.13 (D10)
- net TXD: now also A1.1 (D1/TX)
- net at C57.1: now also A1.18 (AREF)
Other:
- sheet RFBitBangerRadio renamed RFBitBangerNanoRadio
- sheet RFBitBangerNanoRadio: file RFBitBangerRadio.kicad_sch -> RFBitBangerNanoRadio.kicad_sch
- note added: "RFBitBangerNano 20m to 80m BAND DRAFT V5 BY KW4TI"
- note removed: "RFBITBANGER 20m to 80m BAND DRAFT V5 BY KW4TI"
- moved on the sheet: C57, C7
