File: RFBitBangerNano/RFBitBangerNanoRadio.kicad_sch (KiCad schematic)
At the start: 135 parts, among them J10 si5351mod, J12 Conn_Coaxial, J17 Filt1, J18 Filt2, Q1 2N3904, Q10 2N3904, Q11 2N3904, Q12 2N3904, Q13 SS8550, Q15 NC, Q2 2N3904, Q3 2N7000, Q5 NC, Q6 2N7000, Q7 2N7000, Q8 SS8550, Q9 2N7000, T1 Trifilar, T2 Trifilar, T3 Current, U4 LM358, U6 SI5351A, Y2 7.X MHz, Y3 27 MHz, Y4 7.X MHz, Y5 7.X MHz

Commit message: Added RFBitBangerNano
Parts:
- C12, C14, C36, C39, C40, C49, C50, C52: symbol RFBitBanger-rescue:CP_Small -> RFBitBangerNano-rescue:CP_Small
- C13, C20, C21, C22, C23, C24, C25, C26, C27, C30, C32, C33, C35, C38, C43, C45, C46, C47, C48, C51, C54, C55, C56: symbol RFBitBanger-rescue:C_Small -> RFBitBangerNano-rescue:C_Small
- D10, D11, D12, D13, D14, D15, D17, D18, D4, D5, D8, D9: symbol RFBitBanger-rescue:D -> RFBitBangerNano-rescue:D
- D16, D19: symbol RFBitBanger-rescue:LED -> RFBitBangerNano-rescue:LED
- D6: symbol RFBitBanger-rescue:D_Zener -> RFBitBangerNano-rescue:D_Zener
- J10: symbol RFBitBanger-rescue:Conn_01x07 -> RFBitBangerNano-rescue:Conn_01x07
- J12: footprint RFBitBanger:bnc_90_1-1337543-0_pad_combo -> RFBitBangerNano:bnc_90_1-1337543-0_pad_combo; symbol RFBitBanger-rescue:Conn_Coaxial -> RFBitBangerNano-rescue:Conn_Coaxial
- J17, J18: symbol RFBitBanger-rescue:Conn_01x04 -> RFBitBangerNano-rescue:Conn_01x04
- JP1, JP2, JP8: symbol RFBitBanger-rescue:Jumper_NC_Small -> RFBitBangerNano-rescue:Jumper_NC_Small
- JP4: symbol RFBitBanger-rescue:Jumper_NO_Small -> RFBitBangerNano-rescue:Jumper_NO_Small
- JP5, JP7: symbol RFBitBanger-rescue:Jumper_NC_Dual -> RFBitBangerNano-rescue:Jumper_NC_Dual
- L11, L3, L5, L9: symbol RFBitBanger-rescue:L -> RFBitBangerNano-rescue:L
- L4, L6: footprint RFBitBanger:SmallVerticalToroid -> RFBitBangerNano:SmallVerticalToroid; symbol RFBitBanger-rescue:L -> RFBitBangerNano-rescue:L
- Q1, Q10, Q11, Q12, Q2: symbol RFBitBanger-rescue:2N3904 -> RFBitBangerNano-rescue:2N3904
- Q13, Q8: symbol RFBitBanger-rescue:2N3906 -> RFBitBangerNano-rescue:2N3906
- Q15: symbol RFBitBanger-rescue:IRF540N -> RFBitBangerNano-rescue:IRF540N
- Q3, Q5, Q6, Q7, Q9: symbol RFBitBanger-rescue:2N7000 -> RFBitBangerNano-rescue:2N7000
- R14, R15, R16, R17, R18, R19, R20, R21, R22, R23, R24, R25, R26, R27, R28, R35, R36, R37, R38, R39, R41, R48, R49, R5, R50, R51, R52, R53, R54, R55, R56, R57, R58, R59, R60, R61, R62, R63, R65, R66, R67, R68, R7, R71, R73, R74, R8, R9: symbol RFBitBanger-rescue:R -> RFBitBangerNano-rescue:R
- RLY1: footprint RFBitBanger:G2VRelay -> RFBitBangerNano:G2VRelay
- RV2: footprint RFBitBanger:Potentiometer_Big_Small_Combined -> RFBitBangerNano:Potentiometer_Big_Small_Combined; symbol RFBitBanger-rescue:POT -> RFBitBangerNano-rescue:POT
- RV4: symbol RFBitBanger-rescue:POT -> RFBitBangerNano-rescue:POT
- T1, T2: footprint RFBitBanger:TripleWindingTransformerRef -> RFBitBangerNano:TripleWindingTransformerRef
- T3: footprint RFBitBanger:SamplingTransformer -> RFBitBangerNano:SamplingTransformer
- U4: symbol RFBitBanger-rescue:LM358 -> RFBitBangerNano-rescue:LM358
- Y2, Y3, Y4, Y5: symbol RFBitBanger-rescue:Crystal -> RFBitBangerNano-rescue:Crystal
Other:
- moved on the sheet: C54

Commit message: Added two dual capacitor footprints to RFBitBanger
Parts:
- C26, C32: footprint Capacitors_THT:C_Disc_D5.0mm_W2.5mm_P5.00mm -> RFBitBangerNano:C_Disc_D5.0mm_W2.5mm_P5.00mm_Dual
Changed lines of the file:
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@@
       (effects (font (size 1.27 1.27)) (justify left))
     )
-    (property "Footprint" "Capacitors_THT:C_Disc_D5.0mm_W2.5mm_P5.00mm" (id 2) (at 213.36 132.08 0)
+    (property "Footprint" "RFBitBangerNano:C_Disc_D5.0mm_W2.5mm_P5.00mm_Dual" (id 2) (at 213.36 132.08 0)
       (effects (font (size 1.27 1.27)) hide)
     )
@@
       (effects (font (size 1.27 1.27)) (justify left))
     )
-    (property "Footprint" "Capacitors_THT:C_Disc_D5.0mm_W2.5mm_P5.00mm" (id 2) (at 262.89 66.04 0)
-      (effects (font (size 1.27 1.27)) hide)
-    )
+    (property "Footprint" "RFBitBangerNano:C_Disc_D5.0mm_W2.5mm_P5.00mm_Dual" (id 2) (at 262.89 66.04 0)
+      (effects (font (size 1.27 1.27)) hide)
+    )

Commit message: Fixed problems with manual, added filters
Parts:
- R38: value 33R -> 2R2
Changed lines of the file:
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@@
     (in_bom yes) (on_board yes)
     (property "Reference" "R38" (id 0) (at 248.92 43.18 90))
-    (property "Value" "33R" (id 1) (at 246.38 43.18 90))
+    (property "Value" "2R2" (id 1) (at 246.38 43.18 90))
     (property "Footprint" "Resistors_THT:R_Axial_DIN0207_L6.3mm_D2.5mm_P7.62mm_Horizontal" (id 2) (at 248.158 43.18 90)
       (effects (font (size 1.27 1.27)) hide)
