File: SerialResonantFilter/SerialResonantFilter.kicad_sch (KiCad schematic)
At the start: 11 parts, among them J1 OUT, J2 INP

Commit message: Made capacitors on board dual footprint
Parts:
- C1, C2, C3, C4, C5, C6, C7: footprint Capacitors_THT:C_Disc_D5.0mm_W2.5mm_P5.00mm -> SerialResonantFilter:C_Disc_D5.0mm_W2.5mm_P5.00mm_Dual
Changed lines of the file:
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@@
       (effects (font (size 1.27 1.27)) (justify left))
     )
-    (property "Footprint" "Capacitors_THT:C_Disc_D5.0mm_W2.5mm_P5.00mm" (id 2) (at 59.69 34.29 0)
+    (property "Footprint" "SerialResonantFilter:C_Disc_D5.0mm_W2.5mm_P5.00mm_Dual" (id 2) (at 59.69 34.29 0)
       (effects (font (size 1.27 1.27)) hide)
     )
@@
       (effects (font (size 1.27 1.27)) (justify left))
     )
-    (property "Footprint" "Capacitors_THT:C_Disc_D5.0mm_W2.5mm_P5.00mm" (id 2) (at 72.39 29.21 0)
+    (property "Footprint" "SerialResonantFilter:C_Disc_D5.0mm_W2.5mm_P5.00mm_Dual" (id 2) (at 72.39 29.21 0)
       (effects (font (size 1.27 1.27)) hide)
     )
@@
       (effects (font (size 1.27 1.27)) (justify left))
     )
-    (property "Footprint" "Capacitors_THT:C_Disc_D5.0mm_W2.5mm_P5.00mm" (id 2) (at 72.39 22.86 0)
+    (property "Footprint" "SerialResonantFilter:C_Disc_D5.0mm_W2.5mm_P5.00mm_Dual" (id 2) (at 72.39 22.86 0)
       (effects (font (size 1.27 1.27)) hide)
     )
@@
       (effects (font (size 1.27 1.27)) (justify left))
     )
-    (property "Footprint" "Capacitors_THT:C_Disc_D5.0mm_W2.5mm_P5.00mm" (id 2) (at 85.09 34.29 0)
+    (property "Footprint" "SerialResonantFilter:C_Disc_D5.0mm_W2.5mm_P5.00mm_Dual" (id 2) (at 85.09 34.29 0)
       (effects (font (size 1.27 1.27)) hide)
     )
@@
       (effects (font (size 1.27 1.27)) (justify left))
     )
-    (property "Footprint" "Capacitors_THT:C_Disc_D5.0mm_W2.5mm_P5.00mm" (id 2) (at 100.33 34.29 0)
+    (property "Footprint" "SerialResonantFilter:C_Disc_D5.0mm_W2.5mm_P5.00mm_Dual" (id 2) (at 100.33 34.29 0)
       (effects (font (size 1.27 1.27)) hide)
     )
@@
       (effects (font (size 1.27 1.27)) (justify left))
     )
-    (property "Footprint" "Capacitors_THT:C_Disc_D5.0mm_W2.5mm_P5.00mm" (id 2) (at 91.44 24.13 0)
+    (property "Footprint" "SerialResonantFilter:C_Disc_D5.0mm_W2.5mm_P5.00mm_Dual" (id 2) (at 91.44 24.13 0)
       (effects (font (size 1.27 1.27)) hide)
     )
@@
       (effects (font (size 1.27 1.27)) (justify left))
     )
-    (property "Footprint" "Capacitors_THT:C_Disc_D5.0mm_W2.5mm_P5.00mm" (id 2) (at 91.44 19.05 0)
+    (property "Footprint" "SerialResonantFilter:C_Disc_D5.0mm_W2.5mm_P5.00mm_Dual" (id 2) (at 91.44 19.05 0)
       (effects (font (size 1.27 1.27)) hide)
     )
@@
     )
     (path "/00000000-0000-0000-0000-000063aa79da"
-      (reference "C1") (unit 1) (value "C1") (footprint "Capacitors_THT:C_Disc_D5.0mm_W2.5mm_P5.00mm")
+      (reference "C1") (unit 1) (value "C1") (footprint "SerialResonantFilter:C_Disc_D5.0mm_W2.5mm_P5.00mm_Dual")
     )
     (path "/00000000-0000-0000-0000-000063aa7b73"
-      (reference "C2") (unit 1) (value "C2") (footprint "Capacitors_THT:C_Disc_D5.0mm_W2.5mm_P5.00mm")
+      (reference "C2") (unit 1) (value "C2") (footprint "SerialResonantFilter:C_Disc_D5.0mm_W2.5mm_P5.00mm_Dual")
     )
     (path "/00000000-0000-0000-0000-000063aa7c3c"
-      (reference "C3") (unit 1) (value "C3") (footprint "Capacitors_THT:C_Disc_D5.0mm_W2.5mm_P5.00mm")
+      (reference "C3") (unit 1) (value "C3") (footprint "SerialResonantFilter:C_Disc_D5.0mm_W2.5mm_P5.00mm_Dual")
     )
     (path "/00000000-0000-0000-0000-000063aa7cef"
-      (reference "C4") (unit 1) (value "C4") (footprint "Capacitors_THT:C_Disc_D5.0mm_W2.5mm_P5.00mm")
+      (reference "C4") (unit 1) (value "C4") (footprint "SerialResonantFilter:C_Disc_D5.0mm_W2.5mm_P5.00mm_Dual")
     )
     (path "/00000000-0000-0000-0000-000063aa7ebd"
-      (reference "C5") (unit 1) (value "C5") (footprint "Capacitors_THT:C_Disc_D5.0mm_W2.5mm_P5.00mm")
+      (reference "C5") (unit 1) (value "C5") (footprint "SerialResonantFilter:C_Disc_D5.0mm_W2.5mm_P5.00mm_Dual")
     )
     (path "/00000000-0000-0000-0000-000063aa7db8"
-      (reference "C6") (unit 1) (value "C6") (footprint "Capacitors_THT:C_Disc_D5.0mm_W2.5mm_P5.00mm")
+      (reference "C6") (unit 1) (value "C6") (footprint "SerialResonantFilter:C_Disc_D5.0mm_W2.5mm_P5.00mm_Dual")
     )
     (path "/00000000-0000-0000-0000-000063abc991"
-      (reference "C7") (unit 1) (value "C7") (footprint "Capacitors_THT:C_Disc_D5.0mm_W2.5mm_P5.00mm")
+      (reference "C7") (unit 1) (value "C7") (footprint "SerialResonantFilter:C_Disc_D5.0mm_W2.5mm_P5.00mm_Dual")
     )
     (path "/00000000-0000-0000-0000-000063abbf6f"
