File: RFBitBangSMT/RFBitBangSMT.kicad_pcb (KiCad board)
At the start: 2 copper layers, 152 x 88 mm, 258 parts, among them J1 POWER, J10 si5351mod, J11 AudioJack2_Dual_Ground_Switch, J12 Conn_Coaxial, J13 Conn_01x01, J14 Conn_01x01, J15 Conn_01x01, J16 Conn_01x01, J17 Filt1, J18 Filt2, J19 AudioJack2_Dual_Ground_Switch, J2 Barrel_Jack, J20 Conn_01x01, J21 Conn_01x01, J3 Conn_01x01, J4 Conn_01x01, J5 Conn_01x04, J6 Conn_01x01, J7 Conn_01x01, J8 AudioJack2_Dual_Ground_Switch, J9 ICSP, P1 Mini-DIN_6pins_ver4, Q1 MMBT3904, Q10 MMBT3904, Q11 MMBT3904, Q12 MMBT3904, Q13 SS8550, Q14 MMBT3904, Q15 NC, Q16 SS8550, Q2 MMBT3904, Q3 2N7000, Q4 MMBT3904, Q5 NC, Q6 2N7000, Q7 2N7000, Q8 SS8550, Q9 2N7000, SW1 SW_Push, SW2 SW_Push, SW3 SW_Push, SW4 SW_Push, SW5 SW_Push, SW6 SW_Push, T1 Trifilar, T2 Trifilar, T3 Current, T4 Common-Mode Choke, U1 ATmega328P-A, U2 LM78M05_TO252, U3 LM386, U4 LM358, U5 LM358, U6 SI5351A, Y1 16 MHz, Y2 7.X MHz, Y3 25 MHz, Y4 7.X MHz, Y5 7.X MHz

Commit message: Tested with JLCPCB but not fabricated
Parts:
- C32: value 33 pF -> NC

Commit message: Minor fixes to SMT
Parts:
- added C70: 100 nF, Capacitor_SMD:C_0805_2012Metric_Pad1.18x1.45mm_HandSolder, F.Cu at (90.1, 70.2)
- moved J15 21.6 mm to (134.1, 126.2)
- moved J17 2.54 mm to (154.9, 120.7)
- moved J18 2.54 mm to (154.9, 141.0)
- moved SW2 2.46 mm to (70.6, 126.1)
- moved T3 2.30 mm to (175.9, 141.0)
- moved SW5 2.25 mm to (70.6, 133.9)
- moved J10 1.41 mm to (141.1, 70.8)
- moved D16 1.36 mm to (178.8, 132.4), turned to -90 degrees
- moved R65 1.13 mm to (144.8, 69.9)
- moved R63 0.34 mm to (131.5, 119.4)
- moved D11 0.30 mm to (157.9, 105.8)
Connections:
- L12 pad 2: Net-(C67-Pad2) -> Net-(C68-Pad2)
- L8 pad 2: Net-(C68-Pad2) -> Net-(C67-Pad2)
Routing:
- net GND: track 254.6 -> 341.5 mm, vias 93 -> 132
- net Net-(C67-Pad2): track 16.9 -> 24.6 mm
- net Net-(C16-Pad2): track 50.7 -> 46.3 mm
- net +5V: track 538.8 -> 543.1 mm
- net Net-(C68-Pad2): track 7.45 -> 11.0 mm
- net Net-(C17-Pad2): track 44.5 -> 47.6 mm
- net Net-(C19-Pad1): track 61.4 -> 58.5 mm
- net Net-(D16-Pad1): track 2.10 -> 4.97 mm
- net Net-(D16-Pad2): track 4.07 -> 6.62 mm
- net Net-(C26-Pad2): track 15.9 -> 18.4 mm
- net SCL: track 82.2 -> 84.6 mm
- net SDA: track 83.4 -> 85.8 mm
- net Net-(J12-Pad1): track 22.5 -> 24.5 mm
- net Net-(C11-Pad2): track 55.1 -> 57.1 mm
- net Net-(C14-Pad1): track 68.0 -> 69.9 mm
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
Commit message: Some more minor SMT fixed
Parts:
- added R86: 1k, Resistor_SMD:R_0805_2012Metric_Pad1.20x1.40mm_HandSolder, F.Cu at (77.8, 89.1)
- moved C32 4.79 mm to (170.7, 95.5), turned to 0 degrees
- moved C2 3.64 mm to (47.0, 81.8)
- moved J19 1.52 mm to (38.9, 117.6)
- moved J11 1.45 mm to (39.0, 130.7)
- moved C5 1.27 mm to (45.2, 84.8)
- moved D15 0.83 mm to (173.4, 60.0)
- moved Q14 0.77 mm to (104.1, 75.5)
- moved R72 0.69 mm to (107.4, 75.4)
- moved L7 0.67 mm to (53.4, 141.8)
- moved C58 0.59 mm to (45.1, 67.1), turned to 180 degrees
- moved C62 0.56 mm to (50.9, 140.8)
- moved D11 0.37 mm to (158.0, 106.1)
- moved J8 0.26 mm to (61.0, 143.5)
- moved C36 0.25 mm to (39.9, 141.0)
- moved R42 0.25 mm to (40.7, 137.9)
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Connections:
- D19 pad 2: +12V -> Net-(C31-Pad2)
- R80 pad 1: SCK -> Net-(R80-Pad1)
- R82 pad 2: SCK -> Net-(R80-Pad1)
Routing:
- net SCK: track 75.9 -> 36.8 mm
- net Net-(R80-Pad1): track 0.00 -> 37.9 mm
- net TRANSMIT: track 75.0 -> 41.6 mm, vias 2 -> 0
- net Net-(C23-Pad2): track 74.0 -> 88.5 mm
- net +12V: track 299.0 -> 290.5 mm
- net Net-(C58-Pad1): track 41.9 -> 49.1 mm
- net Net-(C31-Pad2): track 130.7 -> 137.1 mm
- net RESET: track 103.5 -> 108.6 mm
- net Net-(C2-Pad2): track 12.6 -> 8.09 mm
- net Net-(C58-Pad2): track 25.1 -> 28.6 mm
- net DB7: track 59.8 -> 63.2 mm
- net +5V: track 543.1 -> 546.2 mm
- net Net-(C10-Pad2): track 49.3 -> 52.1 mm
- net Net-(C11-Pad2): track 57.1 -> 59.5 mm
- net AMPOUT: track 99.7 -> 101.7 mm
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
Commit message: Added Low Pass Filter
Parts:
- moved R71 0.44 mm to (164.6, 60.2)
- moved D19 0.41 mm to (160.9, 59.2)
- moved R38 0.40 mm to (168.9, 60.2)

Commit message: JLCPCB order
Changed lines of the file:
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@@
     (fp_arc (start 0.20066 22.9997) (mid -0.153162 22.853142) (end -0.29972 22.49932) (layer "F.SilkS") (width 0.12))
     (fp_arc (start 63.7 8) (mid 64.053553 8.146447) (end 64.2 8.5) (layer "F.SilkS") (width 0.12))
-    (fp_arc (start 64.20104 22.49932) (mid 64.054479 22.85315) (end 63.70066 22.9997) (layer "F.SilkS") (width 0.12))
+    (fp_arc (start 64.20104 22.49932) (mid 64.054473 22.853115) (end 63.70066 22.9997) (layer "F.SilkS") (width 0.12))
     (fp_arc (start -0.29972 8.49884) (mid -0.153162 8.145018) (end 0.20066 7.99846) (layer "F.SilkS") (width 0.12))
     (fp_line (start -8.25 -2.75) (end 72.25 -2.75) (layer "F.CrtYd") (width 0.05))
@@
     (fp_line (start -1 0.625) (end -1 -0.625) (layer "F.Fab") (width 0.1))
     (fp_line (start 1 0.625) (end -1 0.625) (layer "F.Fab") (width 0.1))
-    (pad "1" smd roundrect (at -1.0375 0 90) (size 1.175 1.45) (layers "F.Cu" "F.Paste" "F.Mask") (roundrect_rratio 0.212766)
+    (pad "1" smd roundrect (at -1.0375 0 90) (size 1.175 1.45) (layers "F.Cu" "F.Paste" "F.Mask") (roundrect_rratio 0.2127659574)
       (net 2 "GND") (pintype "passive"))
-    (pad "2" smd roundrect (at 1.0375 0 90) (size 1.175 1.45) (layers "F.Cu" "F.Paste" "F.Mask") (roundrect_rratio 0.212766)
+    (pad "2" smd roundrect (at 1.0375 0 90) (size 1.175 1.45) (layers "F.Cu" "F.Paste" "F.Mask") (roundrect_rratio 0.2127659574)
       (net 1 "+5V") (pintype "passive"))
     (model "${KICAD6_3DMODEL_DIR}/Capacitor_SMD.3dshapes/C_0805_2012Metric.wrl"
@@
     (fp_line (start -1 0.625) (end -1 -0.625) (layer "F.Fab") (width 0.1))
     (fp_line (start -1 -0.625) (end 1 -0.625) (layer "F.Fab") (width 0.1))
-    (pad "1" smd roundrect (at -1 0) (size 1.2 1.4) (layers "F.Cu" "F.Paste" "F.Mask") (roundrect_rratio 0.208333)
+    (pad "1" smd roundrect (at -1 0) (size 1.2 1.4) (layers "F.Cu" "F.Paste" "F.Mask") (roundrect_rratio 0.2083333333)
       (net 163 "Net-(R80-Pad1)") (pintype "passive"))
-    (pad "2" smd roundrect (at 1 0) (size 1.2 1.4) (layers "F.Cu" "F.Paste" "F.Mask") (roundrect_rratio 0.208333)
+    (pad "2" smd roundrect (at 1 0) (size 1.2 1.4) (layers "F.Cu" "F.Paste" "F.Mask") (roundrect_rratio 0.2083333333)
       (net 17 "SCK") (pintype "passive"))
     (model "${KICAD6_3DMODEL_DIR}/Resistor_SMD.3dshapes/R_0805_2012Metric.wrl"

Commit message: A few minor fixes to SMT
Parts:
- added J22: Conn_01x02, Connector_PinHeader_2.54mm:PinHeader_1x02_P2.54mm_Vertical, F.Cu at (58.4, 118.6)
- L10: value FB -> 100 uH; footprint Inductor_SMD:L_0805_2012Metric_Pad1.15x1.40mm_HandSolder -> Inductor_THT:L_Axial_L6.6mm_D2.7mm_P10.16mm_Horizontal_Vishay_IM-2
- moved L10 10.9 mm to (95.8, 121.9), turned to -90 degrees
- moved C61 9.73 mm to (94.2, 116.6)
- moved C53 5.33 mm to (102.9, 116.3), turned to 180 degrees
- moved C63 5.01 mm to (56.9, 113.8)
- moved C67 4.67 mm to (54.4, 113.8)
- moved L12 4.11 mm to (55.6, 109.5)
- moved C37 3.45 mm to (105.9, 128.8), turned to 90 degrees
- moved C41 3.32 mm to (99.8, 129.3)
- moved L8 2.03 mm to (55.6, 106.4), turned to 0 degrees
- moved R43 1.48 mm to (60.5, 112.8)
- moved R69 1.40 mm to (64.0, 112.8)
Routing:
- net Net-(L10-Pad1): track 5.16 -> 22.2 mm
- net +12V: track 290.5 -> 297.3 mm
- net SPKR: track 23.1 -> 29.4 mm
- net Net-(C68-Pad2): track 11.7 -> 7.41 mm
- net Net-(L12-Pad1): track 50.8 -> 46.9 mm
- net Net-(C63-Pad1): track 26.9 -> 30.1 mm
- net Net-(C61-Pad2): track 35.5 -> 32.6 mm
- net Net-(C67-Pad2): track 24.2 -> 22.0 mm
- net Net-(C63-Pad2): track 2.21 -> 3.99 mm
- net GND: track 342.8 -> 344.4 mm
- net Net-(L8-Pad1): track 3.93 -> 2.30 mm
- net Net-(C19-Pad1): track 58.5 -> 59.8 mm
- net Net-(JP6-Pad2): track 9.98 -> 9.44 mm
- net Net-(C66-Pad1): track 21.4 -> 20.9 mm

Commit message: Added heatsink pad for Q16 RFBitBangSMT
Parts:
- added J23: Conn_01x01, MountingHole:MountingHole_3.2mm_M3, F.Cu at (159.5, 67.6)
- moved C38 9.82 mm to (147.1, 73.1), turned to -90 degrees
- moved C24 8.54 mm to (164.5, 64.5)
- moved C29 8.13 mm to (166.7, 64.5)
- moved Q8 7.82 mm to (174.2, 64.5)
- moved C14 6.87 mm to (168.9, 64.5)
- moved C23 6.43 mm to (162.2, 90.5), turned to 90 degrees
- moved R39 6.21 mm to (178.7, 64.7)
- moved C53 5.89 mm to (103.6, 122.2)
- moved Q13 5.85 mm to (183.2, 66.0)
- moved C61 5.73 mm to (93.0, 122.2), turned to -90 degrees
- moved L6 5.26 mm to (163.8, 82.9)
- moved R8 4.67 mm to (171.1, 64.5), turned to 90 degrees
- moved D8 4.12 mm to (187.2, 69.0), turned to -90 degrees
- moved R51 4.00 mm to (166.5, 90.8)
- moved Q9 3.30 mm to (167.6, 95.2)
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Routing:
- net GND: track 344.4 -> 392.3 mm, vias 132 -> 150
- net Net-(C14-Pad1): track 69.9 -> 78.2 mm
- net +12V: track 297.3 -> 291.1 mm
- net Net-(C14-Pad2): track 34.3 -> 28.3 mm
- net Net-(C31-Pad2): track 137.5 -> 141.8 mm
- net Net-(C23-Pad2): track 88.5 -> 92.7 mm
- net AMPOUT: track 101.7 -> 105.8 mm
- net Net-(Q12-Pad1): track 4.94 -> 8.71 mm
- net Net-(Q9-Pad2): track 14.4 -> 18.1 mm
- net Net-(D18-Pad1): track 26.5 -> 29.4 mm
- net Net-(C38-Pad1): track 14.9 -> 17.5 mm
- net Net-(L10-Pad1): track 22.2 -> 19.8 mm
- net TXRELAY: track 40.7 -> 38.4 mm
- net Net-(D19-Pad1): track 2.76 -> 5.04 mm
- net Net-(D15-Pad2): track 10.4 -> 12.5 mm
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