File: RFBitBangSMT/RFBitBangSMT.kicad_pcb (KiCad board)
At the start: 2 copper layers, 152 x 88 mm, 262 parts, among them J1 POWER, J10 si5351mod, J11 AudioJack2_Dual_Ground_Switch, J12 Conn_Coaxial, J13 Conn_01x01, J14 Conn_01x01, J15 Conn_01x01, J16 Conn_01x01, J17 Filt1, J18 Filt2, J19 AudioJack2_Dual_Ground_Switch, J2 Barrel_Jack, J20 Conn_01x01, J21 Conn_01x01, J22 Conn_01x02, J23 Conn_01x01, J3 Conn_01x01, J4 Conn_01x01, J5 Conn_01x04, J6 Conn_01x01, J7 Conn_01x01, J8 AudioJack2_Dual_Ground_Switch, J9 ICSP, P1 Mini-DIN_6pins_ver4, Q1 MMBT3904, Q10 MMBT3904, Q11 MMBT3904, Q12 MMBT3904, Q13 SS8550, Q14 MMBT3904, Q15 NC, Q16 SS8550, Q2 MMBT3904, Q3 2N7000, Q4 MMBT3904, Q5 NC, Q6 2N7000, Q7 2N7000, Q8 SS8550, Q9 2N7000, SW1 SW_Push, SW2 SW_Push, SW3 SW_Push, SW4 SW_Push, SW5 SW_Push, SW6 SW_Push, T1 Trifilar, T2 Trifilar, T3 Current, T4 Common-Mode Choke, U1 ATmega328P-A, U2 LM78M05_TO252, U3 LM386, U4 LM358, U5 LM358, U6 SI5351A, Y1 16 MHz, Y2 7.X MHz, Y3 25 MHz, Y4 7.X MHz, Y5 7.X MHz

Commit message: Removed SMT Q8
Parts:
- removed Q16: SS8550, Package_TO_SOT_THT:TO-92_Inline_Wide
- Q8: footprint Package_TO_SOT_SMD:SOT-23 -> Package_TO_SOT_THT:TO-92_Inline_Wide
- moved Q8 11.0 mm to (165.6, 71.4), turned to -90 degrees
- moved C14 4.26 mm to (173.2, 64.8), turned to 0 degrees
- moved C29 3.07 mm to (169.7, 65.1), turned to 90 degrees
- moved R8 2.86 mm to (173.2, 62.5), turned to 0 degrees
- moved C24 2.40 mm to (166.8, 65.1), turned to -90 degrees
- moved C55 2.18 mm to (146.3, 88.4)
- moved R39 0.41 mm to (179.0, 64.9)
Connections:
- Q8 pad 1: Net-(C14-Pad2) -> Net-(C31-Pad2)
- Q8 pad 2: Net-(C31-Pad2) -> Net-(C14-Pad2)
Routing:
- net Net-(C14-Pad2): track 28.3 -> 41.9 mm
- net Net-(C14-Pad1): track 78.2 -> 69.9 mm
- net Net-(C31-Pad2): track 141.8 -> 134.4 mm

Commit message: Updated documentation
Parts:
- moved R14 1.89 mm to (152.5, 70.7)
- moved Q12 1.72 mm to (149.6, 70.6)
- moved L11 1.38 mm to (147.1, 66.5)
- moved D18 1.20 mm to (150.5, 73.8)
- moved C38 1.11 mm to (146.0, 73.2)
- moved C46 0.84 mm to (148.8, 63.0)
- moved C24 0.64 mm to (167.5, 65.1)
- moved R49 0.28 mm to (147.6, 77.4)
- moved R50 0.12 mm to (147.6, 80.8)
Routing:
- net Net-(C14-Pad2): track 41.9 -> 46.1 mm
- net Net-(C38-Pad1): track 17.5 -> 19.7 mm
- net Net-(Q12-Pad1): track 8.71 -> 10.3 mm
- net Net-(L11-Pad2): track 6.83 -> 5.54 mm
- net Net-(D18-Pad1): track 29.4 -> 30.5 mm
- net Net-(J10-Pad1): track 16.9 -> 17.9 mm
- net PLLOSC: track 7.85 -> 6.87 mm
- net GND: track 391.8 -> 392.7 mm
- net Net-(C14-Pad1): track 69.9 -> 69.3 mm
- net Net-(D18-Pad2): track 2.92 -> 2.30 mm
- net Net-(J10-Pad2): track 15.7 -> 16.2 mm

Commit message: Fixed problems with manual, added filters
Parts:
- added C71: NC, Capacitor_SMD:C_0805_2012Metric_Pad1.18x1.45mm_HandSolder, F.Cu at (101.6, 140.0)
- R38: value 22R -> 2R2
- moved C60 7.34 mm to (108.7, 135.1), turned to 90 degrees
- moved C15 2.38 mm to (96.0, 138.0)
- moved R11 1.16 mm to (95.8, 134.6)
- moved R31 0.55 mm to (108.7, 131.3)
Connections:
- U3 pad 1: unconnected-(U3-Pad1) -> Net-(C71-Pad1)
- U3 pad 8: unconnected-(U3-Pad8) -> Net-(C71-Pad2)
Routing:
- net Net-(C60-Pad2): track 48.2 -> 39.1 mm
- net Net-(RV1-Pad2): track 30.7 -> 35.9 mm
- net Net-(C71-Pad1): track 0.00 -> 4.38 mm
- net Net-(C15-Pad1): track 7.81 -> 4.24 mm
- net Net-(C71-Pad2): track 0.00 -> 3.32 mm
- net Net-(D3-Pad2): track 33.9 -> 36.2 mm
- net Net-(C19-Pad1): track 59.8 -> 58.2 mm
- net Net-(C34-Pad2): track 38.2 -> 39.8 mm
- net Net-(C34-Pad1): track 8.20 -> 8.81 mm

Commit message: Manufactured RFBitBangSMT
Parts:
- added JP10: BTP, Connector_PinHeader_2.54mm:PinHeader_1x02_P2.54mm_Vertical, F.Cu at (138.4, 65.5)
- C49, C50, C52: footprint Capacitor_SMD:C_0805_2012Metric_Pad1.18x1.45mm_HandSolder -> Capacitor_THT:CP_Radial_D5.0mm_P2.50mm
- D1: value 1N4007 -> 1N4745A
- D6: value D_Zener -> 1N4757
- moved C36 36.6 mm to (76.4, 142.5), turned to 180 degrees
- moved C41 35.0 mm to (64.9, 126.9), turned to 90 degrees
- moved L7 27.1 mm to (54.9, 114.7)
- moved R42 23.6 mm to (54.8, 119.0), turned to 90 degrees
- moved J15 14.9 mm to (135.0, 141.0)
- moved R22 12.2 mm to (145.4, 110.5), turned to 90 degrees
- moved C50 8.66 mm to (132.1, 126.2), turned to -90 degrees
- moved C44 7.27 mm to (52.3, 71.8), turned to 0 degrees
- moved C42 6.47 mm to (57.8, 72.7), turned to 0 degrees
- moved JP9 6.45 mm to (83.5, 108.2)
- moved JP6 6.35 mm to (73.7, 108.1), turned to 90 degrees
- moved R43 5.80 mm to (66.1, 111.4)
- moved C58 5.38 mm to (39.9, 65.8), turned to -90 degrees
- moved RV4 5.35 mm to (143.0, 65.3), turned to -90 degrees
- moved C63 5.22 mm to (62.0, 112.7), turned to 0 degrees
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Connections:
- C49 pad 1: Net-(C43-Pad1) -> Net-(C49-Pad1)
- C49 pad 2: Net-(C49-Pad2) -> Net-(C43-Pad1)
- Q1 pad 2: Net-(C49-Pad2) -> Net-(C49-Pad1)
- R22 pad 1: Net-(C49-Pad2) -> Net-(C49-Pad1)
Routing:
- net GND: track 393.2 -> 517.3 mm, vias 150 -> 227
- net Net-(C63-Pad1): track 30.1 -> 7.00 mm
- net Net-(C62-Pad2): track 20.4 -> 34.6 mm
- net +5V: track 546.2 -> 557.4 mm
- net Net-(JP6-Pad2): track 9.44 -> 19.4 mm
- net Net-(C49-Pad1): track 0.00 -> 8.27 mm
- net Net-(C39-Pad1): track 51.9 -> 43.6 mm
- net Net-(C31-Pad2): track 134.6 -> 142.7 mm
- net Net-(C49-Pad2): track 6.00 -> 0.00 mm
- net +12V: track 291.4 -> 296.6 mm
- net Net-(C19-Pad1): track 58.2 -> 53.5 mm
- net IF: track 34.3 -> 29.7 mm
- net Net-(JP10-Pad2): track 5.54 -> 9.89 mm
- net Net-(C58-Pad1): track 49.1 -> 45.1 mm
- net Net-(JP9-Pad2): track 13.1 -> 17.1 mm
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Other:
- board text added: "12-14V"
- board text added: "BYP"
- board text added: "CONTRAST"
- board text added: "CURRENT SENSE BYPASS"
- board text added: "FILT BYPASS"
- board text added: "FLT"
- board text added: "ICSP PWR"
- board text added: "KEY/PTT"
- board text added: "MIC/ LINE IN"
- board text added: "PA BIAS (2-2.5V NOMINAL)"
- board text added: "PIN +"
- board text added: "PLL"
- board text added: "QSK"
- board text added: "RFBitBanger V9 SMT BY DANIEL MARKS KW4TI CC-BY-SA 4.0"
- board text added: "SPKR"
- board text added: "XTAL OFF"
- board text added: "XTL"
- board text removed: "CENTER PIN+"
- board text removed: "KEY/PADDLE/ PTT"
- board text removed: "MIC/LINE IN"
- board text removed: "PWR+"
- board text removed: "RFBitBanger V8 SMT BY DANIEL MARKS KW4TI CC-BY-SA 4.0"

Commit message: Added TCXO option to RFBitBanger SMT
Parts:
- added C72: 100 nF, Capacitor_SMD:C_0805_2012Metric_Pad1.18x1.45mm_HandSolder, F.Cu at (126.0, 79.6)
- added R87: 470R, Resistor_THT:R_Axial_DIN0207_L6.3mm_D2.5mm_P7.62mm_Horizontal, F.Cu at (129.5, 79.2)
- moved Y3 0.48 mm to (125.9, 75.5)
Connections:
- Y3 pad 2: unconnected-(Y3-Pad2) -> GND
- Y3 pad 4: unconnected-(Y3-Pad4) -> Net-(C72-Pad2)
Routing:
- net SCL: track 84.7 -> 91.5 mm
- net Net-(C72-Pad2): track 0.00 -> 6.33 mm
- net Net-(C47-Pad2): track 30.6 -> 35.0 mm
- net GND: track 517.3 -> 520.1 mm, vias 227 -> 229
- net SDA: track 86.0 -> 87.7 mm
- net Net-(U6-Pad3): track 5.45 -> 4.86 mm
Other:
- board text added: "RFBitBanger V10 SMT BY DANIEL MARKS KW4TI CC-BY-SA 4.0"
- board text removed: "RFBitBanger V9 SMT BY DANIEL MARKS KW4TI CC-BY-SA 4.0"

Commit message: Added cut slots around crystal
Parts:
- added H1: MountingHole, RFBitBangSMT:CutSlot, F.Cu at (125.7, 80.0)
- added H2: MountingHole, RFBitBangSMT:CutSlot, F.Cu at (128.7, 73.7)
- added H3: MountingHole, RFBitBangSMT:CutSlot, F.Cu at (125.8, 71.3)
- added H4: MountingHole, RFBitBangSMT:CutSlot, F.Cu at (128.6, 77.7)
- added H5: MountingHole, RFBitBangSMT:CutSlot, F.Cu at (122.7, 75.7)
- R87: value 470R -> NC
- Y3: footprint Crystal:Crystal_SMD_3225-4Pin_3.2x2.5mm_HandSoldering -> Crystal:Crystal_SMD_3225-4Pin_3.2x2.5mm
- moved L9 1.88 mm to (117.0, 70.9)
- moved D14 1.57 mm to (124.6, 67.5)
- moved C72 1.55 mm to (125.8, 78.1)
- moved R87 1.09 mm to (130.5, 78.8)
- moved Y3 0.67 mm to (125.6, 74.9)
Routing:
- net SDA: track 87.7 -> 91.6 mm
- net Net-(C72-Pad2): track 6.33 -> 9.68 mm
- net Net-(C47-Pad2): track 35.0 -> 38.1 mm
- net Net-(L9-Pad2): track 25.9 -> 28.2 mm
- net TRANSMIT: track 41.6 -> 39.7 mm
- net GND: track 520.1 -> 519.5 mm
- net Net-(U6-Pad2): track 9.32 -> 9.86 mm
- net SCL: vias 0 -> 2
