File: RFBitBangSMT/RFBitBangSMT.kicad_pcb (KiCad board)
At the start: 2 copper layers, 152 x 88 mm, 270 parts, among them J1 POWER, J10 si5351mod, J11 AudioJack2_Dual_Ground_Switch, J12 Conn_Coaxial, J13 Conn_01x01, J14 Conn_01x01, J15 Conn_01x01, J16 Conn_01x01, J17 Filt1, J18 Filt2, J19 AudioJack2_Dual_Ground_Switch, J2 Barrel_Jack, J20 Conn_01x01, J21 Conn_01x01, J22 Conn_01x02, J23 Conn_01x01, J3 Conn_01x01, J4 Conn_01x01, J5 Conn_01x04, J6 Conn_01x01, J7 Conn_01x01, J8 AudioJack2_Dual_Ground_Switch, J9 ICSP, P1 Mini-DIN_6pins_ver4, Q1 MMBT3904, Q10 MMBT3904, Q11 MMBT3904, Q12 MMBT3904, Q13 SS8550, Q14 MMBT3904, Q15 NC, Q2 MMBT3904, Q3 2N7000, Q4 MMBT3904, Q5 NC, Q6 2N7000, Q7 2N7000, Q8 SS8550, Q9 2N7000, SW1 SW_Push, SW2 SW_Push, SW3 SW_Push, SW4 SW_Push, SW5 SW_Push, SW6 SW_Push, T1 Trifilar, T2 Trifilar, T3 Current, T4 Common-Mode Choke, U1 ATmega328P-A, U2 LM78M05_TO252, U3 LM386, U4 LM358, U5 LM358, U6 SI5351A, Y1 16 MHz, Y2 7.X MHz, Y3 25 MHz, Y4 7.X MHz, Y5 7.X MHz

Commit message: Batch 2 test PCBs
Parts:
- removed C72: 100 nF, Capacitor_SMD:C_0805_2012Metric_Pad1.18x1.45mm_HandSolder
- removed R87: NC, Resistor_THT:R_Axial_DIN0207_L6.3mm_D2.5mm_P7.62mm_Horizontal
- R79: value 100k -> 22k
- moved H3 1.33 mm to (125.0, 72.4)
- moved H1 1.21 mm to (125.0, 79.0)
- moved Y3 1.02 mm to (126.0, 75.8)
- moved H2 0.76 mm to (128.9, 73.0)
- moved H4 0.39 mm to (129.0, 77.7)
- moved H5 0.34 mm to (123.0, 75.7)
Connections:
- Y3 pad 2: GND -> unconnected-(Y3-Pad2)
- Y3 pad 4: Net-(C72-Pad2) -> unconnected-(Y3-Pad4)
Routing:
- net Net-(C72-Pad2): track 9.68 -> 0.00 mm
- net SDA: track 91.6 -> 85.5 mm
- net SCL: track 91.5 -> 85.8 mm, vias 2 -> 0
- net Net-(C47-Pad2): track 38.1 -> 33.4 mm
- net Net-(U6-Pad2): track 9.86 -> 7.27 mm
- net GND: track 519.5 -> 517.3 mm, vias 229 -> 227
Other:
- board text added: "Crystal Frequency"
- board text added: "Serial Number"

Commit message: Moved PLLBoard to its own project
Parts:
- added C72: 100 nF, Capacitor_SMD:C_0805_2012Metric_Pad1.18x1.45mm_HandSolder, F.Cu at (126.3, 77.7)
- added J25: Conn_01x01, Connector_PinHeader_2.00mm:PinHeader_1x01_P2.00mm_Vertical, F.Cu at (129.2, 68.1)
- added JP11: TCXO, Jumper:SolderJumper-2_P1.3mm_Open_Pad1.0x1.5mm, F.Cu at (120.5, 72.1)
- moved R70 1.63 mm to (116.1, 66.7)
- moved H3 1.39 mm to (125.2, 71.0)
- moved H2 1.36 mm to (129.6, 71.8)
- moved Y3 1.35 mm to (126.4, 74.6)
- moved L9 1.15 mm to (116.9, 69.8)
- moved H1 0.93 mm to (125.2, 79.9)
- moved U6 0.54 mm to (134.0, 75.2)
- moved H4 0.39 mm to (129.4, 77.7)
- moved H5 0.37 mm to (123.4, 75.6)
Connections:
- Y3 pad 2: unconnected-(Y3-Pad2) -> GND
- Y3 pad 4: unconnected-(Y3-Pad4) -> Net-(C72-Pad2)
Routing:
- net GND: track 517.3 -> 529.8 mm, vias 227 -> 229
- net Net-(C72-Pad2): track 0.00 -> 9.06 mm
- net +5V: track 557.4 -> 554.7 mm, vias 16 -> 14
- net Net-(U6-Pad2): track 7.27 -> 8.84 mm
- net Net-(C47-Pad2): track 33.4 -> 34.9 mm
- net Net-(J10-Pad1): track 17.9 -> 16.6 mm
- net SDA: track 85.5 -> 86.6 mm
- net Net-(U6-Pad3): track 5.46 -> 4.73 mm
- net MISO: track 52.5 -> 51.8 mm
- net Net-(L9-Pad2): track 28.2 -> 28.9 mm
- net Net-(J10-Pad2): track 16.2 -> 15.6 mm
Other:
- board text added: "PA BIAS (2-2.8V NOMINAL)"
- board text removed: "PA BIAS (2-2.5V NOMINAL)"
