File: RFBitBangSMT/RFBitBangSMT.kicad_sch (KiCad schematic)
At the start: 120 parts, among them J1 POWER, J11 AudioJack2_Dual_Ground_Switch, J13 Conn_01x01, J14 Conn_01x01, J15 Conn_01x01, J16 Conn_01x01, J19 AudioJack2_Dual_Ground_Switch, J2 Barrel_Jack, J20 Conn_01x01, J21 Conn_01x01, J3 Conn_01x01, J4 Conn_01x01, J5 Conn_01x04, J6 Conn_01x01, J7 Conn_01x01, J8 AudioJack2_Dual_Ground_Switch, J9 ICSP, P1 Mini-DIN_6pins_ver4, Q14 MMBT3904, Q4 MMBT3904, SW1 SW_Push, SW2 SW_Push, SW3 SW_Push, SW4 SW_Push, SW5 SW_Push, SW6 SW_Push, T4 Common-Mode Choke, U1 ATmega328P-A, U2 LM78M05_TO252, U3 LM386, U5 LM358, Y1 16 MHz

Commit message: Tested with JLCPCB but not fabricated
Parts:
- U3: LCSC C5157706 -> C383071
Changed lines of the file:
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@@
       (effects (font (size 1.27 1.27)) hide)
     )
-    (property "LCSC" "C5157706" (id 4) (at 220.98 102.235 0)
+    (property "LCSC" "C383071" (id 4) (at 220.98 102.235 0)
       (effects (font (size 1.524 1.524)) hide)
     )
@@
     )
     (path "/00000000-0000-0000-0000-000061b53775/00000000-0000-0000-0000-000061bd962e"
-      (reference "C32") (unit 1) (value "33 pF") (footprint "Capacitor_SMD:C_0805_2012Metric_Pad1.18x1.45mm_HandSolder")
+      (reference "C32") (unit 1) (value "NC") (footprint "Capacitor_SMD:C_0805_2012Metric_Pad1.18x1.45mm_HandSolder")
     )
     (path "/00000000-0000-0000-0000-000061b53775/00000000-0000-0000-0000-0000615ae388"

Commit message: Minor fixes to SMT
Parts:
- added C70: 100 nF, Capacitor_SMD:C_0805_2012Metric_Pad1.18x1.45mm_HandSolder, symbol RFBitBangSMT-rescue:C_Small
Connections:
- net +5V: now also C70.2
- net GND: now also C70.1
- net at C68.2, J19.S1: now also L12.2; no longer L8.2
- net at C67.2, J19.T1: now also L8.2; no longer L12.2
Other:
- moved on the sheet: R83
Changed lines of the file:
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@@
   (junction (at 31.115 67.945) (diameter 0) (color 0 0 0 0)
   )
+  (junction (at 102.87 25.4) (diameter 0) (color 0 0 0 0)
+  )
   (junction (at 229.235 39.37) (diameter 0) (color 0 0 0 0)
   )
@@
   (junction (at 134.62 148.59) (diameter 0) (color 0 0 0 0)
   )
+  (junction (at 102.87 41.91) (diameter 0) (color 0 0 0 0)
+  )
   (junction (at 270.51 132.08) (diameter 0) (color 0 0 0 0)
   )
@@
   (junction (at 270.51 124.46) (diameter 0) (color 0 0 0 0)
   )
+  (junction (at 236.22 30.48) (diameter 0) (color 0 0 0 0)
+  )
   (junction (at 204.47 57.785) (diameter 0) (color 0 0 0 0)
   )
@@
   (junction (at 31.115 60.325) (diameter 0) (color 0 0 0 0)
   )
-  (junction (at 242.57 25.4) (diameter 0) (color 0 0 0 0)
-  )
   (junction (at 230.505 55.245) (diameter 0) (color 0 0 0 0)
   )
@@
   (junction (at 222.885 64.135) (diameter 0) (color 0 0 0 0)
   )
+  (junction (at 269.24 60.96) (diameter 0) (color 0 0 0 0)
+  )
   (junction (at 274.32 52.705) (diameter 0) (color 0 0 0 0)
   )
@@
   (junction (at 185.42 40.64) (diameter 0) (color 0 0 0 0)
   )
-  (junction (at 269.24 63.5) (diameter 0) (color 0 0 0 0)
+  (junction (at 242.57 30.48) (diameter 0) (color 0 0 0 0)
   )
   (junction (at 252.73 60.96) (diameter 0) (color 0 0 0 0)
@@
   (junction (at 134.62 81.28) (diameter 0) (color 0 0 0 0)
   )
-  (junction (at 236.22 30.48) (diameter 0) (color 0 0 0 0)
-  )
   (junction (at 213.995 57.785) (diameter 0) (color 0 0 0 0)
   )
@@
     (stroke (width 0) (type default) (color 0 0 0 0))
   )
-  (wire (pts (xy 261.62 63.5) (xy 260.35 63.5))
-    (stroke (width 0) (type default) (color 0 0 0 0))
-  )
   (wire (pts (xy 189.23 78.105) (xy 195.58 78.105))
     (stroke (width 0) (type default) (color 0 0 0 0))
@@
     (stroke (width 0) (type default) (color 0 0 0 0))
   )
-  (wire (pts (xy 106.68 25.4) (xy 95.25 25.4))
+  (wire (pts (xy 106.68 25.4) (xy 102.87 25.4))
     (stroke (width 0) (type default) (color 0 0 0 0))
   )
@@
     (stroke (width 0) (type default) (color 0 0 0 0))
   )
+  (wire (pts (xy 260.35 60.96) (xy 261.62 60.96))
+    (stroke (width 0) (type default) (color 0 0 0 0))
+  )
   (wire (pts (xy 194.31 86.995) (xy 195.58 86.995))
     (stroke (width 0) (type default) (color 0 0 0 0))
   )
+  (wire (pts (xy 236.22 24.13) (xy 245.11 24.13))
+    (stroke (width 0) (type default) (color 0 0 0 0))
+  )
   (wire (pts (xy 90.17 179.07) (xy 90.17 180.34))
     (stroke (width 0) (type default) (color 0 0 0 0))
@@
     (stroke (width 0) (type default) (color 0 0 0 0))
   )
+  (wire (pts (xy 102.87 25.4) (xy 95.25 25.4))
+    (stroke (width 0) (type default) (color 0 0 0 0))
+  )
   (wire (pts (xy 30.48 27.94) (xy 33.02 27.94))
     (stroke (width 0) (type default) (color 0 0 0 0))
@@
     (stroke (width 0) (type default) (color 0 0 0 0))
   )
+  (wire (pts (xy 260.35 63.5) (xy 260.35 60.96))
+    (stroke (width 0) (type default) (color 0 0 0 0))
+  )
   (wire (pts (xy 270.51 109.22) (xy 270.51 116.84))
     (stroke (width 0) (type default) (color 0 0 0 0))
@@
     (stroke (width 0) (type default) (color 0 0 0 0))
   )
+  (wire (pts (xy 102.87 25.4) (xy 102.87 29.845))
+    (stroke (width 0) (type default) (color 0 0 0 0))
+  )
   (wire (pts (xy 93.98 95.25) (xy 93.98 97.79))
     (stroke (width 0) (type default) (color 0 0 0 0))
@@
     (stroke (width 0) (type default) (color 0 0 0 0))
   )
-  (wire (pts (xy 236.22 32.385) (xy 236.22 30.48))
-    (stroke (width 0) (type default) (color 0 0 0 0))
-  )
   (wire (pts (xy 218.44 88.265) (xy 231.14 88.265))
     (stroke (width 0) (type default) (color 0 0 0 0))
@@
     (stroke (width 0) (type default) (color 0 0 0 0))
   )
-  (wire (pts (xy 269.24 63.5) (xy 269.24 67.31))
+  (wire (pts (xy 269.24 60.96) (xy 269.24 67.31))
     (stroke (width 0) (type default) (color 0 0 0 0))
   )
@@
     (stroke (width 0) (type default) (color 0 0 0 0))
   )
-  (wire (pts (xy 242.57 25.4) (xy 245.11 25.4))
-    (stroke (width 0) (type default) (color 0 0 0 0))
-  )
   (wire (pts (xy 93.98 83.82) (xy 97.79 83.82))
     (stroke (width 0) (type default) (color 0 0 0 0))
@@
     (stroke (width 0) (type default) (color 0 0 0 0))
   )
-  (wire (pts (xy 242.57 32.385) (xy 242.57 25.4))
+  (wire (pts (xy 242.57 32.385) (xy 242.57 30.48))
     (stroke (width 0) (type default) (color 0 0 0 0))
   )
@@
     (stroke (width 0) (type default) (color 0 0 0 0))
   )
+  (wire (pts (xy 236.22 30.48) (xy 236.22 32.385))
+    (stroke (width 0) (type default) (color 0 0 0 0))
+  )
   (wire (pts (xy 206.375 48.26) (xy 244.475 48.26))
     (stroke (width 0) (type default) (color 0 0 0 0))
@@
     (stroke (width 0) (type default) (color 0 0 0 0))
   )
+  (wire (pts (xy 102.87 41.91) (xy 106.68 41.91))
+    (stroke (width 0) (type default) (color 0 0 0 0))
+  )
   (wire (pts (xy 230.505 55.245) (xy 230.505 62.23))
     (stroke (width 0) (type default) (color 0 0 0 0))
@@
     (stroke (width 0) (type default) (color 0 0 0 0))
   )
+  (wire (pts (xy 102.87 34.925) (xy 102.87 41.91))
+    (stroke (width 0) (type default) (color 0 0 0 0))
+  )
   (polyline (pts (xy 166.37 53.34) (xy 16.51 53.34))
     (stroke (width 0) (type default) (color 0 0 0 0))
@@
     (stroke (width 0) (type default) (color 0 0 0 0))
   )
-  (wire (pts (xy 236.22 30.48) (xy 245.11 30.48))
-    (stroke (width 0) (type default) (color 0 0 0 0))
-  )
   (wire (pts (xy 128.27 86.36) (xy 125.73 86.36))
     (stroke (width 0) (type default) (color 0 0 0 0))
@@
     (stroke (width 0) (type default) (color 0 0 0 0))
   )
+  (wire (pts (xy 242.57 30.48) (xy 242.57 25.4))
+    (stroke (width 0) (type default) (color 0 0 0 0))
+  )
   (wire (pts (xy 213.995 57.785) (xy 215.265 57.785))
     (stroke (width 0) (type default) (color 0 0 0 0))
@@
     (stroke (width 0) (type default) (color 0 0 0 0))
   )
-  (wire (pts (xy 269.24 52.705) (xy 269.24 63.5))
+  (wire (pts (xy 269.24 52.705) (xy 269.24 60.96))
     (stroke (width 0) (type default) (color 0 0 0 0))
   )
@@
     (stroke (width 0) (type default) (color 0 0 0 0))
   )
+  (wire (pts (xy 245.11 24.13) (xy 245.11 25.4))
+    (stroke (width 0) (type default) (color 0 0 0 0))
+  )
   (wire (pts (xy 74.93 158.75) (xy 74.93 161.29))
     (stroke (width 0) (type default) (color 0 0 0 0))
@@
     (stroke (width 0) (type default) (color 0 0 0 0))
   )
+  (wire (pts (xy 236.22 24.13) (xy 236.22 30.48))
+    (stroke (width 0) (type default) (color 0 0 0 0))
+  )
   (wire (pts (xy 226.06 93.345) (xy 231.14 93.345))
     (stroke (width 0) (type default) (color 0 0 0 0))
@@
     (stroke (width 0) (type default) (color 0 0 0 0))
   )
-  (wire (pts (xy 95.25 41.91) (xy 106.68 41.91))
+  (wire (pts (xy 95.25 41.91) (xy 102.87 41.91))
     (stroke (width 0) (type default) (color 0 0 0 0))
   )
@@
     (stroke (width 0) (type default) (color 0 0 0 0))
   )
+  (wire (pts (xy 242.57 30.48) (xy 245.11 30.48))
+    (stroke (width 0) (type default) (color 0 0 0 0))
+  )
   (wire (pts (xy 95.25 33.02) (xy 91.44 33.02))
     (stroke (width 0) (type default) (color 0 0 0 0))
@@
   (symbol (lib_id "RFBitBangSMT-rescue:C_Small") (at 266.065 67.31 90) (unit 1)
     (in_bom yes) (on_board yes)
-    (property "Reference" "C69" (id 0) (at 264.16 66.04 90)
+    (property "Reference" "C69" (id 0) (at 267.97 64.135 90)
       (effects (font (size 1.27 1.27)) (justify left))
     )
@@
   (symbol (lib_id "RFBitBangSMT-rescue:C_Small") (at 227.33 67.31 90) (unit 1)
     (in_bom yes) (on_board yes)
-    (property "Reference" "C66" (id 0) (at 225.425 66.04 90)
+    (property "Reference" "C66" (id 0) (at 229.235 64.77 90)
       (effects (font (size 1.27 1.27)) (justify left))
     )
@@
     (pin "2")
   )
+  (symbol (lib_id "RFBitBangSMT-rescue:C_Small") (at 102.87 32.385 180) (unit 1)
+    (in_bom yes) (on_board yes)
+    (property "Reference" "C70" (id 0) (at 101.6 31.115 0)
+      (effects (font (size 1.27 1.27)) (justify left))
+    )
+    (property "Value" "100 nF" (id 1) (at 105.41 27.305 0)
+      (effects (font (size 1.27 1.27)) (justify left))
+    )
+    (property "Footprint" "Capacitor_SMD:C_0805_2012Metric_Pad1.18x1.45mm_HandSolder" (id 2) (at 102.87 32.385 0)
+      (effects (font (size 1.27 1.27)) hide)
+    )
+    (property "Datasheet" "" (id 3) (at 102.87 32.385 0)
+      (effects (font (size 1.27 1.27)) hide)
+    )
+    (property "LCSC" "C49678" (id 4) (at 102.87 32.385 0)
+      (effects (font (size 1.524 1.524)) hide)
+    )
+    (pin "1")
+    (pin "2")
+  )
   (symbol (lib_id "RFBitBangSMT-rescue:C_Small") (at 181.61 43.18 180) (unit 1)
     (in_bom yes) (on_board yes)
@@
     (pin "2")
   )
-  (symbol (lib_id "RFBitBangSMT-rescue:R") (at 265.43 63.5 270) (mirror x) (unit 1)
+  (symbol (lib_id "RFBitBangSMT-rescue:R") (at 265.43 60.96 270) (mirror x) (unit 1)
     (in_bom yes) (on_board yes)
-    (property "Reference" "R83" (id 0) (at 265.43 60.96 90))
-    (property "Value" "100k" (id 1) (at 265.43 63.5 90))
-    (property "Footprint" "Resistor_SMD:R_0805_2012Metric_Pad1.20x1.40mm_HandSolder" (id 2) (at 265.43 65.278 90)
+    (property "Reference" "R83" (id 0) (at 265.43 58.42 90))
+    (property "Value" "100k" (id 1) (at 265.43 60.96 90))
+    (property "Footprint" "Resistor_SMD:R_0805_2012Metric_Pad1.20x1.40mm_HandSolder" (id 2) (at 265.43 62.738 90)
       (effects (font (size 1.27 1.27)) hide)
     )
-    (property "Datasheet" "" (id 3) (at 265.43 63.5 0)
+    (property "Datasheet" "" (id 3) (at 265.43 60.96 0)
       (effects (font (size 1.27 1.27)) hide)
     )
-    (property "LCSC" "C149504" (id 4) (at 265.43 63.5 90)
+    (property "LCSC" "C149504" (id 4) (at 265.43 60.96 90)
       (effects (font (size 1.524 1.524)) hide)
     )
@@
       (reference "C69") (unit 1) (value "100 pF") (footprint "Capacitor_SMD:C_0805_2012Metric_Pad1.18x1.45mm_HandSolder")
     )
+    (path "/c2552891-e2c9-4b18-82ac-174a4f812b0c"
+      (reference "C70") (unit 1) (value "100 nF") (footprint "Capacitor_SMD:C_0805_2012Metric_Pad1.18x1.45mm_HandSolder")
+    )
     (path "/00000000-0000-0000-0000-0000615b9029"
