File: RFBitBangSMT/RFBitBangSMT.kicad_sch (KiCad schematic)
At the start: 125 parts, among them J1 POWER, J11 AudioJack2_Dual_Ground_Switch, J13 Conn_01x01, J14 Conn_01x01, J15 Conn_01x01, J16 Conn_01x01, J19 AudioJack2_Dual_Ground_Switch, J2 Barrel_Jack, J20 Conn_01x01, J21 Conn_01x01, J22 Conn_01x02, J23 Conn_01x01, J3 Conn_01x01, J4 Conn_01x01, J5 Conn_01x04, J6 Conn_01x01, J7 Conn_01x01, J8 AudioJack2_Dual_Ground_Switch, J9 ICSP, P1 Mini-DIN_6pins_ver4, Q14 MMBT3904, Q4 MMBT3904, SW1 SW_Push, SW2 SW_Push, SW3 SW_Push, SW4 SW_Push, SW5 SW_Push, SW6 SW_Push, T4 Common-Mode Choke, U1 ATmega328P-A, U2 LM78M05_TO252, U3 LM386, U5 LM358, Y1 16 MHz

Commit message: Batch 2 test PCBs
Parts:
- J13, J23: now left out of the parts list
- R79: value 100k -> 22k; LCSC C149504 -> C17560
Changed lines of the file:
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@@
   )
   (symbol (lib_id "RFBitBangSMT-rescue:Conn_01x01") (at 280.67 158.75 0) (unit 1)
-    (in_bom yes) (on_board yes)
+    (in_bom no) (on_board yes)
     (property "Reference" "J13" (id 0) (at 280.67 156.21 0))
     (property "Value" "Conn_01x01" (id 1) (at 280.67 161.29 0))
@@
     (in_bom yes) (on_board yes)
     (property "Reference" "R79" (id 0) (at 247.65 53.213 90))
-    (property "Value" "100k" (id 1) (at 247.65 55.245 90))
+    (property "Value" "22k" (id 1) (at 247.65 55.245 90))
     (property "Footprint" "Resistor_SMD:R_0805_2012Metric_Pad1.20x1.40mm_HandSolder" (id 2) (at 247.65 57.023 90)
       (effects (font (size 1.27 1.27)) hide)
@@
       (effects (font (size 1.27 1.27)) hide)
     )
-    (property "LCSC" "C149504" (id 4) (at 247.65 55.245 90)
+    (property "LCSC" "C17560" (id 4) (at 247.65 55.245 90)
       (effects (font (size 1.524 1.524)) hide)
     )
@@
   )
   (symbol (lib_id "RFBitBangSMT-rescue:Conn_01x01") (at 280.035 149.86 0) (unit 1)
-    (in_bom yes) (on_board yes)
+    (in_bom no) (on_board yes)
     (property "Reference" "J23" (id 0) (at 280.035 147.32 0))
     (property "Value" "Conn_01x01" (id 1) (at 280.035 152.4 0))
@@
       (reference "#PWR0114") (unit 1) (value "GND") (footprint "")
     )
-    (path "/00000000-0000-0000-0000-000061b53775/68d5e815-716f-42ad-92f1-33c0a4ecbd9b"
-      (reference "#PWR0115") (unit 1) (value "GND") (footprint "")
-    )
-    (path "/00000000-0000-0000-0000-000061b53775/55529ebf-472b-4343-a525-ad54ec009f40"
-      (reference "#PWR0116") (unit 1) (value "GND") (footprint "")
-    )
     (path "/00000000-0000-0000-0000-0000615917e6"
       (reference "C1") (unit 1) (value "100 nF") (footprint "Capacitor_SMD:C_0805_2012Metric_Pad1.18x1.45mm_HandSolder")
@@
       (reference "C71") (unit 1) (value "NC") (footprint "Capacitor_SMD:C_0805_2012Metric_Pad1.18x1.45mm_HandSolder")
     )
-    (path "/00000000-0000-0000-0000-000061b53775/511d8b43-bd62-4118-be0a-e7bfbcb4d955"
-      (reference "C72") (unit 1) (value "100 nF") (footprint "Capacitor_SMD:C_0805_2012Metric_Pad1.18x1.45mm_HandSolder")
-    )
     (path "/00000000-0000-0000-0000-0000615b9029"
       (reference "D1") (unit 1) (value "1N4745A") (footprint "Diode_THT:D_DO-41_SOD81_P7.62mm_Horizontal")
@@
     )
     (path "/85fa61fd-91bd-4c21-a338-cf4f66942d8b"
-      (reference "R79") (unit 1) (value "100k") (footprint "Resistor_SMD:R_0805_2012Metric_Pad1.20x1.40mm_HandSolder")
+      (reference "R79") (unit 1) (value "22k") (footprint "Resistor_SMD:R_0805_2012Metric_Pad1.20x1.40mm_HandSolder")
     )
     (path "/b1f914c4-7562-41ac-9463-d926890ed957"
@@
       (reference "R86") (unit 1) (value "1k") (footprint "Resistor_SMD:R_0805_2012Metric_Pad1.20x1.40mm_HandSolder")
     )
-    (path "/00000000-0000-0000-0000-000061b53775/27935f41-b08c-4eb0-b491-8fb61581495d"
-      (reference "R87") (unit 1) (value "NC") (footprint "Resistor_THT:R_Axial_DIN0207_L6.3mm_D2.5mm_P7.62mm_Horizontal")
-    )
     (path "/00000000-0000-0000-0000-000061b53775/00000000-0000-0000-0000-00006183a50a"
