File: RFBitBangSMT/RFBitBangSMTRadio.kicad_sch (KiCad schematic)
At the start: 138 parts, among them J10 si5351mod, J12 Conn_Coaxial, J17 Filt1, J18 Filt2, Q1 MMBT3904, Q10 MMBT3904, Q11 MMBT3904, Q12 MMBT3904, Q13 SS8550, Q15 NC, Q16 SS8550, Q2 MMBT3904, Q3 2N7000, Q5 NC, Q6 2N7000, Q7 2N7000, Q8 SS8550, Q9 2N7000, T1 Trifilar, T2 Trifilar, T3 Current, U4 LM358, U6 SI5351A, Y2 7.X MHz, Y3 25 MHz, Y4 7.X MHz, Y5 7.X MHz

Commit message: Tested with JLCPCB but not fabricated
Parts:
- C32: value 33 pF -> NC
- D17: LCSC (none) -> C81598
Changed lines of the file:
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@@
       (effects (font (size 1.27 1.27)) hide)
+    )
+    (property "LCSC" "C81598" (id 4) (at 207.01 74.93 0)
+      (effects (font (size 1.524 1.524)) hide)
     )
     (pin "1")
@@
       (effects (font (size 1.27 1.27)) (justify left))
     )
-    (property "Value" "33 pF" (id 1) (at 260.35 68.58 90)
-      (effects (font (size 1.27 1.27)) (justify left))
-    )
+    (property "Value" "NC" (id 1) (at 260.35 68.58 90)
+      (effects (font (size 1.27 1.27)) (justify left))
+    )

Commit message: Some more minor SMT fixed
Connections:
- net +12V: no longer D19.2 (A)
- net at C31.2, C46.2, C55.2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: now also D19.2 (A)
Changed lines of the file:
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@@
   (junction (at 44.45 52.07) (diameter 0) (color 0 0 0 0)
   )
+  (junction (at 187.96 16.51) (diameter 0) (color 0 0 0 0)
+  )
   (junction (at 81.28 187.96) (diameter 0) (color 0 0 0 0)
   )
@@
     (stroke (width 0) (type default) (color 0 0 0 0))
   )
+  (wire (pts (xy 187.96 16.51) (xy 187.96 17.78))
+    (stroke (width 0) (type default) (color 0 0 0 0))
+  )
   (wire (pts (xy 137.16 118.11) (xy 137.16 125.73))
     (stroke (width 0) (type default) (color 0 0 0 0))
@@
     (stroke (width 0) (type default) (color 0 0 0 0))
   )
-  (wire (pts (xy 182.88 21.59) (xy 182.88 17.78))
-    (stroke (width 0) (type default) (color 0 0 0 0))
-  )
   (wire (pts (xy 129.54 163.83) (xy 130.81 163.83))
     (stroke (width 0) (type default) (color 0 0 0 0))
@@
     (stroke (width 0) (type default) (color 0 0 0 0))
   )
-  (wire (pts (xy 69.85 16.51) (xy 215.9 16.51))
+  (wire (pts (xy 69.85 16.51) (xy 187.96 16.51))
     (stroke (width 0) (type default) (color 0 0 0 0))
   )
@@
     (stroke (width 0) (type default) (color 0 0 0 0))
   )
-  (wire (pts (xy 182.88 17.78) (xy 187.96 17.78))
-    (stroke (width 0) (type default) (color 0 0 0 0))
-  )
   (wire (pts (xy 44.45 116.84) (xy 44.45 123.19))
     (stroke (width 0) (type default) (color 0 0 0 0))
@@
     (stroke (width 0) (type default) (color 0 0 0 0))
   )
-  (wire (pts (xy 179.07 21.59) (xy 182.88 21.59))
-    (stroke (width 0) (type default) (color 0 0 0 0))
-  )
   (wire (pts (xy 223.52 26.67) (xy 226.06 26.67))
     (stroke (width 0) (type default) (color 0 0 0 0))
@@
     (stroke (width 0) (type default) (color 0 0 0 0))
   )
+  (wire (pts (xy 187.96 16.51) (xy 215.9 16.51))
+    (stroke (width 0) (type default) (color 0 0 0 0))
+  )
   (wire (pts (xy 44.45 68.58) (xy 44.45 67.31))
     (stroke (width 0) (type default) (color 0 0 0 0))
@@
     (pin "2")
   )
-  (symbol (lib_id "RFBitBangSMT-rescue:+12V") (at 179.07 21.59 0) (unit 1)
-    (in_bom yes) (on_board yes)
-    (property "Reference" "#PWR094" (id 0) (at 179.07 25.4 0)
-      (effects (font (size 1.27 1.27)) hide)
-    )
-    (property "Value" "+12V" (id 1) (at 179.07 18.034 0))
-    (property "Footprint" "" (id 2) (at 179.07 21.59 0)
-      (effects (font (size 1.27 1.27)) hide)
-    )
-    (property "Datasheet" "" (id 3) (at 179.07 21.59 0)
-      (effects (font (size 1.27 1.27)) hide)
-    )
-    (pin "1")
-  )
   (symbol (lib_id "RFBitBangSMT-rescue:C_Small") (at 20.32 177.8 180) (unit 1)

Commit message: A few minor fixes to SMT
Parts:
- C33: LCSC C49678 -> C1710
Changed lines of the file:
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@@
       (effects (font (size 1.27 1.27)) hide)
     )
-    (property "LCSC" "C49678" (id 4) (at 160.02 177.8 0)
+    (property "LCSC" "C1710" (id 4) (at 160.02 177.8 0)
       (effects (font (size 1.524 1.524)) hide)
     )

Commit message: Removed SMT Q8
Parts:
- removed Q8: SS8550, Package_TO_SOT_SMD:SOT-23, symbol Transistor_BJT:MMBT3906
- R38: value 22R -> 2R2; LCSC C17561 -> C137549
- renumbered Q16 to Q8
Other:
- moved on the sheet: Q8
Changed lines of the file:
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@@
   (junction (at 234.95 83.82) (diameter 0) (color 0 0 0 0)
   )
-  (junction (at 231.14 16.51) (diameter 0) (color 0 0 0 0)
-  )
   (junction (at 262.89 59.69) (diameter 0) (color 0 0 0 0)
   )
-  (junction (at 237.49 31.75) (diameter 0) (color 0 0 0 0)
-  )
   (junction (at 52.07 58.42) (diameter 0) (color 0 0 0 0)
   )
@@
   (junction (at 81.28 187.96) (diameter 0) (color 0 0 0 0)
   )
-  (junction (at 223.52 26.67) (diameter 0) (color 0 0 0 0)
-  )
   (junction (at 182.88 68.58) (diameter 0) (color 0 0 0 0)
   )
@@
     (stroke (width 0) (type default) (color 0 0 0 0))
   )
-  (wire (pts (xy 231.14 16.51) (xy 237.49 16.51))
+  (wire (pts (xy 215.9 16.51) (xy 237.49 16.51))
     (stroke (width 0) (type default) (color 0 0 0 0))
   )
@@
     (stroke (width 0) (type default) (color 0 0 0 0))
   )
-  (wire (pts (xy 223.52 23.495) (xy 223.52 26.67))
-    (stroke (width 0) (type default) (color 0 0 0 0))
-  )
   (polyline (pts (xy 283.21 109.22) (xy 283.21 162.56))
     (stroke (width 0) (type default) (color 0 0 0 0))
@@
     (stroke (width 0) (type default) (color 0 0 0 0))
   )
-  (wire (pts (xy 231.14 31.75) (xy 237.49 31.75))
-    (stroke (width 0) (type default) (color 0 0 0 0))
-  )
   (wire (pts (xy 146.05 147.32) (xy 146.05 146.05))
     (stroke (width 0) (type default) (color 0 0 0 0))
@@
     (stroke (width 0) (type default) (color 0 0 0 0))
   )
-  (wire (pts (xy 215.9 26.67) (xy 223.52 26.67))
+  (wire (pts (xy 215.9 26.67) (xy 226.06 26.67))
     (stroke (width 0) (type default) (color 0 0 0 0))
   )
@@
     (stroke (width 0) (type default) (color 0 0 0 0))
   )
-  (wire (pts (xy 223.52 26.67) (xy 226.06 26.67))
-    (stroke (width 0) (type default) (color 0 0 0 0))
-  )
   (wire (pts (xy 20.32 175.26) (xy 20.32 173.99))
     (stroke (width 0) (type default) (color 0 0 0 0))
@@
     (stroke (width 0) (type default) (color 0 0 0 0))
   )
-  (wire (pts (xy 231.14 28.575) (xy 231.14 31.75))
-    (stroke (width 0) (type default) (color 0 0 0 0))
-  )
   (wire (pts (xy 146.05 182.88) (xy 140.97 182.88))
     (stroke (width 0) (type default) (color 0 0 0 0))
@@
     (stroke (width 0) (type default) (color 0 0 0 0))
   )
-  (wire (pts (xy 231.14 16.51) (xy 231.14 18.415))
-    (stroke (width 0) (type default) (color 0 0 0 0))
-  )
   (wire (pts (xy 140.97 52.07) (xy 140.97 64.77))
     (stroke (width 0) (type default) (color 0 0 0 0))
@@
     (stroke (width 0) (type default) (color 0 0 0 0))
   )
-  (wire (pts (xy 215.9 16.51) (xy 231.14 16.51))
-    (stroke (width 0) (type default) (color 0 0 0 0))
-  )
   (wire (pts (xy 207.01 60.96) (xy 217.17 60.96))
     (stroke (width 0) (type default) (color 0 0 0 0))
@@
     (in_bom yes) (on_board yes)
     (property "Reference" "R38" (id 0) (at 248.92 43.18 90))
-    (property "Value" "22R" (id 1) (at 246.38 43.18 90))
+    (property "Value" "2R2" (id 1) (at 246.38 43.18 90))
     (property "Footprint" "Resistor_SMD:R_0805_2012Metric_Pad1.20x1.40mm_HandSolder" (id 2) (at 248.158 43.18 90)
       (effects (font (size 1.27 1.27)) hide)
@@
       (effects (font (size 1.27 1.27)) hide)
     )
-    (property "LCSC" "C17561" (id 4) (at 246.38 43.18 90)
+    (property "LCSC" "C137549" (id 4) (at 246.38 43.18 90)
       (effects (font (size 1.524 1.524)) hide)
     )
@@
     (pin "2")
   )
-  (symbol (lib_id "Transistor_BJT:MMBT3906") (at 234.95 26.67 0) (mirror x) (unit 1)
-    (in_bom yes) (on_board yes)
-    (property "Reference" "Q8" (id 0) (at 239.395 28.575 0)
-      (effects (font (size 1.27 1.27)) (justify left))
-    )
-    (property "Value" "SS8550" (id 1) (at 238.76 31.115 0)
-      (effects (font (size 1.27 1.27)) (justify left))
-    )
-    (property "Footprint" "Package_TO_SOT_SMD:SOT-23" (id 2) (at 240.03 24.765 0)
-      (effects (font (size 1.27 1.27) italic) (justify left) hide)
-    )
-    (property "Datasheet" "" (id 3) (at 234.95 26.67 0)
-      (effects (font (size 1.27 1.27)) (justify left) hide)
-    )
-    (property "LCSC" "C8542" (id 4) (at 234.95 26.67 0)
-      (effects (font (size 1.524 1.524)) hide)
-    )
-    (pin "1")
-    (pin "2")
-    (pin "3")
-  )
   (symbol (lib_id "RFBitBangSMT-rescue:C_Small") (at 43.18 185.42 0) (unit 1)
     (in_bom yes) (on_board yes)
@@
     (pin "3")
   )
-  (symbol (lib_id "RFBitBangSMT-rescue:2N3906") (at 228.6 23.495 0) (mirror x) (unit 1)
+  (symbol (lib_id "RFBitBangSMT-rescue:2N3906") (at 234.95 26.67 0) (mirror x) (unit 1)
     (in_bom yes) (on_board yes)
-    (property "Reference" "Q16" (id 0) (at 223.52 18.415 0)
+    (property "Reference" "Q8" (id 0) (at 229.87 21.59 0)
       (effects (font (size 1.27 1.27)) (justify left))
     )
-    (property "Value" "SS8550" (id 1) (at 219.71 20.955 0)
+    (property "Value" "SS8550" (id 1) (at 226.06 24.13 0)
       (effects (font (size 1.27 1.27)) (justify left))
     )
-    (property "Footprint" "Package_TO_SOT_THT:TO-92_Inline_Wide" (id 2) (at 233.68 21.59 0)
+    (property "Footprint" "Package_TO_SOT_THT:TO-92_Inline_Wide" (id 2) (at 240.03 24.765 0)
       (effects (font (size 1.27 1.27) italic) (justify left) hide)
     )
-    (property "Datasheet" "" (id 3) (at 228.6 23.495 0)
+    (property "Datasheet" "" (id 3) (at 234.95 26.67 0)
       (effects (font (size 1.27 1.27)) (justify left) hide)
     )

Commit message: Manufactured RFBitBangSMT
Parts:
- removed C49: 22 uF, Capacitor_SMD:C_0805_2012Metric_Pad1.18x1.45mm_HandSolder, symbol RFBitBangSMT-rescue:C_Small
- removed C50, C52: 10 uF, Capacitor_SMD:C_0805_2012Metric_Pad1.18x1.45mm_HandSolder, symbol RFBitBangSMT-rescue:C_Small
- added C49: 22 uF, Capacitor_THT:CP_Radial_D5.0mm_P2.50mm, symbol RFBitBangSMT-rescue:CP_Small
- added C50, C52: 10 uF, Capacitor_THT:CP_Radial_D5.0mm_P2.50mm, symbol RFBitBangSMT-rescue:CP_Small
- added JP10: BTP, Connector_PinHeader_2.54mm:PinHeader_1x02_P2.54mm_Vertical, symbol RFBitBangSMT-rescue:Jumper_NC_Small
- D6: value D_Zener -> 1N4757
- U6: LCSC C5451727 -> C1509083
Connections:
- net GND: now also C50.2, C52.2, JP10.1
- net at C43.1, L5.2: now also C49.2
- net at Q1.2 (E), R22.1: now also C49.1
- net at Q1.1 (B), R58.1, R60.2: now also C50.1
- net at Q11.1 (B), R61.2: now also C52.1
- net at L11.2, RV4.2: now also JP10.2
Other:
- moved on the sheet: C27, C43, L5, Q9, R21, R22, R41, R51, RV4
