File: RFBitBangSMT/RFBitBangSMTRadio.kicad_sch (KiCad schematic)
At the start: 143 parts, among them J10 si5351mod, J12 Conn_Coaxial, J17 Filt1, J18 Filt2, Q1 MMBT3904, Q10 MMBT3904, Q11 MMBT3904, Q12 MMBT3904, Q13 SS8550, Q15 NC, Q2 MMBT3904, Q3 2N7000, Q5 NC, Q6 2N7000, Q7 2N7000, Q8 SS8550, Q9 2N7000, T1 Trifilar, T2 Trifilar, T3 Current, U4 LM358, U6 SI5351A, Y2 7.X MHz, Y3 25 MHz, Y4 7.X MHz, Y5 7.X MHz

Commit message: Moved PLLBoard to its own project
Parts:
- added C72: 100 nF, Capacitor_SMD:C_0805_2012Metric_Pad1.18x1.45mm_HandSolder, symbol RFBitBangSMT-rescue:C_Small
- added J25: Conn_01x01, Connector_PinHeader_2.00mm:PinHeader_1x01_P2.00mm_Vertical, symbol Connector_Generic:Conn_01x01
- added JP11: TCXO, Jumper:SolderJumper-2_P1.3mm_Open_Pad1.0x1.5mm, symbol Jumper:SolderJumper_2_Open
Connections:
- net GND: now also Y3.2, C72.1, J25.1 (Pin_1)
- net at C47.2, D14.1 (K), R35.2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: now also JP11.2 (B)
- net at Y3.4: now also C72.2, JP11.1 (A)
Other:
- moved on the sheet: D14
Changed lines of the file:
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@@
   (junction (at 189.23 49.53) (diameter 0) (color 0 0 0 0)
   )
+  (junction (at 100.965 44.45) (diameter 0) (color 0 0 0 0)
+  )
   (junction (at 138.43 49.53) (diameter 0) (color 0 0 0 0)
   )
@@
   (junction (at 237.49 35.56) (diameter 0) (color 0 0 0 0)
   )
+  (junction (at 123.19 34.29) (diameter 0) (color 0 0 0 0)
+  )
   (junction (at 109.22 63.5) (diameter 0) (color 0 0 0 0)
   )
@@
   (junction (at 177.8 68.58) (diameter 0) (color 0 0 0 0)
   )
+  (junction (at 109.22 44.45) (diameter 0) (color 0 0 0 0)
+  )
   (junction (at 246.38 59.69) (diameter 0) (color 0 0 0 0)
   )
@@
     (stroke (width 0) (type default) (color 0 0 0 0))
   )
+  (wire (pts (xy 94.615 48.26) (xy 109.22 48.26))
+    (stroke (width 0) (type default) (color 0 0 0 0))
+  )
   (wire (pts (xy 95.25 130.81) (xy 123.19 130.81))
     (stroke (width 0) (type default) (color 0 0 0 0))
@@
     (stroke (width 0) (type default) (color 0 0 0 0))
   )
+  (wire (pts (xy 100.965 44.45) (xy 100.965 41.91))
+    (stroke (width 0) (type default) (color 0 0 0 0))
+  )
   (wire (pts (xy 118.11 194.31) (xy 133.985 194.31))
     (stroke (width 0) (type default) (color 0 0 0 0))
@@
     (stroke (width 0) (type default) (color 0 0 0 0))
   )
+  (wire (pts (xy 100.965 44.45) (xy 101.6 44.45))
+    (stroke (width 0) (type default) (color 0 0 0 0))
+  )
   (wire (pts (xy 152.4 40.64) (xy 152.4 45.72))
     (stroke (width 0) (type default) (color 0 0 0 0))
@@
     (stroke (width 0) (type default) (color 0 0 0 0))
   )
+  (wire (pts (xy 95.885 41.91) (xy 95.885 43.18))
+    (stroke (width 0) (type default) (color 0 0 0 0))
+  )
   (wire (pts (xy 177.8 49.53) (xy 177.8 52.07))
     (stroke (width 0) (type default) (color 0 0 0 0))
@@
     (stroke (width 0) (type default) (color 0 0 0 0))
   )
-  (wire (pts (xy 94.615 48.26) (xy 109.22 48.26))
-    (stroke (width 0) (type default) (color 0 0 0 0))
-  )
   (wire (pts (xy 129.54 160.02) (xy 129.54 163.83))
     (stroke (width 0) (type default) (color 0 0 0 0))
@@
     (stroke (width 0) (type default) (color 0 0 0 0))
   )
-  (wire (pts (xy 109.22 37.465) (xy 109.22 38.1))
+  (wire (pts (xy 109.22 36.83) (xy 109.22 38.1))
     (stroke (width 0) (type default) (color 0 0 0 0))
   )
@@
     (stroke (width 0) (type default) (color 0 0 0 0))
   )
+  (wire (pts (xy 123.19 34.29) (xy 128.27 34.29))
+    (stroke (width 0) (type default) (color 0 0 0 0))
+  )
   (wire (pts (xy 217.17 60.96) (xy 218.44 60.96))
     (stroke (width 0) (type default) (color 0 0 0 0))
@@
     (stroke (width 0) (type default) (color 0 0 0 0))
   )
+  (wire (pts (xy 106.68 53.34) (xy 106.68 47.625))
+    (stroke (width 0) (type default) (color 0 0 0 0))
+  )
   (wire (pts (xy 69.85 31.75) (xy 82.55 31.75))
     (stroke (width 0) (type default) (color 0 0 0 0))
@@
     (stroke (width 0) (type default) (color 0 0 0 0))
   )
+  (wire (pts (xy 106.68 47.625) (xy 100.965 47.625))
+    (stroke (width 0) (type default) (color 0 0 0 0))
+  )
   (wire (pts (xy 223.52 146.05) (xy 223.52 148.59))
     (stroke (width 0) (type default) (color 0 0 0 0))
@@
     (stroke (width 0) (type default) (color 0 0 0 0))
   )
+  (wire (pts (xy 100.965 47.625) (xy 100.965 44.45))
+    (stroke (width 0) (type default) (color 0 0 0 0))
+  )
   (wire (pts (xy 226.06 59.69) (xy 237.49 59.69))
     (stroke (width 0) (type default) (color 0 0 0 0))
@@
     (stroke (width 0) (type default) (color 0 0 0 0))
   )
-  (wire (pts (xy 118.11 41.91) (xy 139.7 41.91))
-    (stroke (width 0) (type default) (color 0 0 0 0))
-  )
   (polyline (pts (xy 20.32 22.86) (xy 90.17 22.86))
     (stroke (width 0) (type default) (color 0 0 0 0))
@@
     (stroke (width 0) (type default) (color 0 0 0 0))
   )
+  (wire (pts (xy 96.52 53.34) (xy 96.52 57.15))
+    (stroke (width 0) (type default) (color 0 0 0 0))
+  )
   (wire (pts (xy 163.83 171.45) (xy 160.02 171.45))
     (stroke (width 0) (type default) (color 0 0 0 0))
@@
     (stroke (width 0) (type default) (color 0 0 0 0))
   )
-  (wire (pts (xy 109.22 45.085) (xy 109.22 48.26))
+  (wire (pts (xy 118.11 41.91) (xy 139.7 41.91))
+    (stroke (width 0) (type default) (color 0 0 0 0))
+  )
+  (wire (pts (xy 109.22 44.45) (xy 109.22 48.26))
     (stroke (width 0) (type default) (color 0 0 0 0))
   )
@@
     (pin "9")
   )
-  (symbol (lib_id "RFBitBangSMT-rescue:D") (at 109.22 41.275 90) (unit 1)
+  (symbol (lib_id "RFBitBangSMT-rescue:D") (at 109.22 40.64 90) (unit 1)
     (in_bom yes) (on_board yes)
-    (property "Reference" "D14" (id 0) (at 106.68 41.275 0))
-    (property "Value" "1N4148" (id 1) (at 111.76 41.275 0))
-    (property "Footprint" "Diode_SMD:D_SOD-123" (id 2) (at 109.22 41.275 0)
+    (property "Reference" "D14" (id 0) (at 106.68 40.64 0))
+    (property "Value" "1N4148" (id 1) (at 111.76 40.64 0))
+    (property "Footprint" "Diode_SMD:D_SOD-123" (id 2) (at 109.22 40.64 0)
       (effects (font (size 1.27 1.27)) hide)
     )
-    (property "Datasheet" "" (id 3) (at 109.22 41.275 0)
+    (property "Datasheet" "" (id 3) (at 109.22 40.64 0)
       (effects (font (size 1.27 1.27)) hide)
     )
-    (property "LCSC" "C81598" (id 4) (at 109.22 41.275 0)
+    (property "LCSC" "C81598" (id 4) (at 109.22 40.64 0)
       (effects (font (size 1.524 1.524)) hide)
     )
@@
     )
   )
+  (symbol (lib_id "Jumper:SolderJumper_2_Open") (at 105.41 44.45 0) (unit 1)
+    (in_bom yes) (on_board yes)
+    (property "Reference" "JP11" (id 0) (at 103.505 40.005 0))
+    (property "Value" "TCXO" (id 1) (at 103.505 41.91 0))
+    (property "Footprint" "Jumper:SolderJumper-2_P1.3mm_Open_Pad1.0x1.5mm" (id 2) (at 105.41 44.45 0)
+      (effects (font (size 1.27 1.27)) hide)
+    )
+    (property "Datasheet" "~" (id 3) (at 105.41 44.45 0)
+      (effects (font (size 1.27 1.27)) hide)
+    )
+    (pin "1")
+    (pin "2")
+  )
+  (symbol (lib_id "RFBitBangSMT-rescue:GND") (at 95.885 43.18 0) (unit 1)
+    (in_bom yes) (on_board yes)
+    (property "Reference" "#PWR0115" (id 0) (at 95.885 49.53 0)
+      (effects (font (size 1.27 1.27)) hide)
+    )
+    (property "Value" "GND" (id 1) (at 95.885 46.99 0))
+    (property "Footprint" "" (id 2) (at 95.885 43.18 0)
+      (effects (font (size 1.27 1.27)) hide)
+    )
+    (property "Datasheet" "" (id 3) (at 95.885 43.18 0)
+      (effects (font (size 1.27 1.27)) hide)
+    )
+    (pin "1")
+  )
   (symbol (lib_id "Transistor_BJT:MMBT3904") (at 49.53 116.84 0) (unit 1)
     (in_bom yes) (on_board yes)
@@
     (pin "1")
   )
+  (symbol (lib_id "Connector_Generic:Conn_01x01") (at 133.35 34.29 0) (unit 1)
+    (in_bom yes) (on_board yes)
+    (property "Reference" "J25" (id 0) (at 136.525 33.02 0)
+      (effects (font (size 1.27 1.27)) (justify left))
+    )
+    (property "Value" "Conn_01x01" (id 1) (at 137.16 35.56 0)
+      (effects (font (size 1.27 1.27)) (justify left))
+    )
+    (property "Footprint" "Connector_PinHeader_2.00mm:PinHeader_1x01_P2.00mm_Vertical" (id 2) (at 133.35 34.29 0)
+      (effects (font (size 1.27 1.27)) hide)
+    )
+    (property "Datasheet" "~" (id 3) (at 133.35 34.29 0)
+      (effects (font (size 1.27 1.27)) hide)
+    )
+    (pin "1")
+  )
   (symbol (lib_id "RFBitBangSMT-rescue:CP_Small") (at 32.385 173.99 270) (unit 1)
     (in_bom yes) (on_board yes)
@@
     )
   )
+  (symbol (lib_id "RFBitBangSMT-rescue:C_Small") (at 98.425 41.91 90) (unit 1)
+    (in_bom yes) (on_board yes)
+    (property "Reference" "C72" (id 0) (at 99.695 36.83 90)
+      (effects (font (size 1.27 1.27)) (justify left))
+    )
+    (property "Value" "100 nF" (id 1) (at 101.6 38.735 90)
+      (effects (font (size 1.27 1.27)) (justify left))
+    )
+    (property "Footprint" "Capacitor_SMD:C_0805_2012Metric_Pad1.18x1.45mm_HandSolder" (id 2) (at 98.425 41.91 0)
+      (effects (font (size 1.27 1.27)) hide)
+    )
+    (property "Datasheet" "" (id 3) (at 98.425 41.91 0)
+      (effects (font (size 1.27 1.27)) hide)
+    )
+    (property "LCSC" "C49678" (id 4) (at 98.425 41.91 0)
+      (effects (font (size 1.524 1.524)) hide)
+    )
+    (pin "1")
+    (pin "2")
+  )
   (symbol (lib_id "RFBitBangSMT-rescue:C_Small") (at 105.41 175.26 90) (unit 1)
     (in_bom yes) (on_board yes)
@@
     )
   )
+  (symbol (lib_id "RFBitBangSMT-rescue:GND") (at 96.52 57.15 0) (unit 1)
+    (in_bom yes) (on_board yes)
+    (property "Reference" "#PWR0116" (id 0) (at 96.52 63.5 0)
+      (effects (font (size 1.27 1.27)) hide)
+    )
+    (property "Value" "GND" (id 1) (at 96.52 60.96 0))
+    (property "Footprint" "" (id 2) (at 96.52 57.15 0)
+      (effects (font (size 1.27 1.27)) hide)
+    )
+    (property "Datasheet" "" (id 3) (at 96.52 57.15 0)
+      (effects (font (size 1.27 1.27)) hide)
+    )
+    (pin "1")
+  )
   (symbol (lib_id "Mechanical:MountingHole") (at 120.65 88.9 0) (unit 1)
