File: SerialResonantFilterSMT/SerialResonantFilter.kicad_sch (KiCad schematic)
At the start: 44 parts, among them J1 OUT, J2 INP, J3 INP, J4 OUT, J5 INP, J6 OUT, J7 INP, J8 OUT

Commit message: Made six panel version of SerialResonantFilterSMT
Parts:
- added C29, C32: 330 pF, Capacitor_SMD:C_1206_3216Metric_Pad1.33x1.80mm_HandSolder, symbol SerialResonantFilter-rescue:C_Small
- added C30, C33: 150 pF, Capacitor_SMD:C_1206_3216Metric_Pad1.33x1.80mm_HandSolder, symbol SerialResonantFilter-rescue:C_Small
- added C31, C34, C51, C52: 470 pF, Capacitor_SMD:C_1206_3216Metric_Pad1.33x1.80mm_HandSolder, symbol SerialResonantFilter-rescue:C_Small
- added C35, C38: 680 pF, Capacitor_SMD:C_1206_3216Metric_Pad1.33x1.80mm_HandSolder, symbol SerialResonantFilter-rescue:C_Small
- added C36, C39: 2200 pF, Capacitor_SMD:C_1206_3216Metric_Pad1.33x1.80mm_HandSolder, symbol SerialResonantFilter-rescue:C_Small
- added C37, C40, C57, C58: 1000 pF, Capacitor_SMD:C_1206_3216Metric_Pad1.33x1.80mm_HandSolder, symbol SerialResonantFilter-rescue:C_Small
- added C41, C44, C46, C47: 100 pF, Capacitor_SMD:C_1206_3216Metric_Pad1.33x1.80mm_HandSolder, symbol SerialResonantFilter-rescue:C_Small
- added C42, C45: 47 pF, Capacitor_SMD:C_1206_3216Metric_Pad1.33x1.80mm_HandSolder, symbol SerialResonantFilter-rescue:C_Small
- added C43, C48: 220 pF, Capacitor_SMD:C_1206_3216Metric_Pad1.33x1.80mm_HandSolder, symbol SerialResonantFilter-rescue:C_Small
- added C49, C50: 33 pF, Capacitor_SMD:C_1206_3216Metric_Pad1.33x1.80mm_HandSolder, symbol SerialResonantFilter-rescue:C_Small
- added C53, C54: 68 pF, Capacitor_SMD:C_1206_3216Metric_Pad1.33x1.80mm_HandSolder, symbol SerialResonantFilter-rescue:C_Small
- added C55, C56: 1500 pF, Capacitor_SMD:C_1206_3216Metric_Pad1.33x1.80mm_HandSolder, symbol SerialResonantFilter-rescue:C_Small
- C1: value C1 -> 330 pF
- C10: value C2 -> 470 pF
- C11: value C4 -> 470 pF
- C13: value C5 -> 150 pF; LCSC C577182 -> C577189
- C14: value C6 -> 470 pF
- C15: value C1 -> 680 pF
- C17: value C2 -> 2200 pF
- C18: value C4 -> 2200 pF
- C2: value C2 -> 1000 pF
- C20: value C5 -> 680 pF
- C21: value C6 -> 2200 pF
- C22, C27: LCSC C527299 -> (none)
- C24: LCSC C527339 -> (none)
- C25, C28: Field4 C527339 -> (none)
- C4: value C4 -> 1000 pF
- C5: value C5 -> 330 pF
- C6: value C6 -> 1000 pF
- C8: value C1 -> 150 pF; LCSC C577182 -> C577189
- L1: value L2 -> 0.39 uH
- L2: value L2 -> 0.77 uH
- L3: value L3 -> 0.36 uH
- L4: value L3 -> 0.18 uH
- L5: value L2 -> 1.45 uH
- L6: value L3 -> 0.68 uH
